Commit message: adding ray to TOF sensor

File: ros_ws/src/pipe_swarm/urdf/tof.xacro (robot description, xacro)
@@ -36,4 +36,17 @@
             <visualize>true</visualize>
             <update_rate>10.0</update_rate>
+            <ray>
+                <scan>
+                    <horizontal>
+                        <samples>10</samples>
+                        <resolution>1</resolution>
+                    </horizontal>
+                </scan>
+                <range>
+                    <min>0.1</min>
+                    <max>10.0</max>
+                    <resolution>0.01</resolution>
+                </range>
+            </ray>
             <plugin name="tof_controller" filename="libgazebo_ros_ray_sensor.so">
                 <ros>
@@ -42,11 +55,7 @@
                 </ros>
                 <output_type>sensor_msgs/Range</output_type>
-                <min_intensity>100.0</min_intensity>
                 <frame_name>${agent_namespace}_tof_link</frame_name>
             </plugin>
         </sensor>
     </gazebo>
-    <gazebo reference="${agent_namespace}_tof_link">
-        <material>Gazebo/Red</material>
-    </gazebo>
 </robot>

Commit message: adding dual time of flight sensors facing sideways

File: ros_ws/src/pipe_swarm/urdf/tof.xacro (robot description, xacro)
@@ -6,5 +6,22 @@
     <xacro:property name="tof_h" value="0.01" />  <!-- height /m -->
     <!-- LINKS -->
-    <link name="${agent_namespace}_tof_link">
+    <link name="${agent_namespace}_right_tof_link">
+        <visual>
+            <origin xyz="0.0 0.0 0.0" rpy="0.0 0.0 0.0"/>
+            <geometry>
+                <box size="${tof_w} ${tof_l} ${tof_h}"/>
+            </geometry>
+            <material name="red">
+                <color rgba="1 0 0 1"/>
+            </material>
+        </visual>
+        <collision>
+            <geometry>
+                <box size="${tof_w} ${tof_l} ${tof_h}"/>
+            </geometry>
+        </collision>
+        <xacro:box_inertial m="${tof_m}" w="${tof_w}" l="${tof_l}" h="${tof_h}" xyz="0 0 0 " rpy="0 0 0"/>
+    </link>
+    <link name="${agent_namespace}_left_tof_link">
         <visual>
             <origin xyz="0.0 0.0 0.0" rpy="0.0 0.0 0.0"/>
@@ -24,13 +41,18 @@
     </link>
     <!-- JOINTS -->
-    <joint name="${agent_namespace}_base_tof_joint" type="fixed">
-        <origin xyz="${-(base_w*0.5)} 0 ${(base_h*0.5)+(tof_h*0.5)}" rpy="0 0 ${pi}"/>
+    <joint name="${agent_namespace}_base_right_tof_joint" type="fixed">
+        <origin xyz="0 ${-(base_l*0.5)} ${(base_h*0.5)+(tof_h*0.5)}" rpy="0 0 ${-pi/2}"/>
         <parent link="${agent_namespace}_base_link"/>
-        <child link="${agent_namespace}_tof_link"/>
+        <child link="${agent_namespace}_right_tof_link"/>
+    </joint>
+    <joint name="${agent_namespace}_base_left_tof_joint" type="fixed">
+        <origin xyz="0 ${(base_l*0.5)} ${(base_h*0.5)+(tof_h*0.5)}" rpy="0 0 ${pi/2}"/>
+        <parent link="${agent_namespace}_base_link"/>
+        <child link="${agent_namespace}_left_tof_link"/>
     </joint>
     <!-- GAZEBO -->
-    <gazebo reference="${agent_namespace}_tof_link">
+    <gazebo reference="${agent_namespace}_right_tof_link">
         <material>Gazebo/Green</material>
-        <sensor name="tof_sensor" type="ray">
+        <sensor name="${agent_namespace}_right_tof_sensor" type="ray">
             <pose>0 0 0 0 0 0</pose>
             <visualize>true</visualize>
@@ -49,11 +71,42 @@
                 </range>
             </ray>
-            <plugin name="tof_controller" filename="libgazebo_ros_ray_sensor.so">
+            <plugin name="${agent_namespace}_right_tof_controller" filename="libgazebo_ros_ray_sensor.so">
                 <ros>
                     <namespace>${agent_namespace}</namespace>
-                    <remapping>~/out:=infrared_range</remapping>
+                    <remapping>~/out:=right_infrared_range</remapping>
                 </ros>
                 <output_type>sensor_msgs/Range</output_type>
-                <frame_name>${agent_namespace}_tof_link</frame_name>
+                <radiation_type>infrared</radiation_type>
+                <frame_name>${agent_namespace}_right_tof_link</frame_name>
+            </plugin>
+        </sensor>
+    </gazebo>
+    <gazebo reference="${agent_namespace}_left_tof_link">
+        <material>Gazebo/Green</material>
+        <sensor name="${agent_namespace}_left_tof_sensor" type="ray">
+            <pose>0 0 0 0 0 0</pose>
+            <visualize>true</visualize>
+            <update_rate>10.0</update_rate>
+            <ray>
+                <scan>
+                    <horizontal>
+                        <samples>10</samples>
+                        <resolution>1</resolution>
+                    </horizontal>
+                </scan>
+                <range>
+                    <min>0.1</min>
+                    <max>10.0</max>
+                    <resolution>0.01</resolution>
+                </range>
+            </ray>
+            <plugin name="${agent_namespace}_left_tof_controller" filename="libgazebo_ros_ray_sensor.so">
+                <ros>
+                    <namespace>${agent_namespace}</namespace>
+                    <remapping>~/out:=left_infrared_range</remapping>
+                </ros>
+                <output_type>sensor_msgs/Range</output_type>
+                <frame_name>${agent_namespace}_left_tof_link</frame_name>
+                <radiation_type>infrared</radiation_type>
             </plugin>
         </sensor>
