Commit message: New File Changes

File: ros_ws/src/pipe_swarm/urdf/lidar.xacro (robot description, xacro)
@@ -25,5 +25,5 @@
     <!-- JOINTS -->
     <joint name="${agent_namespace}_base_lidar_joint" type="fixed">
-        <origin xyz="0 ${-(base_l*0.5 + lidar_l*0.5)} 0" rpy="${pi/2} 0 0"/>
+        <origin xyz="${(base_w*0.5)} ${-(base_l*0.5 - lidar_l*0.5)} ${(base_h*0.5)}" rpy="${pi/2} 0 0"/>
         <parent link="${agent_namespace}_base_link"/>
         <child link="${agent_namespace}_lidar_link"/>

File: ros_ws/src/pipe_swarm/urdf/pipe_robot.urdf.xacro (robot description, xacro)
@@ -5,6 +5,6 @@
     <xacro:include filename="mobile_base.xacro"/>
     <xacro:include filename="lidar.xacro"/>
-    <xacro:include filename="tof.xacro"/>
-    <xacro:include filename="camera.xacro"/>
+    <!-- <xacro:include filename="tof.xacro"/> -->
+    <!-- <xacro:include filename="camera.xacro"/> -->
     <xacro:include filename="wheels.xacro"/>
     <xacro:include filename="linkage.xacro"/>
