Commit message: Move IMU to robot bottom

File: ros_ws/src/pipe_swarm/urdf/imu.xacro (robot description, xacro)
@@ -25,5 +25,5 @@
     <!-- JOINTS -->
     <joint name="${agent_namespace}_base_imu_joint" type="fixed">
-        <origin xyz="${(base_w*0.5)} ${(base_l*0.5 - imu_l*0.5)} ${(base_h*0.5)}" rpy="0 0 ${-pi/2}"/>
+        <origin xyz="0 0 ${-(base_h*0.5)}" rpy="0 0 ${-pi/2}"/>
         <parent link="${agent_namespace}_base_link"/>
         <child link="${agent_namespace}_imu_link"/>
