Commit message: varying whether URDF uses gazebo

File: ros_ws/src/pipe_swarm/urdf/pipe_agent.urdf.xacro (robot description, xacro)
@@ -5,4 +5,4 @@
     <xacro:include filename="pipe_robot.xacro"/>
     <!-- Call pipe_robot with agent_namespace -->
-    <xacro:pipe_robot namespace="${agent_namespace}" />
+    <xacro:pipe_robot namespace="${agent_namespace}" include_gazebo="true"/>
 </robot>

File: ros_ws/src/pipe_swarm/urdf/pipe_robot.xacro (robot description, xacro)
@@ -1,5 +1,5 @@
 <?xml version="1.0"?>
 <robot name="pipe_robot" xmlns:xacro="http://www.ros.org/wiki/xacro">
-    <xacro:macro name="pipe_robot" params="namespace">
+    <xacro:macro name="pipe_robot" params="namespace include_gazebo">
         <xacro:property name="agent_namespace" value="${namespace}" />
         <!-- Include shared components -->
@@ -11,5 +11,7 @@
         <xacro:include filename="wheels.xacro"/>
         <xacro:include filename="linkage.xacro"/>
-        <xacro:include filename="gazebo/pipe_robot.xacro"/>
+        <xacro:if value="${include_gazebo}">
+            <xacro:include filename="gazebo/pipe_robot.xacro"/>
+        </xacro:if>
     </xacro:macro>
 </robot>
