Commit message: adjusting robot body length

File: ros_ws/src/pipe_swarm/urdf/mobile_base.xacro (robot description, xacro)
@@ -3,5 +3,5 @@
     <xacro:property name="base_m" value="1" />  <!-- mass /kg -->
     <xacro:property name="base_w" value="0.15" />  <!-- width /m -->
-    <xacro:property name="base_l" value="0.075" />  <!-- length /m -->
+    <xacro:property name="base_l" value="0.05" />  <!-- length /m -->
     <xacro:property name="base_h" value="0.045" />  <!-- height /m -->
     <!-- LINKS -->

Commit message: Changes to base

File: ros_ws/src/pipe_swarm/urdf/mobile_base.xacro (robot description, xacro)
@@ -2,7 +2,7 @@
 <robot name="mobile_base" xmlns:xacro="http://www.ros.org/wiki/xacro">
     <xacro:property name="base_m" value="1" />  <!-- mass /kg -->
-    <xacro:property name="base_w" value="0.15" />  <!-- width /m -->
-    <xacro:property name="base_l" value="0.05" />  <!-- length /m -->
-    <xacro:property name="base_h" value="0.045" />  <!-- height /m -->
+    <xacro:property name="base_w" value="0.1045" />  <!-- width /m -->
+    <xacro:property name="base_l" value="0.055" />  <!-- length /m -->
+    <xacro:property name="base_h" value="0.062" />  <!-- height /m -->
     <!-- LINKS -->
     <link name="${agent_namespace}_footprint_link" />

Commit message: using multiple boxes for base link to include gap within male linkage

File: ros_ws/src/pipe_swarm/urdf/mobile_base.xacro (robot description, xacro)
@@ -3,5 +3,8 @@
     <xacro:property name="base_m" value="1" />  <!-- mass /kg -->
     <xacro:property name="base_w" value="0.1045" />  <!-- width /m -->
+    <xacro:property name="base_w_offset" value="0.05" />  <!-- offset /m -->
+    <xacro:property name="base_w_main" value="${base_w - base_w_offset}" />  <!-- width /m -->
     <xacro:property name="base_l" value="0.055" />  <!-- length /m -->
+    <xacro:property name="base_l_offset" value="0.015" />  <!-- length /m -->
     <xacro:property name="base_h" value="0.062" />  <!-- height /m -->
     <!-- LINKS -->
@@ -9,7 +12,43 @@
     <link name="${agent_namespace}_base_link">
         <visual>
-            <origin xyz="0.0 0.0 0.0" rpy="0.0 0.0 0.0"/>
+            <origin xyz="${(-base_w/2)+(base_w_main/2)} 0 0" rpy="0 0 0"/>
             <geometry>
-                <box size="${base_w} ${base_l} ${base_h}"/>
+                <box size="${base_w_main} ${base_l} ${base_h}"/>
+            </geometry>
+            <material name="blue">
+                <color rgba="0 0 1 1"/>
+            </material>
+        </visual>
+        <visual>
+            <origin xyz="${(base_w/2)-(base_w_offset/2)} ${(base_l/2) - (base_l_offset/2)} 0" rpy="0 0 0"/>
+            <geometry>
+                <box size="${base_w_offset} ${base_l_offset} ${base_h}"/>
+            </geometry>
+            <material name="blue">
+                <color rgba="0 0 1 1"/>
+            </material>
+        </visual>
+        <visual>
+            <origin xyz="${(base_w/2)-(base_w_offset/2)} ${-((base_l/2) - (base_l_offset/2))} 0" rpy="0 0 0"/>
+            <geometry>
+                <box size="${base_w_offset} ${base_l_offset} ${base_h}"/>
+            </geometry>
+            <material name="blue">
+                <color rgba="0 0 1 1"/>
+            </material>
+        </visual>
+        <visual>
+            <origin xyz="${(base_w/2)-(base_w_offset/2)} 0 ${(base_l/2) - (base_l_offset/2)}" rpy="0 0 0"/>
+            <geometry>
+                <box size="${base_w_offset} ${base_l} ${base_l_offset}"/>
+            </geometry>
+            <material name="blue">
+                <color rgba="0 0 1 1"/>
+            </material>
+        </visual>
+        <visual>
+            <origin xyz="${(base_w/2)-(base_w_offset/2)} 0 ${-((base_l/2) - (base_l_offset/2))}" rpy="0 0 0"/>
+            <geometry>
+                <box size="${base_w_offset} ${base_l} ${base_l_offset}"/>
             </geometry>
             <material name="blue">
@@ -18,6 +57,31 @@
         </visual>
         <collision>
+            <origin xyz="${(-base_w/2)+(base_w_main/2)} 0 0" rpy="0 0 0"/>
             <geometry>
-                <box size="${base_w} ${base_l} ${base_h}"/>
+                <box size="${base_w_main} ${base_l} ${base_h}"/>
+            </geometry>
+        </collision>
+        <collision>
+            <origin xyz="${(base_w/2)-(base_w_offset/2)} ${(base_l/2) - (base_l_offset/2)} 0" rpy="0 0 0"/>
+            <geometry>
+                <box size="${base_w_offset} ${base_l_offset} ${base_h}"/>
+            </geometry>
+        </collision>
+        <collision>
+            <origin xyz="${(base_w/2)-(base_w_offset/2)} ${-((base_l/2) - (base_l_offset/2))} 0" rpy="0 0 0"/>
+            <geometry>
+                <box size="${base_w_offset} ${base_l_offset} ${base_h}"/>
+            </geometry>
+        </collision>
+        <collision>
+            <origin xyz="${(base_w/2)-(base_w_offset/2)} 0 ${(base_l/2) - (base_l_offset/2)}" rpy="0 0 0"/>
+            <geometry>
+                <box size="${base_w_offset} ${base_l} ${base_l_offset}"/>
+            </geometry>
+        </collision>
+        <collision>
+            <origin xyz="${(base_w/2)-(base_w_offset/2)} 0 ${-((base_l/2) - (base_l_offset/2))}" rpy="0 0 0"/>
+            <geometry>
+                <box size="${base_w_offset} ${base_l} ${base_l_offset}"/>
             </geometry>
         </collision>

Commit message: Closed material tag

File: ros_ws/src/pipe_swarm/urdf/mobile_base.xacro (robot description, xacro)
@@ -26,4 +26,6 @@
             </geometry>
             <material name="grey">
+                <color rgba="0.86 0.86 0.86 1"/>
+            </material>
         </visual>
         <visual>
@@ -33,4 +35,6 @@
             </geometry>
             <material name="grey">
+                    <color rgba="0.86 0.86 0.86 1"/>
+            </material>
         </visual>
         <visual>
@@ -40,4 +44,6 @@
             </geometry>
             <material name="grey">
+                    <color rgba="0.86 0.86 0.86 1"/>
+            </material>
         </visual>
         <visual>
@@ -47,4 +53,6 @@
             </geometry>
             <material name="grey">
+                    <color rgba="0.86 0.86 0.86 1"/>
+            </material>
         </visual>
         <collision>

Commit message: Missing material closing line added

File: ros_ws/src/pipe_swarm/urdf/mobile_base.xacro (robot description, xacro)
@@ -26,4 +26,6 @@
             </geometry>
             <material name="grey">
+                <color rgba="0.86 0.86 0.86 1"/>
+            </material>
         </visual>
         <visual>
@@ -33,4 +35,6 @@
             </geometry>
             <material name="grey">
+                <color rgba="0.86 0.86 0.86 1"/>
+            </material>
         </visual>
         <visual>
@@ -40,4 +44,6 @@
             </geometry>
             <material name="grey">
+                <color rgba="0.86 0.86 0.86 1"/>
+            </material>
         </visual>
         <visual>
@@ -47,4 +53,6 @@
             </geometry>
             <material name="grey">
+                <color rgba="0.86 0.86 0.86 1"/>
+            </material>
         </visual>
         <collision>
