Commit message: fixing wheels with new stl

File: ros_ws/src/pipe_swarm/urdf/wheels.xacro (robot description, xacro)
@@ -2,6 +2,6 @@
 <robot name="wheels" xmlns:xacro="http://www.ros.org/wiki/xacro">
     <xacro:property name="wheel_m" value="0.1" />  <!-- mass /kg -->
-    <xacro:property name="wheel_r" value="0.0175" />  <!-- radius /m -->
-    <xacro:property name="wheel_l" value="0.01" />  <!-- length /m -->
+    <xacro:property name="wheel_r" value="0.015" />  <!-- radius /m -->
+    <xacro:property name="wheel_l" value="0.008" />  <!-- length /m 8 or 3 -->
     <xacro:property name="wheel_y_offset" value="0.002" />  <!-- length /m -->
     <xacro:property name="wheel_x_offset_front" value="0.012" />  <!-- length /m -->
@@ -10,5 +10,5 @@
         <link name="${agent_namespace}_wheel_${prefix}_left_link">
             <visual>
-                <origin xyz="0.0 0.0 0.0" rpy="0 0.0 0.0"/>
+                <origin xyz="${-wheel_r} ${-wheel_r} ${-wheel_l/2}" rpy="0 0 0"/>
                 <geometry>
                     <mesh filename="package://pipe_swarm/models/hollow_pipe/meshes/wheel.stl" scale="0.001 0.001 0.001"/>
@@ -20,5 +20,5 @@
             </visual>
             <collision>
-                <origin xyz="0.0 0.0 0.0" rpy="0 0.0 0.0"/>
+                <origin xyz="${-wheel_r} ${-wheel_r} ${-wheel_l/2}" rpy="0 0 0"/>
                 <geometry>
                     <mesh filename="package://pipe_swarm/models/hollow_pipe/meshes/wheel.stl" scale="0.001 0.001 0.001"/>
@@ -30,5 +30,5 @@
         <link name="${agent_namespace}_wheel_${prefix}_right_link">
             <visual>
-                <origin xyz="0.0 0.0 0.0" rpy="0 0.0 0.0"/>
+                <origin xyz="${-wheel_r} ${-wheel_r} ${-wheel_l/2}" rpy="0 0 0"/>
                 <geometry>
                     <mesh filename="package://pipe_swarm/models/hollow_pipe/meshes/wheel.stl" scale="0.001 0.001 0.001"/>
@@ -40,5 +40,5 @@
             </visual>
             <collision>
-                <origin xyz="0.0 0.0 0.0" rpy="0 0.0 0.0"/>
+                <origin xyz="${-wheel_r} ${-wheel_r} ${-wheel_l/2}" rpy="0 0 0"/>
                 <geometry>
                     <mesh filename="package://pipe_swarm/models/hollow_pipe/meshes/wheel.stl" scale="0.001 0.001 0.001"/>
@@ -54,5 +54,5 @@
     <!-- JOINTS -->
     <joint name="${agent_namespace}_base_wheel_front_right_joint" type="continuous">
-        <origin xyz="${(base_w)/2 - wheel_x_offset_front} ${-((base_l/2) + wheel_y_offset)} ${-base_h/2}" rpy="${-pi/2} 0 0"/>
+        <origin xyz="${(base_w)/2 - wheel_x_offset_front} ${-((base_l/2) + (wheel_l/2) + wheel_y_offset)} ${-base_h/2}" rpy="${-pi/2} 0 0"/>
         <parent link="${agent_namespace}_base_link"/>
         <child link="${agent_namespace}_wheel_front_right_link"/>
@@ -60,5 +60,5 @@
     </joint>
     <joint name="${agent_namespace}_base_wheel_front_left_joint" type="continuous">
-        <origin xyz="${(base_w)/2 - wheel_x_offset_front} ${(base_l/2) + wheel_y_offset} ${-base_h/2}" rpy="${pi/2} 0 0"/>
+        <origin xyz="${(base_w)/2 - wheel_x_offset_front} ${(base_l/2) + (wheel_l/2) + wheel_y_offset} ${-base_h/2}" rpy="${pi/2} 0 0"/>
         <parent link="${agent_namespace}_base_link"/>
         <child link="${agent_namespace}_wheel_front_left_link"/>
@@ -66,5 +66,5 @@
     </joint>
     <joint name="${agent_namespace}_base_wheel_back_right_joint" type="continuous">
-        <origin xyz="${-((base_w)/2 - wheel_x_offset_back)} ${-((base_l/2) + wheel_y_offset)} ${-base_h/2}" rpy="${-pi/2} 0 0"/>
+        <origin xyz="${-((base_w)/2 - wheel_x_offset_back)} ${-((base_l/2) + (wheel_l/2) + wheel_y_offset)} ${-base_h/2}" rpy="${-pi/2} 0 0"/>
         <parent link="${agent_namespace}_base_link"/>
         <child link="${agent_namespace}_wheel_back_right_link"/>
@@ -73,5 +73,5 @@
     </joint>
     <joint name="${agent_namespace}_base_wheel_back_left_joint" type="continuous">
-        <origin xyz="${-((base_w)/2 - wheel_x_offset_back)} ${(base_l/2) + wheel_y_offset} ${-base_h/2}" rpy="${pi/2} 0 0"/>
+        <origin xyz="${-((base_w)/2 - wheel_x_offset_back)} ${(base_l/2) + (wheel_l/2) + wheel_y_offset} ${-base_h/2}" rpy="${pi/2} 0 0"/>
         <parent link="${agent_namespace}_base_link"/>
         <child link="${agent_namespace}_wheel_back_left_link"/>
