Commit message: renaming front_tof properties

File: ros_ws/src/pipe_swarm/urdf/front_tof.xacro (robot description, xacro)
@@ -1,14 +1,14 @@
 <?xml version="1.0"?>
 <robot name="front_tof" xmlns:xacro="http://www.ros.org/wiki/xacro">
-    <xacro:property name="tof_m" value="0.1" />  <!-- mass /kg -->
-    <xacro:property name="tof_w" value="0.01" />  <!-- width /m -->
-    <xacro:property name="tof_l" value="0.01" />  <!-- length /m -->
-    <xacro:property name="tof_h" value="0.01" />  <!-- height /m -->
+    <xacro:property name="front_tof_m" value="0.1" />  <!-- mass /kg -->
+    <xacro:property name="front_tof_w" value="0.01" />  <!-- width /m -->
+    <xacro:property name="front_tof_l" value="0.01" />  <!-- length /m -->
+    <xacro:property name="front_tof_h" value="0.01" />  <!-- height /m -->
     <!-- LINKS -->
-    <link name="${agent_namespace}_tof_link">
+    <link name="${agent_namespace}_front_tof_link">
         <visual>
             <origin xyz="0.0 0.0 0.0" rpy="0.0 0.0 0.0"/>
             <geometry>
-                <box size="${tof_w} ${tof_l} ${tof_h}"/>
+                <box size="${front_tof_w} ${front_tof_l} ${front_tof_h}"/>
             </geometry>
             <material name="red">
@@ -18,14 +18,14 @@
         <collision>
             <geometry>
-                <box size="${tof_w} ${tof_l} ${tof_h}"/>
+                <box size="${front_tof_w} ${front_tof_l} ${front_tof_h}"/>
             </geometry>
         </collision>
-        <xacro:box_inertial m="${tof_m}" w="${tof_w}" l="${tof_l}" h="${tof_h}" xyz="0 0 0 " rpy="0 0 0"/>
+        <xacro:box_inertial m="${front_tof_m}" w="${front_tof_w}" l="${front_tof_l}" h="${front_tof_h}" xyz="0 0 0 " rpy="0 0 0"/>
     </link>
     <!-- JOINTS -->
-    <joint name="${agent_namespace}_base_tof_joint" type="fixed">
-        <origin xyz="${(base_w*0.5)} ${-(base_l*0.5 - tof_l)} ${(base_h*0.5)}" rpy="${pi/2} 0 0"/>
+    <joint name="${agent_namespace}_base_front_tof_joint" type="fixed">
+        <origin xyz="${(base_w/2)} ${-(base_l/2 - front_tof_l)} ${(base_h/2)}" rpy="${pi/2} 0 0"/>
         <parent link="${agent_namespace}_base_link"/>
-        <child link="${agent_namespace}_tof_link"/>
+        <child link="${agent_namespace}_front_tof_link"/>
     </joint>
 </robot>

File: ros_ws/src/pipe_swarm/urdf/gazebo/pipe_robot.xacro (robot description, xacro)
@@ -4,13 +4,13 @@
         <!-- Include shared components -->
         <xacro:include filename="mobile_base.xacro"/>
+        <xacro:include filename="imu.xacro"/>
         <!-- <xacro:include filename="lidar.xacro"/> -->
-        <xacro:include filename="imu.xacro"/>
-        <xacro:include filename="tof_lidar.xacro"/>
-        <xacro:include filename="tof.xacro"/>
+        <!-- <xacro:include filename="tof_lidar.xacro"/> -->
+        <!-- <xacro:include filename="tof.xacro"/> -->
+        <xacro:include filename="front_tof.xacro"/>
         <xacro:include filename="camera.xacro"/>
         <xacro:include filename="linkage.xacro"/>
         <xacro:include filename="wheels.xacro"/>
         <xacro:include filename="detection_object.xacro"/>
-        <xacro:include filename="front_tof.xacro"/>
     </xacro:macro>
     <xacro:gazebo_pipe_robot namespace="${agent_namespace}" />

File: ros_ws/src/pipe_swarm/urdf/pipe_robot.xacro (robot description, xacro)
@@ -6,9 +6,9 @@
         <xacro:include filename="common.xacro"/>
         <xacro:include filename="mobile_base.xacro"/>
+        <xacro:include filename="imu.xacro"/>
         <!-- <xacro:include filename="lidar.xacro"/> -->
-        <xacro:include filename="imu.xacro"/>
         <!-- <xacro:include filename="tof_lidar.xacro"/> -->
+        <!-- <xacro:include filename="tof.xacro"/> -->
         <xacro:include filename="front_tof.xacro"/>
-        <!-- <xacro:include filename="tof.xacro"/> -->
         <xacro:include filename="camera.xacro"/>
         <xacro:include filename="linkage.xacro"/>

Commit message: Updating name and moving inwards sensor

File: ros_ws/src/pipe_swarm/urdf/front_tof.xacro (robot description, xacro)
@@ -25,5 +25,5 @@
     <!-- JOINTS -->
     <joint name="${agent_namespace}_base_front_tof_joint" type="fixed">
-        <origin xyz="${(base_w/2)} ${-(base_l/2 - front_tof_l)} ${(base_h/2)}" rpy="${pi/2} 0 0"/>
+        <origin xyz="${(base_w/2)} ${-(base_l/2 - front_tof_l*2)} ${(base_h/2)}" rpy="${pi/2} 0 0"/>
         <parent link="${agent_namespace}_base_link"/>
         <child link="${agent_namespace}_front_tof_link"/>

File: ros_ws/src/pipe_swarm/urdf/gazebo/front_tof.xacro (robot description, xacro)
@@ -2,7 +2,7 @@
 <robot name="gazebo_front_tof" xmlns:xacro="http://www.ros.org/wiki/xacro">
     <!-- GAZEBO -->
-    <gazebo reference="${agent_namespace}_tof_link">
+    <gazebo reference="${agent_namespace}_front_tof_link">
         <material>Gazebo/Green</material>
-        <sensor name="${agent_namespace}_tof_sensor" type="ray">
+        <sensor name="${agent_namespace}_front_tof_sensor" type="ray">
             <pose>0 0 0 0 ${pi/2} 0</pose>
             <visualize>true</visualize>
@@ -23,5 +23,5 @@
                 </range>
             </ray>
-            <plugin name="${agent_namespace}_tof_controller" filename="libgazebo_ros_ray_sensor.so">
+            <plugin name="${agent_namespace}_front_tof_controller" filename="libgazebo_ros_ray_sensor.so">
                 <ros>
                     <namespace>${agent_namespace}</namespace>
