Commit message: Added obstacles so the camera/obstacle detection works only straight on

File: ros_ws/src/pipe_swarm/urdf/detection_object.xacro (robot description, xacro)
@@ -6,4 +6,5 @@
     <xacro:property name="obstacle_h" value="0.01" />  <!-- height /m -->
     <!-- LINKS -->
+    <!-- Red Box -->
     <link name="${agent_namespace}_obstacle_link">
         <visual>
@@ -23,9 +24,55 @@
         <xacro:box_inertial m="${obstacle_m}" w="${obstacle_w}" l="${obstacle_l}" h="${obstacle_h}" xyz="0 0 0 " rpy="0 0 0"/>
     </link>
+    <!-- White Box 1 -->
+    <link name="${agent_namespace}_white_box_1_link">
+        <visual>
+            <origin xyz="0.0 0.0 0.0" rpy="0.0 0.0 0.0"/>
+            <geometry>
+                <box size="${obstacle_w} ${obstacle_l} ${obstacle_h}"/>
+            </geometry>
+            <material name="white">
+                <color rgba="1 1 1 1"/>
+            </material>
+        </visual>
+        <collision>
+            <geometry>
+                <box size="${obstacle_w} ${obstacle_l} ${obstacle_h}"/>
+            </geometry>
+        </collision>
+        <xacro:box_inertial m="${obstacle_m}" w="${obstacle_w}" l="${obstacle_l}" h="${obstacle_h}" xyz="0 0 0 " rpy="0 0 0"/>
+    </link>
+    <!-- White Box 2 -->
+    <link name="${agent_namespace}_white_box_2_link">
+        <visual>
+            <origin xyz="0.0 0.0 0.0" rpy="0.0 0.0 0.0"/>
+            <geometry>
+                <box size="${obstacle_w} ${obstacle_l} ${obstacle_h}"/>
+            </geometry>
+            <material name="white">
+                <color rgba="1 1 1 1"/>
+            </material>
+        </visual>
+        <collision>
+            <geometry>
+                <box size="${obstacle_w} ${obstacle_l} ${obstacle_h}"/>
+            </geometry>
+        </collision>
+        <xacro:box_inertial m="${obstacle_m}" w="${obstacle_w}" l="${obstacle_l}" h="${obstacle_h}" xyz="0 0 0 " rpy="0 0 0"/>
+    </link>
     <!-- JOINTS -->
     <joint name="${agent_namespace}_base_obstacle_joint" type="fixed">
-        <origin xyz="${(-base_w*0.5)} 0 ${(base_h*0.5)}" rpy="${pi/2} 0 0"/>
+        <origin xyz="${(-base_w*0.5)+(obstacle_w)} 0 ${(base_h*0.5)}" rpy="${pi/2} 0 0"/>
         <parent link="${agent_namespace}_base_link"/>
         <child link="${agent_namespace}_obstacle_link"/>
+    </joint>
+    <joint name="${agent_namespace}_base_white_box_1_joint" type="fixed">
+        <origin xyz="${(-base_w*0.5)} ${(obstacle_l*0.65)} ${(base_h*0.5)+(obstacle_w*0.5)}" rpy="0.0 0.0 0.0"/>
+        <parent link="${agent_namespace}_base_link"/>
+        <child link="${agent_namespace}_white_box_1_link"/>
+    </joint>
+    <joint name="${agent_namespace}_base_white_box_2_joint" type="fixed">
+        <origin xyz="${(-base_w*0.5)} ${(-obstacle_l*0.65)} ${(base_h*0.5)+(obstacle_w*0.5)}" rpy="0.0 0.0 0.0"/>
+        <parent link="${agent_namespace}_base_link"/>
+        <child link="${agent_namespace}_white_box_2_link"/>
     </joint>
     <!-- GAZEBO -->
@@ -33,3 +80,9 @@
         <material>Gazebo/Red</material>
     </gazebo>
+    <gazebo reference="${agent_namespace}_white_box_1_link">
+        <material>Gazebo/White</material>
+    </gazebo>
+    <gazebo reference="${agent_namespace}_white_box_2_link">
+        <material>Gazebo/White</material>
+    </gazebo>
 </robot>

Commit message: isolating detection_object

File: ros_ws/src/pipe_swarm/urdf/detection_object.xacro (robot description, xacro)
@@ -76,13 +76,3 @@
         <child link="${agent_namespace}_white_box_2_link"/>
     </joint>
-    <!-- GAZEBO -->
-    <gazebo reference="${agent_namespace}_obstacle_link">
-        <material>Gazebo/Red</material>
-    </gazebo>
-    <gazebo reference="${agent_namespace}_white_box_1_link">
-        <material>Gazebo/White</material>
-    </gazebo>
-    <gazebo reference="${agent_namespace}_white_box_2_link">
-        <material>Gazebo/White</material>
-    </gazebo>
 </robot>

Commit message: covering the red box better

File: ros_ws/src/pipe_swarm/urdf/detection_object.xacro (robot description, xacro)
@@ -29,5 +29,5 @@
             <origin xyz="0.0 0.0 0.0" rpy="0.0 0.0 0.0"/>
             <geometry>
-                <box size="${obstacle_w} ${obstacle_l} ${obstacle_h}"/>
+                <box size="${obstacle_w*2} ${obstacle_l} ${obstacle_h}"/>
             </geometry>
             <material name="white">
@@ -37,5 +37,5 @@
         <collision>
             <geometry>
-                <box size="${obstacle_w} ${obstacle_l} ${obstacle_h}"/>
+                <box size="${obstacle_w*2} ${obstacle_l} ${obstacle_h}"/>
             </geometry>
         </collision>
@@ -47,5 +47,5 @@
             <origin xyz="0.0 0.0 0.0" rpy="0.0 0.0 0.0"/>
             <geometry>
-                <box size="${obstacle_w} ${obstacle_l} ${obstacle_h}"/>
+                <box size="${obstacle_w*2} ${obstacle_l} ${obstacle_h}"/>
             </geometry>
             <material name="white">
@@ -55,5 +55,5 @@
         <collision>
             <geometry>
-                <box size="${obstacle_w} ${obstacle_l} ${obstacle_h}"/>
+                <box size="${obstacle_w*2} ${obstacle_l} ${obstacle_h}"/>
             </geometry>
         </collision>
@@ -67,10 +67,10 @@
     </joint>
     <joint name="${agent_namespace}_base_white_box_1_joint" type="fixed">
-        <origin xyz="${(-base_w*0.5)} ${(obstacle_l*0.55)} ${(base_h*0.5)+(obstacle_w*0.5)}" rpy="0.0 0.0 0.0"/>
+        <origin xyz="${(-base_w*0.5)+(obstacle_w)} ${(obstacle_l*0.54)} ${(base_h*0.5)+(obstacle_w*0.5)}" rpy="0.0 0.0 0.0"/>
         <parent link="${agent_namespace}_base_link"/>
         <child link="${agent_namespace}_white_box_1_link"/>
     </joint>
     <joint name="${agent_namespace}_base_white_box_2_joint" type="fixed">
-        <origin xyz="${(-base_w*0.5)} ${(-obstacle_l*0.55)} ${(base_h*0.5)+(obstacle_w*0.5)}" rpy="0.0 0.0 0.0"/>
+        <origin xyz="${(-base_w*0.5)+(obstacle_w)} ${(-obstacle_l*0.54)} ${(base_h*0.5)+(obstacle_w*0.5)}" rpy="0.0 0.0 0.0"/>
         <parent link="${agent_namespace}_base_link"/>
         <child link="${agent_namespace}_white_box_2_link"/>

Commit message: Calibrated detection object and camera

File: ros_ws/src/pipe_swarm/urdf/detection_object.xacro (robot description, xacro)
@@ -67,10 +67,10 @@
     </joint>
     <joint name="${agent_namespace}_base_white_box_1_joint" type="fixed">
-        <origin xyz="${(-base_w*0.5)+(obstacle_w)} ${(obstacle_l*0.54)} ${(base_h*0.5)+(obstacle_w*0.5)}" rpy="0.0 0.0 0.0"/>
+        <origin xyz="${(-base_w*0.5)+(obstacle_w)} ${(obstacle_l*0.6)} ${(base_h*0.5)+(obstacle_w*0.5)}" rpy="0.0 0.0 0.0"/>
         <parent link="${agent_namespace}_base_link"/>
         <child link="${agent_namespace}_white_box_1_link"/>
     </joint>
     <joint name="${agent_namespace}_base_white_box_2_joint" type="fixed">
-        <origin xyz="${(-base_w*0.5)+(obstacle_w)} ${(-obstacle_l*0.54)} ${(base_h*0.5)+(obstacle_w*0.5)}" rpy="0.0 0.0 0.0"/>
+        <origin xyz="${(-base_w*0.5)+(obstacle_w)} ${(-obstacle_l*0.6)} ${(base_h*0.5)+(obstacle_w*0.5)}" rpy="0.0 0.0 0.0"/>
         <parent link="${agent_namespace}_base_link"/>
         <child link="${agent_namespace}_white_box_2_link"/>

File: ros_ws/src/pipe_swarm/urdf/gazebo/camera.xacro (robot description, xacro)
@@ -17,6 +17,6 @@
                 </image>
                 <clip>
-                    <near>0.05</near>
-                    <far>0.3</far>
+                    <near>0.01</near>
+                    <far>0.6</far>
                 </clip>
             </camera>
