Commit message: finalizing female linkage shape and motion

File: ros_ws/src/pipe_swarm/urdf/linkage.xacro (robot description, xacro)
@@ -5,8 +5,11 @@
     <xacro:property name="male_l" value="0.01" />  <!-- length /m -->
     <xacro:property name="male_h" value="0.01" />  <!-- height /m -->
-    <xacro:property name="female_thickness_out" value="0.028" />  <!-- outer thickness /m -->
-    <xacro:property name="female_diameter" value="0.04" />  <!-- outer thickness /m -->
-    <xacro:property name="female_wall_thickness" value="0.05" />  <!-- outer thickness /m -->
-    <xacro:macro name="female_shape_1">
+    <xacro:property name="female_thickness_out" value="0.028" />  <!-- /m -->
+    <xacro:property name="female_diameter" value="0.04" />  <!-- /m -->
+    <xacro:property name="female_stopper_thickness" value="0.05" />  <!-- /m -->
+    <xacro:property name="female_hole_depth" value="0.03" />  <!-- /m -->
+    <xacro:property name="female_wall_thickness" value="0.01" />  <!-- /m -->
+    <xacro:property name="female_hole_thickness" value="0.01" />  <!-- /m -->
+    <xacro:macro name="female_rotation_shape">
             <origin xyz="0 0 0" rpy="${pi/2} 0 0"/>
             <geometry>
@@ -14,16 +17,19 @@
             </geometry>
     </xacro:macro>
-    <xacro:macro name="female_shape_2">
-            <origin xyz="${-female_wall_thickness/2} 0 0" rpy="0 0 0"/>
+    <xacro:macro name="female_stopper_shape">
+            <origin xyz="${-female_stopper_thickness/2} 0 0" rpy="0 0 0"/>
             <geometry>
-                <box size="${female_wall_thickness} ${female_thickness_out} ${female_diameter}"/>
+                <box size="${female_stopper_thickness} ${female_thickness_out} ${female_diameter}"/>
             </geometry>
     </xacro:macro>
-    <!-- <xacro:macro name="female_shape_3">
-            <origin xyz="${-(female_diameter/2)} 0 0" rpy="0 0 0"/>
+    <xacro:macro name="female_wall_shape" params="y_offset z_offset">
+            <origin xyz="${-(female_stopper_thickness + female_hole_depth/2)}
+                        ${y_offset * (female_wall_thickness/2 + female_hole_thickness/2)}
+                        ${z_offset * (female_wall_thickness/2 + female_hole_thickness/2)}"
+                        rpy="0 0 0"/>
             <geometry>
-                <box size="0.05 ${female_thickness_out} ${female_diameter}"/>
+                <box size="${female_hole_depth} ${female_wall_thickness} ${female_wall_thickness}"/>
             </geometry>
-    </xacro:macro> -->
+    </xacro:macro>
     <!-- LINKS -->
     <link name="male_link">
@@ -42,9 +48,9 @@
             </geometry>
         </collision>
-        <xacro:box_inertial m="${male_m}" w="${male_w}" l="${male_l}" h="${male_h}" xyz="0 0 0 " rpy="0 0 0"/>
+        <!-- <xacro:box_inertial m="${male_m}" w="${male_w}" l="${male_l}" h="${male_h}" xyz="0 0 0 " rpy="0 0 0"/> -->
     </link>
     <link name="female_link">
         <visual>
-            <xacro:female_shape_1 />
+            <xacro:female_rotation_shape />
             <material name="base">
                 <color rgba="1.0 1.0 1.0 1.0"/>
@@ -52,5 +58,29 @@
         </visual>
         <visual>
-            <xacro:female_shape_2 />
+            <xacro:female_stopper_shape />
+            <material name="base">
+                <color rgba="1.0 1.0 1.0 1.0"/>
+            </material>
+        </visual>
+        <visual>
+            <xacro:female_wall_shape y_offset="0" z_offset="1"/>
+            <material name="base">
+                <color rgba="1.0 1.0 1.0 1.0"/>
+            </material>
+        </visual>
+        <visual>
+            <xacro:female_wall_shape y_offset="1" z_offset="0"/>
+            <material name="base">
+                <color rgba="1.0 1.0 1.0 1.0"/>
+            </material>
+        </visual>
+        <visual>
+            <xacro:female_wall_shape y_offset="-1" z_offset="0"/>
+            <material name="base">
+                <color rgba="1.0 1.0 1.0 1.0"/>
+            </material>
+        </visual>
+        <visual>
+            <xacro:female_wall_shape y_offset="0" z_offset="-1"/>
             <material name="base">
                 <color rgba="1.0 1.0 1.0 1.0"/>
@@ -58,5 +88,20 @@
         </visual>
         <collision>
-            <xacro:female_shape_1 />
+            <xacro:female_rotation_shape />
+        </collision>
+        <collision>
+            <xacro:female_stopper_shape />
+        </collision>
+        <collision>
+            <xacro:female_wall_shape y_offset="0" z_offset="1"/>
+        </collision>
+        <collision>
+            <xacro:female_wall_shape y_offset="0" z_offset="-1"/>
+        </collision>
+        <collision>
+            <xacro:female_wall_shape y_offset="1" z_offset="0"/>
+        </collision>
+        <collision>
+            <xacro:female_wall_shape y_offset="-1" z_offset="0"/>
         </collision>
         <!-- TODO Fix inertia -->
@@ -69,8 +114,10 @@
         <child link="male_link"/>
     </joint>
-    <joint name="base_female_joint" type="fixed">
+    <joint name="base_female_joint" type="revolute">
         <origin xyz="${-(base_w*0.5) + 0.023} 0 0" rpy="0 0 0"/>
         <parent link="base_link"/>
         <child link="female_link"/>
+        <axis xyz="0 1 0"/>
+        <limit lower="${-pi/2}" upper="${pi/2}" effort="1.0" velocity="1.0"/>
     </joint>
     <!-- GAZEBO -->

Commit message: fixing robot state publisher

File: ros_ws/src/pipe_swarm/urdf/linkage.xacro (robot description, xacro)
@@ -48,5 +48,5 @@
             </geometry>
         </collision>
-        <!-- <xacro:box_inertial m="${male_m}" w="${male_w}" l="${male_l}" h="${male_h}" xyz="0 0 0 " rpy="0 0 0"/> -->
+        <xacro:box_inertial m="${male_m}" w="${male_w}" l="${male_l}" h="${male_h}" xyz="0 0 0 " rpy="0 0 0"/>
     </link>
     <link name="female_link">
@@ -106,5 +106,5 @@
         </collision>
         <!-- TODO Fix inertia -->
-        <!-- <xacro:box_inertial m="${male_m}" w="${male_w}" l="${male_l}" h="${male_h}" xyz="0 0 0 " rpy="0 0 0"/> -->
+        <xacro:box_inertial m="${male_m}" w="${male_w}" l="${male_l}" h="${male_h}" xyz="0 0 0 " rpy="0 0 0"/>
     </link>
     <!-- JOINTS -->
@@ -116,4 +116,5 @@
     <joint name="base_female_joint" type="revolute">
         <origin xyz="${-(base_w*0.5) + 0.023} 0 0" rpy="0 0 0"/>
+        <!-- <origin xyz="${-(base_w*0.5) - 0.023} 0 0" rpy="0 0 0"/> -->
         <parent link="base_link"/>
         <child link="female_link"/>
@@ -122,3 +123,12 @@
     </joint>
     <!-- GAZEBO -->
+    <gazebo reference="female_link">
+        <material>Gazebo/Red</material>
+    </gazebo>
+    <gazebo>
+        <plugin name="gazebo_ros_joint_state_publisher" filename="libgazebo_ros_joint_state_publisher.so">
+            <update_rate>50</update_rate>
+            <joint_name>base_female_joint</joint_name>
+        </plugin>
+    </gazebo>
 </robot>

Commit message: adding ros2 control to female linkage

File: ros_ws/src/pipe_swarm/urdf/linkage.xacro (robot description, xacro)
@@ -115,6 +115,6 @@
     </joint>
     <joint name="base_female_joint" type="revolute">
-        <origin xyz="${-(base_w*0.5) + 0.023} 0 0" rpy="0 0 0"/>
-        <!-- <origin xyz="${-(base_w*0.5) - 0.023} 0 0" rpy="0 0 0"/> -->
+        <!-- <origin xyz="${-(base_w*0.5) + 0.023} 0 0" rpy="0 0 0"/> -->
+        <origin xyz="${-(base_w*0.5) + female_diameter/2} 0 0" rpy="0 0 0"/>
         <parent link="base_link"/>
         <child link="female_link"/>
@@ -129,5 +129,5 @@
         <material>Gazebo/White</material>
     </gazebo>
-    <gazebo>
+    <!-- <gazebo>
         <plugin name="joint_state_publisher" filename="libgazebo_ros_joint_state_publisher.so">
             <ros>
@@ -137,9 +137,30 @@
             <joint_name>base_female_joint</joint_name>
         </plugin>
-    </gazebo>
+    </gazebo> -->
     <gazebo>
-        <plugin name="${agent_namespace}_control" filename="libgazebo_ros_control.so">
-            <robotNamespace>/</robotNamespace>
+        <plugin name="urdf_control" filename="libgazebo_ros2_control.so">
+            <!-- <ros>
+                <namespace>${agent_namespace}</namespace>
+            </ros> -->
+            <update_rate>50</update_rate>
+            <parameters>$(find pipe_swarm)/config/robot_controllers_sim.yaml</parameters>
         </plugin>
     </gazebo>
+    <!-- ros2_control Plugin -->
+    <ros2_control name="GazeboSystem" type="system">
+        <hardware>
+            <plugin>gazebo_ros2_control/GazeboSystem</plugin>
+        </hardware>
+        <joint name="base_female_joint">
+            <command_interface name="position">
+                <param name="min">-1.57</param>
+                <param name="max">1.57</param>
+            </command_interface>
+            <state_interface name="position">
+                <param name="initial_value">1.0</param>
+            </state_interface>
+            <state_interface name="velocity"/>
+            <state_interface name="effort"/>
+        </joint>
+    </ros2_control>
 </robot>

File: ros_ws/src/pipe_swarm/urdf/mobile_base.xacro (robot description, xacro)
@@ -31,4 +31,7 @@
     </joint>
     <!-- GAZEBO -->
+    <gazebo reference="footprint_link">
+        <material>Gazebo/Blue</material>
+    </gazebo>
     <gazebo reference="base_link">
         <material>Gazebo/Blue</material>

File: ros_ws/src/pipe_swarm/urdf/pipe_robot.urdf.xacro (robot description, xacro)
@@ -5,5 +5,5 @@
     <xacro:include filename="mobile_base.xacro"/>
     <xacro:include filename="camera.xacro"/>
-    <xacro:include filename="wheels.xacro"/>
+    <!-- <xacro:include filename="wheels.xacro"/> -->
     <xacro:include filename="linkage.xacro"/>
 </robot>

Commit message: fixing renaming of joint while adhering to ros2 control

File: ros_ws/src/pipe_swarm/urdf/linkage.xacro (robot description, xacro)
@@ -114,5 +114,5 @@
         <child link="${agent_namespace}_male_link"/>
     </joint>
-    <joint name="${agent_namespace}_base_female_joint" type="revolute">
+    <joint name="base_female_joint" type="revolute">
         <origin xyz="${-(base_w*0.5) + female_diameter/2} 0 0" rpy="0 0 0"/>
         <parent link="${agent_namespace}_base_link"/>
@@ -131,5 +131,5 @@
         <plugin name="${agent_namespace}_control" filename="libgazebo_ros2_control.so">
             <robot_param_node>/${agent_namespace}/robot_state_publisher</robot_param_node>
-            <parameters>$(find pipe_swarm)/config/${agent_namespace}_controllers_sim.yaml</parameters>
+            <parameters>$(find pipe_swarm)/config/robot_controllers_sim.yaml</parameters>
             <ros>
                 <namespace>${agent_namespace}</namespace>
@@ -142,5 +142,5 @@
             <plugin>gazebo_ros2_control/GazeboSystem</plugin>
         </hardware>
-        <joint name="${agent_namespace}_base_female_joint">
+        <joint name="base_female_joint">
             <command_interface name="position">
                 <param name="min">-pi/2</param>

Commit message: adding world

File: ros_ws/src/pipe_swarm/urdf/linkage.xacro (robot description, xacro)
@@ -47,4 +47,5 @@
         </visual>
         <collision>
+            <origin xyz="0.0 0.0 0.0" rpy="0.0 0.0 0.0"/>
             <geometry>
                 <box size="${male_w} ${male_l} ${male_h}"/>
@@ -111,8 +112,10 @@
     </link>
     <!-- JOINTS -->
-    <joint name="${agent_namespace}_base_male_joint" type="fixed">
+    <joint name="${agent_namespace}_base_male_joint" type="revolute">
         <origin xyz="${(base_w*0.5) + (male_w*0.5)} 0 0" rpy="0 0 0"/>
         <parent link="${agent_namespace}_base_link"/>
         <child link="${agent_namespace}_male_link"/>
+        <axis xyz="0 1 0"/>
+        <limit lower="${0}" upper="${0}" effort="1.0" velocity="1.0"/>
     </joint>
     <joint name="base_female_joint" type="revolute">

Commit message: fixing male linkage bug

File: ros_ws/src/pipe_swarm/urdf/linkage.xacro (robot description, xacro)
@@ -112,10 +112,8 @@
     </link>
     <!-- JOINTS -->
-    <joint name="${agent_namespace}_base_male_joint" type="revolute">
+    <joint name="${agent_namespace}_base_male_joint" type="fixed">
         <origin xyz="${(base_w*0.5) + (male_w*0.5)} 0 0" rpy="0 0 0"/>
         <parent link="${agent_namespace}_base_link"/>
         <child link="${agent_namespace}_male_link"/>
-        <axis xyz="0 1 0"/>
-        <limit lower="${0}" upper="${0}" effort="1.0" velocity="1.0"/>
     </joint>
     <joint name="base_female_joint" type="revolute">

Commit message: Reduce size of male linkage to allow easier alignment

File: ros_ws/src/pipe_swarm/urdf/linkage.xacro (robot description, xacro)
@@ -3,6 +3,6 @@
     <xacro:property name="male_m" value="0.1" />  <!-- mass /kg -->
     <xacro:property name="male_w" value="0.04" />  <!-- width /m -->
-    <xacro:property name="male_h" value="0.01" />  <!-- height /m -->
-    <xacro:property name="male_l" value="0.01" />  <!-- length /m -->
+    <xacro:property name="male_h" value="0.005" />  <!-- height /m -->
+    <xacro:property name="male_l" value="0.005" />  <!-- length /m -->
     <xacro:property name="female_diameter" value="0.04" />  <!-- /m -->
     <xacro:property name="female_stopper_width" value="0.05" />  <!-- /m -->

Commit message: All other not affect movement

File: ros_ws/src/pipe_swarm/urdf/linkage.xacro (robot description, xacro)
@@ -4,5 +4,5 @@
     <xacro:property name="male_w" value="0.04" />  <!-- width /m -->
     <xacro:property name="male_h" value="0.005" />  <!-- height /m -->
-    <xacro:property name="male_l" value="0.005" />  <!-- length /m -->
+    <xacro:property name="male_l" value="0.0575" />  <!-- length /m -->
     <xacro:property name="female_diameter" value="0.04" />  <!-- /m -->
     <xacro:property name="female_stopper_width" value="0.05" />  <!-- /m -->
@@ -13,9 +13,9 @@
     <xacro:property name="female_w" value="${(female_diameter/2) + female_stopper_width + female_hole_depth}" />  <!-- width /m -->
     <xacro:property name="female_h" value="${female_diameter}" />  <!-- height /m -->
-    <xacro:property name="female_l" value="0.028" />  <!-- /m -->
+    <xacro:property name="female_l" value="0.028" />  /m
     <xacro:macro name="female_rotation_shape">
             <origin xyz="0 0 0" rpy="${pi/2} 0 0"/>
             <geometry>
-                <cylinder radius="${female_diameter/2}" length="${female_l}"/>
+                <mesh filename="model://hollow_pipe/meshes/lock.stl"/>
             </geometry>
     </xacro:macro>
@@ -38,7 +38,7 @@
     <link name="${agent_namespace}_male_link">
         <visual>
-            <origin xyz="0.0 0.0 0.0" rpy="0.0 0.0 0.0"/>
+            <origin xyz="0.0 0.0 0.0" rpy="0.0 ${pi/2} ${-pi/2}"/>
             <geometry>
-                <box size="${male_w} ${male_l} ${male_h}"/>
+                <mesh filename="model://hollow_pipe/meshes/key.stl" scale="0.001 0.001 0.001"/>
             </geometry>
             <material name="base">
@@ -47,7 +47,25 @@
         </visual>
         <collision>
-            <origin xyz="0.0 0.0 0.0" rpy="0.0 0.0 0.0"/>
+            <origin xyz="0.0 0.0 0.0" rpy="0.0 ${pi/2} ${-pi/2}"/>
             <geometry>
-                <box size="${male_w} ${male_l} ${male_h}"/>
+                <mesh filename="model://hollow_pipe/meshes/key.stl" scale="0.001 0.001 0.001"/>
+            </geometry>
+        </collision>
+        <xacro:box_inertial m="${male_m}" w="${male_w}" l="${male_l}" h="${male_h}" xyz="0 0 0 " rpy="0 0 0"/>
+    </link>
+    <link name="${agent_namespace}_cover_link">
+        <visual>
+            <origin xyz="0.0 0.0 0.0" rpy="${pi/2} 0.0 ${pi/2}"/>
+            <geometry>
+                <mesh filename="model://hollow_pipe/meshes/cover.stl" scale="0.001 0.001 0.001"/>
+            </geometry>
+            <material name="base">
+                <color rgba="1.0 1.0 1.0 1.0"/>
+            </material>
+        </visual>
+        <collision>
+            <origin xyz="0.0 0.0 0.0" rpy="${pi/2} 0.0 ${pi/2}"/>
+            <geometry>
+                <mesh filename="model://hollow_pipe/meshes/cover.stl" scale="0.001 0.001 0.001"/>
             </geometry>
         </collision>
@@ -55,36 +73,9 @@
     </link>
     <link name="${agent_namespace}_female_link">
-        <visual>
-            <xacro:female_rotation_shape />
-            <material name="base">
-                <color rgba="1.0 1.0 1.0 1.0"/>
-            </material>
-        </visual>
-        <visual>
-            <xacro:female_stopper_shape />
-            <material name="base">
-                <color rgba="1.0 1.0 1.0 1.0"/>
-            </material>
-        </visual>
-        <visual>
-            <xacro:female_wall_shape y_offset="0" z_offset="1"/>
-            <material name="base">
-                <color rgba="1.0 1.0 1.0 1.0"/>
-            </material>
-        </visual>
-        <visual>
-            <xacro:female_wall_shape y_offset="1" z_offset="0"/>
-            <material name="base">
-                <color rgba="1.0 1.0 1.0 1.0"/>
-            </material>
-        </visual>
-        <visual>
-            <xacro:female_wall_shape y_offset="-1" z_offset="0"/>
-            <material name="base">
-                <color rgba="1.0 1.0 1.0 1.0"/>
-            </material>
-        </visual>
-        <visual>
-            <xacro:female_wall_shape y_offset="0" z_offset="-1"/>
+       <visual>
+            <origin xyz="0 0 0" rpy="0.0 ${pi/2} ${pi/2}"/>
+            <geometry>
+                <mesh filename="model://hollow_pipe/meshes/lock.stl" scale="0.001 0.001 0.001"/>
+            </geometry>
             <material name="base">
                 <color rgba="1.0 1.0 1.0 1.0"/>
@@ -92,35 +83,50 @@
         </visual>
         <collision>
-            <xacro:female_rotation_shape />
+            <origin xyz="0 0 0" rpy="0.0 ${pi/2} ${pi/2}"/>
+            <geometry>
+                <mesh filename="model://hollow_pipe/meshes/lock.stl" scale="0.001 0.001 0.001"/>
+            </geometry>
         </collision>
+    </link>
+    <link name="${agent_namespace}_pivot_link">
+       <visual>
+            <origin xyz="0 0 0" rpy="${pi/2} 0.0 ${-pi/2}"/>
+            <geometry>
+                <mesh filename="model://hollow_pipe/meshes/pivot.stl" scale="0.001 0.001 0.001"/>
+            </geometry>
+            <material name="base">
+                <color rgba="1.0 1.0 1.0 1.0"/>
+            </material>
+        </visual>
         <collision>
-            <xacro:female_stopper_shape />
+            <origin xyz="0 0 0" rpy="${pi/2} 0.0 ${-pi/2}"/>
+            <geometry>
+                <mesh filename="model://hollow_pipe/meshes/pivot.stl" scale="0.001 0.001 0.001"/>
+            </geometry>
         </collision>
-        <collision>
-            <xacro:female_wall_shape y_offset="0" z_offset="1"/>
-        </collision>
-        <collision>
-            <xacro:female_wall_shape y_offset="0" z_offset="-1"/>
-        </collision>
-        <collision>
-            <xacro:female_wall_shape y_offset="1" z_offset="0"/>
-        </collision>
-        <collision>
-            <xacro:female_wall_shape y_offset="-1" z_offset="0"/>
-        </collision>
-        <xacro:box_inertial m="${female_m}" w="${female_w}" l="${female_l}" h="${female_h}" xyz="${female_diameter/2 - female_w/2} 0 0 " rpy="0 0 0"/>
+        <xacro:box_inertial m="${female_m}" w="0.05" l="0.05" h="0.05" xyz="0 0 0" rpy="0 0 0"/>
     </link>
     <!-- JOINTS -->
+    <joint name="${agent_namespace}_base_cover_joint" type="fixed">
+        <origin xyz="${(base_w*0.5)+0.007} 0.0 0.0" rpy="0 0 0"/>
+        <parent link="${agent_namespace}_base_link"/>
+        <child link="${agent_namespace}_cover_link"/>
+    </joint>
     <joint name="${agent_namespace}_base_male_joint" type="fixed">
-        <origin xyz="${(base_w*0.5) + (male_w*0.5)} 0 0" rpy="0 0 0"/>
+        <origin xyz="${(base_w*0.5)+0.007} 0.0 0.0" rpy="0 0 0"/>
         <parent link="${agent_namespace}_base_link"/>
         <child link="${agent_namespace}_male_link"/>
     </joint>
     <joint name="base_female_joint" type="revolute">
-        <origin xyz="${-(base_w*0.5) + female_diameter/2} 0 0" rpy="0 0 0"/>
+        <origin xyz="${-(base_w*0.5)+0.014} 0.0275 0.0" rpy="0 0 0"/>
         <parent link="${agent_namespace}_base_link"/>
-        <child link="${agent_namespace}_female_link"/>
+        <child link="${agent_namespace}_pivot_link"/>
         <axis xyz="0 1 0"/>
         <limit lower="${-pi/2}" upper="${pi/2}" effort="1.0" velocity="1.0"/>
+    </joint>
+    <joint name="${agent_namespace}_base_neutral_joint" type="fixed">
+        <origin xyz="-0.0665 -0.0275 0.0" rpy="0 0 0"/>
+        <parent link="${agent_namespace}_pivot_link"/>
+        <child link="${agent_namespace}_female_link"/>
     </joint>
     <!-- GAZEBO -->
@@ -129,4 +135,10 @@
     </gazebo>
     <gazebo reference="${agent_namespace}_male_link">
+        <material>Gazebo/White</material>
+    </gazebo>
+    <gazebo reference="${agent_namespace}_pivot_link">
+        <material>Gazebo/White</material>
+    </gazebo>
+        <gazebo reference="${agent_namespace}_neutral_link">
         <material>Gazebo/White</material>
     </gazebo>
