Commit message: New package path so rvis and gazebo both laod stl

File: ros_ws/src/pipe_swarm/urdf/linkage.xacro (robot description, xacro)
@@ -40,5 +40,5 @@
             <origin xyz="0.0 0.0 0.0" rpy="0.0 ${pi/2} ${-pi/2}"/>
             <geometry>
-                <mesh filename="model://hollow_pipe/meshes/key.stl" scale="0.001 0.001 0.001"/>
+                <mesh filename="package://pipe_swarm/models/hollow_pipe/meshes/key.stl" scale="0.001 0.001 0.001"/>
             </geometry>
             <material name="base">
@@ -49,5 +49,5 @@
             <origin xyz="0.0 0.0 0.0" rpy="0.0 ${pi/2} ${-pi/2}"/>
             <geometry>
-                <mesh filename="model://hollow_pipe/meshes/key.stl" scale="0.001 0.001 0.001"/>
+                <mesh filename="package://pipe_swarm/models/hollow_pipe/meshes/key.stl" scale="0.001 0.001 0.001"/>
             </geometry>
         </collision>
@@ -58,5 +58,5 @@
             <origin xyz="0.0 0.0 0.0" rpy="${pi/2} 0.0 ${pi/2}"/>
             <geometry>
-                <mesh filename="model://hollow_pipe/meshes/cover.stl" scale="0.001 0.001 0.001"/>
+                <mesh filename="package://pipe_swarm/models/hollow_pipe/meshes/cover.stl" scale="0.001 0.001 0.001"/>
             </geometry>
             <material name="base">
@@ -67,5 +67,5 @@
             <origin xyz="0.0 0.0 0.0" rpy="${pi/2} 0.0 ${pi/2}"/>
             <geometry>
-                <mesh filename="model://hollow_pipe/meshes/cover.stl" scale="0.001 0.001 0.001"/>
+                <mesh filename="package://pipe_swarm/models/hollow_pipe/meshes/cover.stl" scale="0.001 0.001 0.001"/>
             </geometry>
         </collision>
@@ -76,5 +76,5 @@
             <origin xyz="0 0 0" rpy="0.0 ${pi/2} ${pi/2}"/>
             <geometry>
-                <mesh filename="model://hollow_pipe/meshes/lock.stl" scale="0.001 0.001 0.001"/>
+                <mesh filename="package://pipe_swarm/models/hollow_pipe/meshes/lock.stl" scale="0.001 0.001 0.001"/>
             </geometry>
             <material name="base">
@@ -85,5 +85,5 @@
             <origin xyz="0 0 0" rpy="0.0 ${pi/2} ${pi/2}"/>
             <geometry>
-                <mesh filename="model://hollow_pipe/meshes/lock.stl" scale="0.001 0.001 0.001"/>
+                <mesh filename="package://pipe_swarm/models/hollow_pipe/meshes/lock.stl" scale="0.001 0.001 0.001"/>
             </geometry>
         </collision>
@@ -93,5 +93,5 @@
             <origin xyz="0 0 0" rpy="${pi/2} 0.0 ${-pi/2}"/>
             <geometry>
-                <mesh filename="model://hollow_pipe/meshes/pivot.stl" scale="0.001 0.001 0.001"/>
+                <mesh filename="package://pipe_swarm/models/hollow_pipe/meshes/pivot.stl" scale="0.001 0.001 0.001"/>
             </geometry>
             <material name="base">
@@ -102,5 +102,5 @@
             <origin xyz="0 0 0" rpy="${pi/2} 0.0 ${-pi/2}"/>
             <geometry>
-                <mesh filename="model://hollow_pipe/meshes/pivot.stl" scale="0.001 0.001 0.001"/>
+                <mesh filename="package://pipe_swarm/models/hollow_pipe/meshes/pivot.stl" scale="0.001 0.001 0.001"/>
             </geometry>
         </collision>

File: ros_ws/src/pipe_swarm/urdf/wheels.xacro (robot description, xacro)
@@ -10,5 +10,5 @@
                 <origin xyz="0.0 0.0 0.0" rpy="0 0.0 0.0"/>
                 <geometry>
-                    <mesh filename="model://hollow_pipe/meshes/wheel_right.stl" scale="0.001 0.001 0.001"/>
+                    <mesh filename="package://pipe_swarm/models/hollow_pipe/meshes/wheel_right.stl" scale="0.001 0.001 0.001"/>
                     <!-- <cylinder radius="${wheel_r}" length="${wheel_l}"/> -->
                 </geometry>
@@ -20,5 +20,5 @@
                 <origin xyz="0.0 0.0 0.0" rpy="0 0.0 0.0"/>
                 <geometry>
-                    <mesh filename="model://hollow_pipe/meshes/wheel_right.stl" scale="0.001 0.001 0.001"/>
+                    <mesh filename="package://pipe_swarm/models/hollow_pipe/meshes/wheel_right.stl" scale="0.001 0.001 0.001"/>
                     <!-- <cylinder radius="${wheel_r}" length="${wheel_l}"/> -->
                 </geometry>
@@ -30,5 +30,5 @@
                 <origin xyz="0.0 0.0 0.0" rpy="0 0.0 0.0"/>
                 <geometry>
-                    <mesh filename="model://hollow_pipe/meshes/wheel.stl" scale="0.001 0.001 0.001"/>
+                    <mesh filename="package://pipe_swarm/models/hollow_pipe/meshes/wheel.stl" scale="0.001 0.001 0.001"/>
                     <!-- <cylinder radius="${wheel_r}" length="${wheel_l}"/> -->
                 </geometry>
@@ -40,5 +40,5 @@
                 <origin xyz="0.0 0.0 0.0" rpy="0 0.0 0.0"/>
                 <geometry>
-                    <mesh filename="model://hollow_pipe/meshes/wheel.stl" scale="0.001 0.001 0.001"/>
+                    <mesh filename="package://pipe_swarm/models/hollow_pipe/meshes/wheel.stl" scale="0.001 0.001 0.001"/>
                     <!-- <cylinder radius="${wheel_r}" length="${wheel_l}"/> -->
                 </geometry>

Commit message: fixing female comment

File: ros_ws/src/pipe_swarm/urdf/linkage.xacro (robot description, xacro)
@@ -13,5 +13,5 @@
     <xacro:property name="female_w" value="${(female_diameter/2) + female_stopper_width + female_hole_depth}" />  <!-- width /m -->
     <xacro:property name="female_h" value="${female_diameter}" />  <!-- height /m -->
-    <xacro:property name="female_l" value="0.028" />  /m
+    <xacro:property name="female_l" value="0.028" />   <!-- length /m -->
     <xacro:macro name="female_rotation_shape">
             <origin xyz="0 0 0" rpy="${pi/2} 0 0"/>

Commit message: making male joint revolute

File: ros_ws/src/pipe_swarm/urdf/linkage.xacro (robot description, xacro)
@@ -116,8 +116,10 @@
         <child link="${agent_namespace}_cover_link"/>
     </joint>
-    <joint name="${agent_namespace}_base_male_joint" type="fixed">
+    <joint name="${agent_namespace}_base_male_joint" type="revolute">
         <origin xyz="${(base_w*0.5)+male_o} 0.0 0.0" rpy="0 0 0"/>
         <parent link="${agent_namespace}_base_link"/>
         <child link="${agent_namespace}_male_link"/>
+        <axis xyz="1 0 0"/>
+        <limit lower="0.0" upper="${-pi/2}" effort="1.0" velocity="1.0"/>
     </joint>
     <joint name="base_female_joint" type="revolute">

Commit message: adding trajectory controller for male joint

File: ros_ws/src/pipe_swarm/urdf/linkage.xacro (robot description, xacro)
@@ -116,10 +116,10 @@
         <child link="${agent_namespace}_cover_link"/>
     </joint>
-    <joint name="${agent_namespace}_base_male_joint" type="revolute">
+    <joint name="base_male_joint" type="revolute">
         <origin xyz="${(base_w*0.5)+male_o} 0.0 0.0" rpy="0 0 0"/>
         <parent link="${agent_namespace}_base_link"/>
         <child link="${agent_namespace}_male_link"/>
         <axis xyz="1 0 0"/>
-        <limit lower="0.0" upper="${-pi/2}" effort="1.0" velocity="1.0"/>
+        <limit lower="${-pi/2}" upper="0" effort="1.0" velocity="1.0"/>
     </joint>
     <joint name="base_female_joint" type="revolute">

Commit message: Update to linkage file

File: ros_ws/src/pipe_swarm/urdf/linkage.xacro (robot description, xacro)
@@ -16,5 +16,5 @@
     <xacro:property name="female_l" value="0.028" />   <!-- length /m -->
     <xacro:property name="pivot_l" value="0.055" />  <!-- length /m -->
-    <xacro:property name="lock_w" value="0.0665" />  <!-- width /m -->
+    <xacro:property name="lock_w" value="0.02" />  <!-- width /m -->
     <xacro:macro name="female_rotation_shape">
             <origin xyz="0 0 0" rpy="${pi/2} 0 0"/>
@@ -61,5 +61,5 @@
             <origin xyz="0.0 0.0 0.0" rpy="${pi/2} 0.0 ${pi/2}"/>
             <geometry>
-                <mesh filename="package://pipe_swarm/models/hollow_pipe/meshes/cover.stl" scale="0.001 0.001 0.001"/>
+                <mesh filename="package://pipe_swarm/models/hollow_pipe/meshes/cover_v2.stl" scale="0.001 0.001 0.001"/>
             </geometry>
             <material name="base">
@@ -70,5 +70,5 @@
             <origin xyz="0.0 0.0 0.0" rpy="${pi/2} 0.0 ${pi/2}"/>
             <geometry>
-                <mesh filename="package://pipe_swarm/models/hollow_pipe/meshes/cover.stl" scale="0.001 0.001 0.001"/>
+                <mesh filename="package://pipe_swarm/models/hollow_pipe/meshes/cover_v2.stl" scale="0.001 0.001 0.001"/>
             </geometry>
         </collision>
@@ -79,5 +79,5 @@
             <origin xyz="${-lock_w/2} 0 0" rpy="0.0 ${pi/2} ${pi/2}"/>
             <geometry>
-                <mesh filename="package://pipe_swarm/models/hollow_pipe/meshes/lock.stl" scale="0.001 0.001 0.001"/>
+                <mesh filename="package://pipe_swarm/models/hollow_pipe/meshes/lock_v2.stl" scale="0.001 0.001 0.001"/>
             </geometry>
             <material name="base">
@@ -88,5 +88,5 @@
             <origin xyz="${-lock_w/2} 0 0" rpy="0.0 ${pi/2} ${pi/2}"/>
             <geometry>
-                <mesh filename="package://pipe_swarm/models/hollow_pipe/meshes/lock.stl" scale="0.001 0.001 0.001"/>
+                <mesh filename="package://pipe_swarm/models/hollow_pipe/meshes/lock_v2.stl" scale="0.001 0.001 0.001"/>
             </geometry>
         </collision>
@@ -112,5 +112,5 @@
     <!-- JOINTS -->
     <joint name="${agent_namespace}_base_cover_joint" type="fixed">
-        <origin xyz="${(base_w*0.5)+male_o} 0.0 0.0" rpy="0 0 0"/>
+        <origin xyz="${(base_w*0.5)-0.003} 0.0 0.0" rpy="0 0 0"/>
         <parent link="${agent_namespace}_base_link"/>
         <child link="${agent_namespace}_cover_link"/>
@@ -124,5 +124,5 @@
     </joint>
     <joint name="base_female_joint" type="revolute">
-        <origin xyz="${-(base_w*0.5)+0.014} 0 0" rpy="0 0 0"/>
+        <origin xyz="${-(base_w*0.5)} 0 0" rpy="0 0 0"/>
         <parent link="${agent_namespace}_base_link"/>
         <child link="${agent_namespace}_pivot_link"/>
@@ -136,5 +136,5 @@
     </joint> -->
     <joint name="${agent_namespace}_base_neutral_joint" type="fixed">
-        <origin xyz="${-lock_w/2} 0 0.0" rpy="0 0 0"/>
+        <origin xyz="${-0.01-pivot_l/2} 0 0.0" rpy="0 0 0"/>
         <parent link="${agent_namespace}_pivot_link"/>
         <child link="${agent_namespace}_female_link"/>

Commit message: No hard values

File: ros_ws/src/pipe_swarm/urdf/linkage.xacro (robot description, xacro)
@@ -17,4 +17,6 @@
     <xacro:property name="pivot_l" value="0.055" />  <!-- length /m -->
     <xacro:property name="lock_w" value="0.02" />  <!-- width /m -->
+    <xacro:property name="lock_o" value="0.01" />  <!-- offset /m -->
+    <xacro:property name="cover_o" value="0.003" />  <!-- offset /m -->
     <xacro:macro name="female_rotation_shape">
             <origin xyz="0 0 0" rpy="${pi/2} 0 0"/>
@@ -112,5 +114,5 @@
     <!-- JOINTS -->
     <joint name="${agent_namespace}_base_cover_joint" type="fixed">
-        <origin xyz="${(base_w*0.5)-0.003} 0.0 0.0" rpy="0 0 0"/>
+        <origin xyz="${(base_w*0.5)-cover_o} 0.0 0.0" rpy="0 0 0"/>
         <parent link="${agent_namespace}_base_link"/>
         <child link="${agent_namespace}_cover_link"/>
@@ -136,5 +138,5 @@
     </joint> -->
     <joint name="${agent_namespace}_base_neutral_joint" type="fixed">
-        <origin xyz="${-0.01-pivot_l/2} 0 0.0" rpy="0 0 0"/>
+        <origin xyz="${-lock_o-pivot_l/2} 0 0.0" rpy="0 0 0"/>
         <parent link="${agent_namespace}_pivot_link"/>
         <child link="${agent_namespace}_female_link"/>

Commit message: Linkage pivot point in correct position

File: ros_ws/src/pipe_swarm/urdf/linkage.xacro (robot description, xacro)
@@ -126,5 +126,5 @@
     </joint>
     <joint name="base_female_joint" type="revolute">
-        <origin xyz="${-(base_w*0.5)} 0 0" rpy="0 0 0"/>
+        <origin xyz="${-(base_w*0.5)+lock_o} 0 0" rpy="0 0 0"/>
         <parent link="${agent_namespace}_base_link"/>
         <child link="${agent_namespace}_pivot_link"/>

Commit message: Slightly edited part inserted into linkage

File: ros_ws/src/pipe_swarm/urdf/linkage.xacro (robot description, xacro)
@@ -81,5 +81,5 @@
             <origin xyz="${-lock_w/2} 0 0" rpy="0.0 ${pi/2} ${pi/2}"/>
             <geometry>
-                <mesh filename="package://pipe_swarm/models/hollow_pipe/meshes/lock_v2.stl" scale="0.001 0.001 0.001"/>
+                <mesh filename="package://pipe_swarm/models/hollow_pipe/meshes/lock_v2_for_sim.stl" scale="0.001 0.001 0.001"/>
             </geometry>
             <material name="base">
@@ -90,5 +90,5 @@
             <origin xyz="${-lock_w/2} 0 0" rpy="0.0 ${pi/2} ${pi/2}"/>
             <geometry>
-                <mesh filename="package://pipe_swarm/models/hollow_pipe/meshes/lock_v2.stl" scale="0.001 0.001 0.001"/>
+                <mesh filename="package://pipe_swarm/models/hollow_pipe/meshes/lock_v2_for_sim.stl" scale="0.001 0.001 0.001"/>
             </geometry>
         </collision>
@@ -123,5 +123,5 @@
         <child link="${agent_namespace}_male_link"/>
         <axis xyz="1 0 0"/>
-        <limit lower="${-pi/2}" upper="0" effort="1.0" velocity="1.0"/>
+        <limit lower="0.0" upper="${pi/2}" effort="1.0" velocity="1.0"/>
     </joint>
     <joint name="base_female_joint" type="revolute">
@@ -130,5 +130,5 @@
         <child link="${agent_namespace}_pivot_link"/>
         <axis xyz="0 1 0"/>
-        <limit lower="${-pi/4}" upper="${pi/4}" effort="1.0" velocity="1.0"/>
+        <limit lower="${-pi/4}" upper="${pi/4}" effort="0.5" velocity="0.5"/>
     </joint>
     <!-- <joint name="${agent_namespace}_footprint_base_joint" type="fixed">

Commit message: fixing male cover inertia

File: ros_ws/src/pipe_swarm/urdf/linkage.xacro (robot description, xacro)
@@ -1,4 +1,9 @@
 <?xml version="1.0"?>
 <robot name="linkage" xmlns:xacro="http://www.ros.org/wiki/xacro">
+    <xacro:property name="cover_m" value="0.1" />  <!-- mass /kg -->
+    <xacro:property name="cover_w" value="0.029" />  <!-- width /m -->
+    <xacro:property name="cover_h" value="0.024" />  <!-- height /m -->
+    <xacro:property name="cover_l" value="0.024" />  <!-- length /m -->
+    <xacro:property name="cover_out" value="0.0015" />  <!-- length /m -->
     <xacro:property name="male_m" value="0.1" />  <!-- mass /kg -->
     <xacro:property name="male_w" value="0.04" />  <!-- width /m -->
@@ -18,26 +23,5 @@
     <xacro:property name="lock_w" value="0.02" />  <!-- width /m -->
     <xacro:property name="lock_o" value="0.01" />  <!-- offset /m -->
-    <xacro:property name="cover_o" value="0.003" />  <!-- offset /m -->
-    <xacro:macro name="female_rotation_shape">
-            <origin xyz="0 0 0" rpy="${pi/2} 0 0"/>
-            <geometry>
-                <mesh filename="model://hollow_pipe/meshes/lock.stl"/>
-            </geometry>
-    </xacro:macro>
-    <xacro:macro name="female_stopper_shape">
-            <origin xyz="${-female_stopper_width/2} 0 0" rpy="0 0 0"/>
-            <geometry>
-                <box size="${female_stopper_width} ${female_l} ${female_diameter}"/>
-            </geometry>
-    </xacro:macro>
-    <xacro:macro name="female_wall_shape" params="y_offset z_offset">
-            <origin xyz="${-(female_stopper_width + female_hole_depth/2)}
-                        ${y_offset * (female_wall_thickness/2 + female_hole_thickness/2)}
-                        ${z_offset * (female_wall_thickness/2 + female_hole_thickness/2)}"
-                        rpy="0 0 0"/>
-            <geometry>
-                <box size="${female_hole_depth} ${female_wall_thickness} ${female_wall_thickness}"/>
-            </geometry>
-    </xacro:macro>
+    <xacro:property name="cover_o" value="0.0045" />  <!-- offset /m -->
     <!-- LINKS -->
     <link name="${agent_namespace}_male_link">
@@ -75,5 +59,5 @@
             </geometry>
         </collision>
-        <xacro:box_inertial m="${male_m}" w="${male_w}" l="${male_l}" h="${male_h}" xyz="0 0 0 " rpy="0 0 0"/>
+        <xacro:box_inertial m="${cover_m}" w="${cover_w}" l="${cover_l}" h="${cover_h}" xyz="${-cover_o} 0 0 " rpy="0 0 0"/>
     </link>
     <link name="${agent_namespace}_female_link">
@@ -114,5 +98,5 @@
     <!-- JOINTS -->
     <joint name="${agent_namespace}_base_cover_joint" type="fixed">
-        <origin xyz="${(base_w*0.5)-cover_o} 0.0 0.0" rpy="0 0 0"/>
+        <origin xyz="${(base_w*0.5) - cover_o + cover_out} 0.0 0.0" rpy="0 0 0"/>
         <parent link="${agent_namespace}_base_link"/>
         <child link="${agent_namespace}_cover_link"/>
@@ -132,9 +116,4 @@
         <limit lower="${-pi/4}" upper="${pi/4}" effort="1.0" velocity="1.0"/>
     </joint>
-    <!-- <joint name="${agent_namespace}_footprint_base_joint" type="fixed">
-        <origin xyz="${(base_w*0.5) - female_diameter/2} 0 0" rpy="0 0 0"/>
-        <parent link="${agent_namespace}_footprint_link"/>
-        <child link="${agent_namespace}_base_link"/>
-    </joint> -->
     <joint name="${agent_namespace}_base_neutral_joint" type="fixed">
         <origin xyz="${-lock_o-pivot_l/2} 0 0.0" rpy="0 0 0"/>

Commit message: fixing male link

File: ros_ws/src/pipe_swarm/urdf/linkage.xacro (robot description, xacro)
@@ -7,7 +7,7 @@
     <xacro:property name="cover_out" value="0.0015" />  <!-- length /m -->
     <xacro:property name="male_m" value="0.1" />  <!-- mass /kg -->
-    <xacro:property name="male_w" value="0.04" />  <!-- width /m -->
-    <xacro:property name="male_h" value="0.005" />  <!-- height /m -->
-    <xacro:property name="male_l" value="0.0575" />  <!-- length /m -->
+    <xacro:property name="male_w" value="0.014" />  <!-- width /m -->
+    <xacro:property name="male_l" value="0.0054" />  <!-- height /m -->
+    <xacro:property name="male_h" value="0.0128" />  <!-- length /m -->
     <xacro:property name="male_o" value="0.007" />  <!-- offset /m -->
     <xacro:property name="female_diameter" value="0.04" />  <!-- /m -->
@@ -41,5 +41,5 @@
             </geometry>
         </collision>
-        <xacro:box_inertial m="${male_m}" w="${male_w}" l="${male_l}" h="${male_h}" xyz="0 0 0 " rpy="0 0 0"/>
+        <xacro:box_inertial m="${male_m}" w="${male_w}" l="${male_l}" h="${male_h}" xyz="${-male_w/2} 0 0 " rpy="0 0 0"/>
     </link>
     <link name="${agent_namespace}_cover_link">

Commit message: fixing pivot link inertia

File: ros_ws/src/pipe_swarm/urdf/linkage.xacro (robot description, xacro)
@@ -5,5 +5,6 @@
     <xacro:property name="cover_h" value="0.024" />  <!-- height /m -->
     <xacro:property name="cover_l" value="0.024" />  <!-- length /m -->
-    <xacro:property name="cover_out" value="0.0015" />  <!-- length /m -->
+    <xacro:property name="cover_o" value="0.0045" />  <!-- offset /m -->
+    <xacro:property name="cover_out" value="0.0015" />  <!-- extruded cover /m -->
     <xacro:property name="male_m" value="0.1" />  <!-- mass /kg -->
     <xacro:property name="male_w" value="0.014" />  <!-- width /m -->
@@ -11,17 +12,11 @@
     <xacro:property name="male_h" value="0.0128" />  <!-- length /m -->
     <xacro:property name="male_o" value="0.007" />  <!-- offset /m -->
-    <xacro:property name="female_diameter" value="0.04" />  <!-- /m -->
-    <xacro:property name="female_stopper_width" value="0.05" />  <!-- /m -->
-    <xacro:property name="female_hole_depth" value="0.03" />  <!-- /m -->
-    <xacro:property name="female_wall_thickness" value="0.01" />  <!-- /m -->
-    <xacro:property name="female_hole_thickness" value="0.01" />  <!-- /m -->
-    <xacro:property name="female_m" value="0.1" />  <!-- mass /kg -->
-    <xacro:property name="female_w" value="${(female_diameter/2) + female_stopper_width + female_hole_depth}" />  <!-- width /m -->
-    <xacro:property name="female_h" value="${female_diameter}" />  <!-- height /m -->
-    <xacro:property name="female_l" value="0.028" />   <!-- length /m -->
-    <xacro:property name="pivot_l" value="0.055" />  <!-- length /m -->
+    <xacro:property name="pivot_m" value="0.1" />  <!-- mass /kg -->
+    <xacro:property name="pivot_w" value="0.035" />  <!-- width /m -->
+    <xacro:property name="pivot_h" value="0.024" />  <!-- height /m -->
+    <xacro:property name="pivot_l" value="0.055" />   <!-- length /m -->
+    <xacro:property name="pivot_o" value="0.0075" />  <!-- offset /m -->
     <xacro:property name="lock_w" value="0.02" />  <!-- width /m -->
     <xacro:property name="lock_o" value="0.01" />  <!-- offset /m -->
-    <xacro:property name="cover_o" value="0.0045" />  <!-- offset /m -->
     <!-- LINKS -->
     <link name="${agent_namespace}_male_link">
@@ -94,5 +89,5 @@
             </geometry>
         </collision>
-        <xacro:box_inertial m="${female_m}" w="0.05" l="0.05" h="0.05" xyz="0 0 0" rpy="0 0 0"/>
+        <xacro:box_inertial m="${pivot_m}" w="${pivot_w}" l="${pivot_l}" h="${pivot_h}" xyz="${-pivot_w/2 + pivot_o} 0 0" rpy="0 0 0"/>
     </link>
     <!-- JOINTS -->

Commit message: fixing female link inertia

File: ros_ws/src/pipe_swarm/urdf/linkage.xacro (robot description, xacro)
@@ -17,5 +17,8 @@
     <xacro:property name="pivot_l" value="0.055" />   <!-- length /m -->
     <xacro:property name="pivot_o" value="0.0075" />  <!-- offset /m -->
-    <xacro:property name="lock_w" value="0.02" />  <!-- width /m -->
+    <xacro:property name="female_m" value="0.1" />  <!-- mass /kg -->
+    <xacro:property name="female_w" value="0.02" />  <!-- width /m -->
+    <xacro:property name="female_h" value="0.024" />  <!-- height /m -->
+    <xacro:property name="female_l" value="0.024" />   <!-- length /m -->
     <xacro:property name="lock_o" value="0.01" />  <!-- offset /m -->
     <!-- LINKS -->
@@ -58,5 +61,5 @@
     <link name="${agent_namespace}_female_link">
        <visual>
-            <origin xyz="${-lock_w/2} 0 0" rpy="0.0 ${pi/2} ${pi/2}"/>
+            <origin xyz="${-female_w/2} 0 0" rpy="0.0 ${pi/2} ${pi/2}"/>
             <geometry>
                 <mesh filename="package://pipe_swarm/models/hollow_pipe/meshes/lock.stl" scale="0.001 0.001 0.001"/>
@@ -67,9 +70,10 @@
         </visual>
         <collision>
-            <origin xyz="${-lock_w/2} 0 0" rpy="0.0 ${pi/2} ${pi/2}"/>
+            <origin xyz="${-female_w/2} 0 0" rpy="0.0 ${pi/2} ${pi/2}"/>
             <geometry>
                 <mesh filename="package://pipe_swarm/models/hollow_pipe/meshes/lock.stl" scale="0.001 0.001 0.001"/>
             </geometry>
         </collision>
+        <xacro:box_inertial m="${female_m}" w="${female_w}" l="${female_l}" h="${female_h}" xyz="0 0 0" rpy="0 0 0"/>
     </link>
     <link name="${agent_namespace}_pivot_link">
