Commit message: renaming no chamfer linkage

File: ros_ws/src/pipe_swarm/urdf/linkage.xacro (robot description, xacro)
@@ -81,5 +81,5 @@
             <origin xyz="${-lock_w/2} 0 0" rpy="0.0 ${pi/2} ${pi/2}"/>
             <geometry>
-                <mesh filename="package://pipe_swarm/models/hollow_pipe/meshes/lock_v2_for_sim.stl" scale="0.001 0.001 0.001"/>
+                <mesh filename="package://pipe_swarm/models/hollow_pipe/meshes/lock_sim.stl" scale="0.001 0.001 0.001"/> <!-- no chamfer-->
             </geometry>
             <material name="base">
@@ -90,5 +90,5 @@
             <origin xyz="${-lock_w/2} 0 0" rpy="0.0 ${pi/2} ${pi/2}"/>
             <geometry>
-                <mesh filename="package://pipe_swarm/models/hollow_pipe/meshes/lock_v2_for_sim.stl" scale="0.001 0.001 0.001"/>
+                <mesh filename="package://pipe_swarm/models/hollow_pipe/meshes/lock_sim.stl" scale="0.001 0.001 0.001"/> <!-- no chamfer-->
             </geometry>
         </collision>

Commit message: Changing linkage settings

File: ros_ws/src/pipe_swarm/urdf/linkage.xacro (robot description, xacro)
@@ -38,4 +38,23 @@
                 <mesh filename="package://pipe_swarm/models/hollow_pipe/meshes/key.stl" scale="0.001 0.001 0.001"/>
             </geometry>
+            <surface>
+                <friction>
+                <ode>
+                    <mu>2.0</mu>   <!-- High friction -->
+                    <mu2>2.0</mu2>  <!-- High friction -->
+                    <slip1>0.0</slip1>
+                    <slip2>0.0</slip2>
+                </ode>
+                </friction>
+                <contact>
+                <ode>
+                    <!-- High stiffness/damping for hard contact -->
+                    <kp>1e7</kp> <!-- Increase stiffness (1e6 to 1e8) -->
+                    <kd>1000.0</kd> <!-- Increase damping (100 to 1000) -->
+                    <max_vel>0.1</max_vel> <!-- Lower max correction velocity for stability -->
+                    <min_depth>0.0005</min_depth> <!-- Smaller penetration depth -->
+                </ode>
+                </contact>
+            </surface>
         </collision>
         <xacro:box_inertial m="${male_m}" w="${male_w}" l="${male_l}" h="${male_h}" xyz="${-male_w/2} 0 0 " rpy="0 0 0"/>
@@ -74,4 +93,23 @@
                 <mesh filename="package://pipe_swarm/models/hollow_pipe/meshes/lock_sim.stl" scale="0.001 0.001 0.001"/> <!-- no chamfer-->
             </geometry>
+            <surface>
+                <friction>
+                <ode>
+                    <mu>2.0</mu>   <!-- High friction -->
+                    <mu2>2.0</mu2>  <!-- High friction -->
+                    <slip1>0.0</slip1>
+                    <slip2>0.0</slip2>
+                </ode>
+                </friction>
+                <contact>
+                <ode>
+                    <!-- High stiffness/damping for hard contact -->
+                    <kp>1e7</kp> <!-- Increase stiffness (1e6 to 1e8) -->
+                    <kd>1000.0</kd> <!-- Increase damping (100 to 1000) -->
+                    <max_vel>0.1</max_vel> <!-- Lower max correction velocity for stability -->
+                    <min_depth>0.0005</min_depth> <!-- Smaller penetration depth -->
+                </ode>
+                </contact>
+            </surface>
         </collision>
         <xacro:box_inertial m="${female_m}" w="${female_w}" l="${female_l}" h="${female_h}" xyz="0 0 0" rpy="0 0 0"/>
@@ -100,4 +138,5 @@
         <parent link="${agent_namespace}_base_link"/>
         <child link="${agent_namespace}_cover_link"/>
+        <dynamics damping="1.0" friction="2.0"/>
     </joint>
     <joint name="base_male_joint" type="revolute">
@@ -106,5 +145,6 @@
         <child link="${agent_namespace}_male_link"/>
         <axis xyz="1 0 0"/>
-        <limit lower="0.0" upper="${pi/2}" effort="1.0" velocity="1.0"/>
+        <limit lower="0.0" upper="${pi/2}" effort="5.0" velocity="2.5"/>
+        <dynamics damping="1.0" friction="2.0"/>
     </joint>
     <joint name="base_female_joint" type="revolute">
@@ -113,6 +153,6 @@
         <child link="${agent_namespace}_pivot_link"/>
         <axis xyz="0 1 0"/>
-        <limit lower="${-pi/4}" upper="${pi/4}" effort="0.5" velocity="0.5"/>
-        <dynamics damping="0.3" friction="0.5"/>
+        <limit lower="${-pi/4}" upper="${pi/4}" effort="50.0" velocity="0.2"/>
+        <dynamics damping="2.0" friction="0.2"/>
     </joint>
     <joint name="${agent_namespace}_base_neutral_joint" type="fixed">
