Commit message: Adjusting robot colours to match solidworks model

File: ros_ws/src/pipe_swarm/urdf/camera.xacro (robot description, xacro)
@@ -12,6 +12,6 @@
                 <box size="${camera_w} ${camera_l} ${camera_h}"/>
             </geometry>
-            <material name="base">
-                <color rgba="1.0 1.0 1.0 1.0"/>
+            <material name="green">
+                <color rgba="0 1 0 1"/>
             </material>
         </visual>
@@ -31,5 +31,5 @@
     <!-- GAZEBO -->
     <gazebo reference="camera_link">
-        <material>Gazebo/Red</material>
+        <material>Gazebo/Green</material>
         <sensor name="camera_sensor" type="camera">
             <pose>0 0 0 0 0 0</pose>

File: ros_ws/src/pipe_swarm/urdf/linkage.xacro (robot description, xacro)
@@ -124,5 +124,8 @@
     <!-- GAZEBO -->
     <gazebo reference="female_link">
-        <material>Gazebo/Red</material>
+        <material>Gazebo/White</material>
+    </gazebo>
+    <gazebo reference="male_link">
+        <material>Gazebo/White</material>
     </gazebo>
     <gazebo>

File: ros_ws/src/pipe_swarm/urdf/mobile_base.xacro (robot description, xacro)
@@ -13,6 +13,6 @@
                 <box size="${base_w} ${base_l} ${base_h}"/>
             </geometry>
-            <material name="red">
-                <color rgba="1 0 0 1"/>
+            <material name="blue">
+                <color rgba="0 0 1 1"/>
             </material>
         </visual>
@@ -30,3 +30,7 @@
         <child link="base_link"/>
     </joint>
+    <!-- GAZEBO -->
+    <gazebo reference="base_link">
+        <material>Gazebo/Blue</material>
+    </gazebo>
 </robot>

File: ros_ws/src/pipe_swarm/urdf/wheels.xacro (robot description, xacro)
@@ -12,5 +12,5 @@
                 </geometry>
                 <material name="wheel">
-                    <color rgba="1 1 1 1.0"/>
+                    <color rgba="0 0 0 1.0"/>
                 </material>
             </visual>
@@ -106,14 +106,14 @@
     </gazebo>
     <gazebo reference="wheel_front_right_link">
-        <material>Gazebo/Blue</material>
+        <material>Gazebo/Black</material>
     </gazebo>
     <gazebo reference="wheel_front_left_link">
-        <material>Gazebo/Blue</material>
+        <material>Gazebo/Black</material>
     </gazebo>
     <gazebo reference="wheel_back_right_link">
-        <material>Gazebo/Blue</material>
+        <material>Gazebo/Black</material>
     </gazebo>
     <gazebo reference="wheel_back_left_link">
-        <material>Gazebo/Blue</material>
+        <material>Gazebo/Black</material>
     </gazebo>
 </robot>

Commit message: adding namespace for camera and diff drive

File: ros_ws/src/pipe_swarm/urdf/camera.xacro (robot description, xacro)
@@ -37,4 +37,7 @@
             <update_rate>10.0</update_rate> <!--update /Hz -->
             <plugin name="camera_controller" filename="libgazebo_ros_camera.so">
+                <ros>
+                    <namespace>${agent_namespace}</namespace>
+                </ros>
                 <frame_name>camera_link</frame_name>
             </plugin>

File: ros_ws/src/pipe_swarm/urdf/pipe_robot.urdf.xacro (robot description, xacro)
@@ -1,4 +1,5 @@
 <?xml version="1.0"?>
-<robot name="pipe_robot" xmlns:xacro="http://www.ros.org/wiki/xacro">
+<robot name="pipe_robot" params="agent_namespace" xmlns:xacro="http://www.ros.org/wiki/xacro">
+     <xacro:property name="agent_namespace" value="$(arg agent_namespace)" />
     <xacro:include filename="common.xacro"/>
     <xacro:include filename="mobile_base.xacro"/>

File: ros_ws/src/pipe_swarm/urdf/wheels.xacro (robot description, xacro)
@@ -58,5 +58,8 @@
     <!-- GAZEBO -->
     <gazebo>
-        <plugin name="gazebo_ros_front_diff_drive" filename="libgazebo_ros_diff_drive.so">
+        <plugin name="front_diff_drive" filename="libgazebo_ros_diff_drive.so">
+            <ros>
+                <namespace>${agent_namespace}</namespace>
+            </ros>
             <!-- Update rate in Hz -->
             <update_rate>50</update_rate>
@@ -73,14 +76,17 @@
             <command_topic>cmd_vel</command_topic>
             <!-- output -->
+            <odometry_frame>odom</odometry_frame>
+            <robot_base_frame>footprint_link</robot_base_frame>
+            <odometry_topic>odom</odometry_topic>
             <publish_odom>true</publish_odom>
             <publish_odom_tf>true</publish_odom_tf>
             <publish_wheel_tf>true</publish_wheel_tf>
-            <odometry_topic>odom</odometry_topic>
-            <odometry_frame>odom</odometry_frame>
-            <robot_base_frame>footprint_link</robot_base_frame>
         </plugin>
     </gazebo>
     <gazebo>
-        <plugin name="gazebo_ros_back_diff_drive" filename="libgazebo_ros_diff_drive.so">
+        <plugin name="back_diff_drive" filename="libgazebo_ros_diff_drive.so">
+            <ros>
+                <namespace>${agent_namespace}</namespace>
+            </ros>
             <!-- Update rate in Hz -->
             <update_rate>50</update_rate>
@@ -97,10 +103,10 @@
             <command_topic>cmd_vel</command_topic>
             <!-- output -->
+            <odometry_frame>odom</odometry_frame>
+            <robot_base_frame>footprint_link</robot_base_frame>
+            <odometry_topic>odom</odometry_topic>
             <publish_odom>true</publish_odom>
             <publish_odom_tf>true</publish_odom_tf>
             <publish_wheel_tf>true</publish_wheel_tf>
-            <odometry_topic>odom</odometry_topic>
-            <odometry_frame>odom</odometry_frame>
-            <robot_base_frame>footprint_link</robot_base_frame>
         </plugin>
     </gazebo>

Commit message: updating link names to include namespace for tf publishing conflicts

File: ros_ws/src/pipe_swarm/urdf/camera.xacro (robot description, xacro)
@@ -6,5 +6,5 @@
     <xacro:property name="camera_h" value="0.01" />  <!-- height /m -->
     <!-- LINKS -->
-    <link name="camera_link">
+    <link name="${agent_namespace}_camera_link">
         <visual>
             <origin xyz="0.0 0.0 0.0" rpy="0.0 0.0 0.0"/>
@@ -24,11 +24,11 @@
     </link>
     <!-- JOINTS -->
-    <joint name="base_camera_joint" type="fixed">
+    <joint name="${agent_namespace}_base_camera_joint" type="fixed">
         <origin xyz="${(base_w*0.5)} 0 ${(base_h*0.5)}" rpy="0 0 0"/>
-        <parent link="base_link"/>
-        <child link="camera_link"/>
+        <parent link="${agent_namespace}_base_link"/>
+        <child link="${agent_namespace}_camera_link"/>
     </joint>
     <!-- GAZEBO -->
-    <gazebo reference="camera_link">
+    <gazebo reference="${agent_namespace}_camera_link">
         <material>Gazebo/Green</material>
         <sensor name="camera_sensor" type="camera">
@@ -40,5 +40,5 @@
                     <namespace>${agent_namespace}</namespace>
                 </ros>
-                <frame_name>camera_link</frame_name>
+                <frame_name>${agent_namespace}_camera_link</frame_name>
             </plugin>
         </sensor>

File: ros_ws/src/pipe_swarm/urdf/linkage.xacro (robot description, xacro)
@@ -33,5 +33,5 @@
     </xacro:macro>
     <!-- LINKS -->
-    <link name="male_link">
+    <link name="${agent_namespace}_male_link">
         <visual>
             <origin xyz="0.0 0.0 0.0" rpy="0.0 0.0 0.0"/>
@@ -50,5 +50,5 @@
         <xacro:box_inertial m="${male_m}" w="${male_w}" l="${male_l}" h="${male_h}" xyz="0 0 0 " rpy="0 0 0"/>
     </link>
-    <link name="female_link">
+    <link name="${agent_namespace}_female_link">
         <visual>
             <xacro:female_rotation_shape />
@@ -109,22 +109,21 @@
     </link>
     <!-- JOINTS -->
-    <joint name="base_male_joint" type="fixed">
+    <joint name="${agent_namespace}_base_male_joint" type="fixed">
         <origin xyz="${(base_w*0.5) + (male_w*0.5)} 0 0" rpy="0 0 0"/>
-        <parent link="base_link"/>
-        <child link="male_link"/>
+        <parent link="${agent_namespace}_base_link"/>
+        <child link="${agent_namespace}_male_link"/>
     </joint>
-    <joint name="base_female_joint" type="revolute">
-        <!-- <origin xyz="${-(base_w*0.5) + 0.023} 0 0" rpy="0 0 0"/> -->
+    <joint name="${agent_namespace}_base_female_joint" type="revolute">
         <origin xyz="${-(base_w*0.5) + female_diameter/2} 0 0" rpy="0 0 0"/>
-        <parent link="base_link"/>
-        <child link="female_link"/>
+        <parent link="${agent_namespace}_base_link"/>
+        <child link="${agent_namespace}_female_link"/>
         <axis xyz="0 1 0"/>
         <limit lower="${-pi/2}" upper="${pi/2}" effort="1.0" velocity="1.0"/>
     </joint>
     <!-- GAZEBO -->
-    <gazebo reference="female_link">
+    <gazebo reference="${agent_namespace}_female_link">
         <material>Gazebo/White</material>
     </gazebo>
-    <gazebo reference="male_link">
+    <gazebo reference="${agent_namespace}_male_link">
         <material>Gazebo/White</material>
     </gazebo>
@@ -132,5 +131,5 @@
         <plugin name="${agent_namespace}_control" filename="libgazebo_ros2_control.so">
             <robot_param_node>/${agent_namespace}/robot_state_publisher</robot_param_node>
-            <parameters>$(find pipe_swarm)/config/robot_controllers_sim.yaml</parameters>
+            <parameters>$(find pipe_swarm)/config/${agent_namespace}_controllers_sim.yaml</parameters>
             <ros>
                 <namespace>${agent_namespace}</namespace>
@@ -143,5 +142,5 @@
             <plugin>gazebo_ros2_control/GazeboSystem</plugin>
         </hardware>
-        <joint name="base_female_joint">
+        <joint name="${agent_namespace}_base_female_joint">
             <command_interface name="position">
                 <param name="min">-pi/2</param>
@@ -149,5 +148,5 @@
             </command_interface>
             <state_interface name="position">
-                <param name="initial_value">1.0</param>
+                <param name="initial_value">0.0</param>
             </state_interface>
             <state_interface name="velocity"/>

File: ros_ws/src/pipe_swarm/urdf/mobile_base.xacro (robot description, xacro)
@@ -6,6 +6,6 @@
     <xacro:property name="base_h" value="0.045" />  <!-- height /m -->
     <!-- LINKS -->
-    <link name="footprint_link" />
-    <link name="base_link">
+    <link name="${agent_namespace}_footprint_link" />
+    <link name="${agent_namespace}_base_link">
         <visual>
             <origin xyz="0.0 0.0 0.0" rpy="0.0 0.0 0.0"/>
@@ -25,14 +25,14 @@
     </link>
     <!-- JOINTS -->
-    <joint name="base_footprint" type="fixed">
+    <joint name="${agent_namespace}_base_footprint" type="fixed">
         <origin xyz="0 0 0.035" rpy="0 0 0"/>
-        <parent link="footprint_link"/>
-        <child link="base_link"/>
+        <parent link="${agent_namespace}_footprint_link"/>
+        <child link="${agent_namespace}_base_link"/>
     </joint>
     <!-- GAZEBO -->
-    <gazebo reference="footprint_link">
+    <gazebo reference="${agent_namespace}_footprint_link">
         <material>Gazebo/Blue</material>
     </gazebo>
-    <gazebo reference="base_link">
+    <gazebo reference="${agent_namespace}_base_link">
         <material>Gazebo/Blue</material>
     </gazebo>

File: ros_ws/src/pipe_swarm/urdf/wheels.xacro (robot description, xacro)
@@ -5,5 +5,5 @@
     <xacro:property name="wheel_l" value="0.01" />  <!-- length /m -->
     <xacro:macro name="wheel_link" params="prefix">
-        <link name="wheel_${prefix}_link">
+        <link name="${agent_namespace}_wheel_${prefix}_link">
             <visual>
                 <origin xyz="0.0 0.0 0.0" rpy="${pi/2} 0.0 0.0"/>
@@ -30,33 +30,33 @@
     <xacro:wheel_link prefix="back_left" />
     <!-- JOINTS -->
-    <joint name="base_wheel_front_right_joint" type="continuous">
+    <joint name="${agent_namespace}_base_wheel_front_right_joint" type="continuous">
         <origin xyz="${(base_w)/2 - wheel_r} ${-((base_l/2) + (wheel_l/2))} ${-base_h/2}" rpy="0 0 0"/>
-        <parent link="base_link"/>
-        <child link="wheel_front_right_link"/>
+        <parent link="${agent_namespace}_base_link"/>
+        <child link="${agent_namespace}_wheel_front_right_link"/>
         <axis xyz="0 1 0"/>
     </joint>
-    <joint name="base_wheel_front_left_joint" type="continuous">
+    <joint name="${agent_namespace}_base_wheel_front_left_joint" type="continuous">
         <origin xyz="${(base_w)/2 - wheel_r} ${(base_l/2) + (wheel_l/2)} ${-base_h/2}" rpy="0 0 0"/>
-        <parent link="base_link"/>
-        <child link="wheel_front_left_link"/>
+        <parent link="${agent_namespace}_base_link"/>
+        <child link="${agent_namespace}_wheel_front_left_link"/>
         <axis xyz="0 1 0"/>
     </joint>
-    <joint name="base_wheel_back_right_joint" type="continuous">
+    <joint name="${agent_namespace}_base_wheel_back_right_joint" type="continuous">
         <origin xyz="${-((base_w)/2 - wheel_r)} ${-((base_l/2) + (wheel_l/2))} ${-base_h/2}" rpy="0 0 0"/>
-        <parent link="base_link"/>
-        <child link="wheel_back_right_link"/>
+        <parent link="${agent_namespace}_base_link"/>
+        <child link="${agent_namespace}_wheel_back_right_link"/>
         <axis xyz="0 1 0"/>
-        <mimic joint="base_wheel_front_right_joint" multiplier="1.0"/>
+        <mimic joint="${agent_namespace}_base_wheel_front_right_joint" multiplier="1.0"/>
     </joint>
-    <joint name="base_wheel_back_left_joint" type="continuous">
+    <joint name="${agent_namespace}_base_wheel_back_left_joint" type="continuous">
         <origin xyz="${-((base_w)/2 - wheel_r)} ${(base_l/2) + (wheel_l/2)} ${-base_h/2}" rpy="0 0 0"/>
-        <parent link="base_link"/>
-        <child link="wheel_back_left_link"/>
+        <parent link="${agent_namespace}_base_link"/>
+        <child link="${agent_namespace}_wheel_back_left_link"/>
         <axis xyz="0 1 0"/>
-        <mimic joint="base_wheel_front_left_joint" multiplier="1.0"/>
+        <mimic joint="${agent_namespace}_base_wheel_front_left_joint" multiplier="1.0"/>
     </joint>
     <!-- GAZEBO -->
     <gazebo>
-        <plugin name="front_diff_drive" filename="libgazebo_ros_diff_drive.so">
+        <plugin name="${agent_namespace}_front_diff_drive" filename="libgazebo_ros_diff_drive.so">
             <ros>
                 <namespace>${agent_namespace}</namespace>
@@ -65,6 +65,6 @@
             <update_rate>50</update_rate>
             <!-- wheels -->
-            <right_joint>base_wheel_front_right_joint</right_joint>
-            <left_joint>base_wheel_front_left_joint</left_joint>
+            <right_joint>${agent_namespace}_base_wheel_front_right_joint</right_joint>
+            <left_joint>${agent_namespace}_base_wheel_front_left_joint</left_joint>
             <!-- kinematics -->
             <wheel_separation>0.85</wheel_separation>
@@ -77,5 +77,5 @@
             <!-- output -->
             <odometry_frame>odom</odometry_frame>
-            <robot_base_frame>footprint_link</robot_base_frame>
+            <robot_base_frame>${agent_namespace}_footprint_link</robot_base_frame>
             <odometry_topic>odom</odometry_topic>
             <publish_odom>true</publish_odom>
@@ -85,5 +85,5 @@
     </gazebo>
     <gazebo>
-        <plugin name="back_diff_drive" filename="libgazebo_ros_diff_drive.so">
+        <plugin name="${agent_namespace}_back_diff_drive" filename="libgazebo_ros_diff_drive.so">
             <ros>
                 <namespace>${agent_namespace}</namespace>
@@ -92,6 +92,6 @@
             <update_rate>50</update_rate>
             <!-- wheels -->
-            <right_joint>base_wheel_back_right_joint</right_joint>
-            <left_joint>base_wheel_back_left_joint</left_joint>
+            <right_joint>${agent_namespace}_base_wheel_back_right_joint</right_joint>
+            <left_joint>${agent_namespace}_base_wheel_back_left_joint</left_joint>
             <!-- kinematics -->
             <wheel_separation>0.85</wheel_separation>
@@ -104,5 +104,5 @@
             <!-- output -->
             <odometry_frame>odom</odometry_frame>
-            <robot_base_frame>footprint_link</robot_base_frame>
+            <robot_base_frame>${agent_namespace}_footprint_link</robot_base_frame>
             <odometry_topic>odom</odometry_topic>
             <publish_odom>true</publish_odom>
