Commit message: isolating gazebo plugins and urdf

File: ros_ws/src/pipe_swarm/urdf/camera.xacro (robot description, xacro)
@@ -29,18 +29,3 @@
         <child link="${agent_namespace}_camera_link"/>
     </joint>
-    <!-- GAZEBO -->
-    <gazebo reference="${agent_namespace}_camera_link">
-        <material>Gazebo/Green</material>
-        <sensor name="camera_sensor" type="camera">
-            <pose>0 0 0 0 0 0</pose>
-            <visualize>true</visualize>
-            <update_rate>10.0</update_rate> <!--update /Hz -->
-            <plugin name="camera_controller" filename="libgazebo_ros_camera.so">
-                <ros>
-                    <namespace>${agent_namespace}</namespace>
-                </ros>
-                <frame_name>${agent_namespace}_camera_link</frame_name>
-            </plugin>
-        </sensor>
-    </gazebo>
 </robot>

File: ros_ws/src/pipe_swarm/urdf/gazebo/pipe_robot.xacro (robot description, xacro)
@@ -1,8 +1,6 @@
 <?xml version="1.0"?>
-<robot name="pipe_robot" xmlns:xacro="http://www.ros.org/wiki/xacro">
-    <xacro:macro name="pipe_robot" params="namespace">
-        <xacro:property name="agent_namespace" value="${namespace}" />
+<robot name="gazebo_pipe_robot" xmlns:xacro="http://www.ros.org/wiki/xacro">
+    <xacro:macro name="gazebo_pipe_robot" params="namespace">
         <!-- Include shared components -->
-        <xacro:include filename="common.xacro"/>
         <xacro:include filename="mobile_base.xacro"/>
         <xacro:include filename="lidar.xacro"/>
@@ -11,5 +9,5 @@
         <xacro:include filename="wheels.xacro"/>
         <xacro:include filename="linkage.xacro"/>
-        <xacro:include filename="gazebo/pipe_robot.xacro"/>
     </xacro:macro>
+    <xacro:gazebo_pipe_robot namespace="${agent_namespace}" />
 </robot>

File: ros_ws/src/pipe_swarm/urdf/lidar.xacro (robot description, xacro)
@@ -29,34 +29,3 @@
         <child link="${agent_namespace}_lidar_link"/>
     </joint>
-    <!-- GAZEBO -->
-    <gazebo reference="${agent_namespace}_lidar_link">
-        <material>Gazebo/Green</material>
-        <sensor name="lidar_sensor" type="lidar">
-            <pose>0 0 0 0 0 0</pose>
-            <visualize>true</visualize>
-            <update_rate>10.0</update_rate>
-            <ray>
-                <scan>
-                    <horizontal>
-                        <samples>100</samples>
-                        <min_angle>${pi/2}</min_angle>
-                        <max_angle>${-pi/2}</max_angle>
-                    </horizontal>
-                </scan>
-                <range>
-                    <min>0.1</min>
-                    <max>1</max>
-                </range>
-            </ray>
-            <plugin name="lidar_controller" filename="libgazebo_ros_ray_sensor.so">
-                <ros>
-                    <namespace>${agent_namespace}</namespace>
-                    <remapping>~/out:=laserscan</remapping>
-                </ros>
-                <output_type>sensor_msgs/LaserScan</output_type>
-                <min_intensity>100.0</min_intensity>
-                <frame_name>${agent_namespace}_lidar_link</frame_name>
-            </plugin>
-        </sensor>
-    </gazebo>
 </robot>

File: ros_ws/src/pipe_swarm/urdf/linkage.xacro (robot description, xacro)
@@ -124,36 +124,3 @@
         <limit lower="${-pi/2}" upper="${pi/2}" effort="1.0" velocity="1.0"/>
     </joint>
-    <!-- GAZEBO -->
-    <gazebo reference="${agent_namespace}_female_link">
-        <material>Gazebo/White</material>
-    </gazebo>
-    <gazebo reference="${agent_namespace}_male_link">
-        <material>Gazebo/White</material>
-    </gazebo>
-    <gazebo>
-        <plugin name="${agent_namespace}_control" filename="libgazebo_ros2_control.so">
-            <robot_param_node>/${agent_namespace}/robot_state_publisher</robot_param_node>
-            <parameters>$(find pipe_swarm)/config/robot_controllers_sim.yaml</parameters>
-            <ros>
-                <namespace>${agent_namespace}</namespace>
-            </ros>
-        </plugin>
-    </gazebo>
-    <!-- ros2_control Plugin -->
-    <ros2_control name="GazeboSystem" type="system">
-        <hardware>
-            <plugin>gazebo_ros2_control/GazeboSystem</plugin>
-        </hardware>
-        <joint name="base_female_joint">
-            <command_interface name="position">
-                <param name="min">-pi/2</param>
-                <param name="max">pi/2</param>
-            </command_interface>
-            <state_interface name="position">
-                <param name="initial_value">0.0</param>
-            </state_interface>
-            <state_interface name="velocity"/>
-            <state_interface name="effort"/>
-        </joint>
-    </ros2_control>
 </robot>

File: ros_ws/src/pipe_swarm/urdf/mobile_base.xacro (robot description, xacro)
@@ -30,10 +30,3 @@
         <child link="${agent_namespace}_base_link"/>
     </joint>
-    <!-- GAZEBO -->
-    <gazebo reference="${agent_namespace}_footprint_link">
-        <material>Gazebo/Blue</material>
-    </gazebo>
-    <gazebo reference="${agent_namespace}_base_link">
-        <material>Gazebo/Blue</material>
-    </gazebo>
 </robot>

File: ros_ws/src/pipe_swarm/urdf/tof.xacro (robot description, xacro)
@@ -51,64 +51,3 @@
         <child link="${agent_namespace}_left_tof_link"/>
     </joint>
-    <!-- GAZEBO -->
-    <gazebo reference="${agent_namespace}_right_tof_link">
-        <material>Gazebo/Green</material>
-        <sensor name="${agent_namespace}_right_tof_sensor" type="ray">
-            <pose>0 0 0 0 0 0</pose>
-            <visualize>true</visualize>
-            <update_rate>10.0</update_rate>
-            <ray>
-                <scan>
-                    <horizontal>
-                        <samples>10</samples>
-                        <resolution>1</resolution>
-                    </horizontal>
-                </scan>
-                <range>
-                    <min>0.1</min>
-                    <max>10.0</max>
-                    <resolution>0.01</resolution>
-                </range>
-            </ray>
-            <plugin name="${agent_namespace}_right_tof_controller" filename="libgazebo_ros_ray_sensor.so">
-                <ros>
-                    <namespace>${agent_namespace}</namespace>
-                    <remapping>~/out:=right_infrared_range</remapping>
-                </ros>
-                <output_type>sensor_msgs/Range</output_type>
-                <radiation_type>infrared</radiation_type>
-                <frame_name>${agent_namespace}_right_tof_link</frame_name>
-            </plugin>
-        </sensor>
-    </gazebo>
-    <gazebo reference="${agent_namespace}_left_tof_link">
-        <material>Gazebo/Green</material>
-        <sensor name="${agent_namespace}_left_tof_sensor" type="ray">
-            <pose>0 0 0 0 0 0</pose>
-            <visualize>true</visualize>
-            <update_rate>10.0</update_rate>
-            <ray>
-                <scan>
-                    <horizontal>
-                        <samples>10</samples>
-                        <resolution>1</resolution>
-                    </horizontal>
-                </scan>
-                <range>
-                    <min>0.1</min>
-                    <max>10.0</max>
-                    <resolution>0.01</resolution>
-                </range>
-            </ray>
-            <plugin name="${agent_namespace}_left_tof_controller" filename="libgazebo_ros_ray_sensor.so">
-                <ros>
-                    <namespace>${agent_namespace}</namespace>
-                    <remapping>~/out:=left_infrared_range</remapping>
-                </ros>
-                <output_type>sensor_msgs/Range</output_type>
-                <frame_name>${agent_namespace}_left_tof_link</frame_name>
-                <radiation_type>infrared</radiation_type>
-            </plugin>
-        </sensor>
-    </gazebo>
 </robot>

File: ros_ws/src/pipe_swarm/urdf/wheels.xacro (robot description, xacro)
@@ -56,112 +56,3 @@
         <!-- <mimic joint="base_wheel_front_left_joint" multiplier="1.0"/> -->
     </joint>
-    <!-- GAZEBO -->
-    <gazebo>
-        <plugin name="${agent_namespace}_diff_drive" filename="libgazebo_ros_diff_drive.so">
-            <ros>
-                <namespace>${agent_namespace}</namespace>
-            </ros>
-            <update_rate>50</update_rate>
-            <right_joint>base_wheel_back_right_joint</right_joint>
-            <left_joint>base_wheel_back_left_joint</left_joint>
-            <wheel_separation>${base_l + wheel_l}</wheel_separation>
-            <wheel_diameter>${wheel_r*2}</wheel_diameter>
-            <max_wheel_torque>20</max_wheel_torque>
-            <max_wheel_acceleration>1</max_wheel_acceleration>
-            <command_topic>cmd_vel</command_topic>
-            <odometry_frame>odom</odometry_frame>
-            <robot_base_frame>${agent_namespace}_footprint_link</robot_base_frame>
-            <odometry_topic>odom</odometry_topic>
-            <publish_odom>true</publish_odom>
-            <publish_odom_tf>true</publish_odom_tf>
-            <publish_wheel_tf>true</publish_wheel_tf>
-        </plugin>
-    </gazebo>
-    <gazebo>
-        <plugin name="${agent_namespace}_diff_drive_2" filename="libgazebo_ros_diff_drive.so">
-            <ros>
-                <namespace>${agent_namespace}</namespace>
-            </ros>
-            <update_rate>50</update_rate>
-            <right_joint>base_wheel_front_right_joint</right_joint>
-            <left_joint>base_wheel_front_left_joint</left_joint>
-            <wheel_separation>${base_l + wheel_l}</wheel_separation>
-            <wheel_diameter>${wheel_r*2}</wheel_diameter>
-            <max_wheel_torque>20</max_wheel_torque>
-            <max_wheel_acceleration>1</max_wheel_acceleration>
-            <command_topic>cmd_vel</command_topic>
-            <odometry_frame>odom</odometry_frame>
-            <robot_base_frame>${agent_namespace}_footprint_link</robot_base_frame>
-            <odometry_topic>odom</odometry_topic>
-            <publish_odom>true</publish_odom>
-            <publish_odom_tf>true</publish_odom_tf>
-            <publish_wheel_tf>true</publish_wheel_tf>
-        </plugin>
-    </gazebo>
-    <!-- <gazebo>
-        <plugin name="${agent_namespace}_control" filename="libgazebo_ros2_control.so">
-            <robot_param_node>/${agent_namespace}/robot_state_publisher</robot_param_node>
-            <parameters>$(find pipe_swarm)/config/robot_controllers_sim.yaml</parameters>
-            <ros>
-                <namespace>${agent_namespace}</namespace>
-            </ros>
-        </plugin>
-    </gazebo>
-    <ros2_control name="GazeboSystem" type="system">
-        <hardware>
-            <plugin>gazebo_ros2_control/GazeboSystem</plugin>
-        </hardware>
-        <joint name="base_wheel_front_right_joint">
-            <command_interface name="velocity">
-                <param name="min">-2</param>
-                <param name="max">2</param>
-            </command_interface>
-            <state_interface name="position"/>
-            <state_interface name="velocity"/>
-        </joint>
-        <joint name="base_wheel_front_left_joint">
-            <command_interface name="velocity">
-                <param name="min">-2</param>
-                <param name="max">2</param>
-            </command_interface>
-            <state_interface name="position"/>
-            <state_interface name="velocity"/>
-        </joint>
-        <joint name="base_wheel_back_right_joint">
-            <command_interface name="velocity">
-                <param name="min">-2</param>
-                <param name="max">2</param>
-            </command_interface>
-            <state_interface name="position"/>
-            <state_interface name="velocity"/>
-        </joint>
-        <joint name="base_wheel_back_left_joint">
-            <command_interface name="velocity">
-                <param name="min">-2</param>
-                <param name="max">2</param>
-            </command_interface>
-            <state_interface name="position"/>
-            <state_interface name="velocity"/>
-        </joint>
-    </ros2_control> -->
-    <gazebo reference="${agent_namespace}_wheel_front_right_link">
-        <material>Gazebo/Black</material>
-        <mu1 value="1.0"/>
-        <mu2 value="1.0"/>
-    </gazebo>
-    <gazebo reference="${agent_namespace}_wheel_front_left_link">
-        <material>Gazebo/Black</material>
-        <mu1 value="1.0"/>
-        <mu2 value="1.0"/>
-    </gazebo>
-    <gazebo reference="${agent_namespace}_wheel_back_right_link">
-        <material>Gazebo/Black</material>
-        <mu1 value="1.0"/>
-        <mu2 value="1.0"/>
-    </gazebo>
-    <gazebo reference="${agent_namespace}_wheel_back_left_link">
-        <material>Gazebo/Black</material>
-        <mu1 value="1.0"/>
-        <mu2 value="1.0"/>
-    </gazebo>
 </robot>

Commit message: Moved camera and changed frame rate for better obstacle detection

File: ros_ws/src/pipe_swarm/urdf/camera.xacro (robot description, xacro)
@@ -25,5 +25,5 @@
     <!-- JOINTS -->
     <joint name="${agent_namespace}_base_camera_joint" type="fixed">
-        <origin xyz="${(base_w*0.5)} 0 ${(base_h*0.5)}" rpy="0 0 0"/>
+        <origin xyz="${(base_w*0.5)} 0 ${(base_h*0.5)+(camera_w*0.5)}" rpy="0 0 0"/>
         <parent link="${agent_namespace}_base_link"/>
         <child link="${agent_namespace}_camera_link"/>
@@ -42,4 +42,5 @@
                     <height>640</height>
                     <format>R8G8B8</format>
+                    <fps>10</fps>
                 </image>
                 <clip>
