Commit message: isolating gazebo plugins from modular files

File: ros_ws/src/pipe_swarm/urdf/camera.xacro (robot description, xacro)
@@ -29,31 +29,3 @@
         <child link="${agent_namespace}_camera_link"/>
     </joint>
-    <!-- GAZEBO -->
-    <gazebo reference="${agent_namespace}_camera_link">
-        <material>Gazebo/Green</material>
-        <sensor name="camera_sensor" type="camera">
-            <pose>0 0 0 0 0 0</pose>
-            <visualize>true</visualize>
-            <update_rate>10.0</update_rate> <!--update /Hz -->
-            <camera>
-                <horizontal_fov>0.02</horizontal_fov>
-                <image>
-                    <width>480</width>
-                    <height>640</height>
-                    <format>R8G8B8</format>
-                    <fps>10</fps>
-                </image>
-                <clip>
-                    <near>0.05</near>
-                    <far>0.3</far>
-                </clip>
-            </camera>
-            <plugin name="camera_controller" filename="libgazebo_ros_camera.so">
-                <ros>
-                    <namespace>${agent_namespace}</namespace>
-                </ros>
-                <frame_name>${agent_namespace}_camera_link</frame_name>
-            </plugin>
-        </sensor>
-    </gazebo>
 </robot>

File: ros_ws/src/pipe_swarm/urdf/gazebo/camera.xacro (robot description, xacro)
@@ -8,4 +8,17 @@
             <visualize>true</visualize>
             <update_rate>10.0</update_rate> <!--update /Hz -->
+            <camera>
+                <horizontal_fov>0.02</horizontal_fov>
+                <image>
+                    <width>480</width>
+                    <height>640</height>
+                    <format>R8G8B8</format>
+                    <fps>10</fps>
+                </image>
+                <clip>
+                    <near>0.05</near>
+                    <far>0.3</far>
+                </clip>
+            </camera>
             <plugin name="camera_controller" filename="libgazebo_ros_camera.so">
                 <ros>

File: ros_ws/src/pipe_swarm/urdf/gazebo/linkage.xacro (robot description, xacro)
@@ -6,4 +6,10 @@
     </gazebo>
     <gazebo reference="${agent_namespace}_male_link">
+        <material>Gazebo/White</material>
+    </gazebo>
+    <gazebo reference="${agent_namespace}_pivot_link">
+        <material>Gazebo/White</material>
+    </gazebo>
+        <gazebo reference="${agent_namespace}_neutral_link">
         <material>Gazebo/White</material>
     </gazebo>
@@ -24,6 +30,6 @@
         <joint name="base_female_joint">
             <command_interface name="position">
-                <param name="min">-pi/2</param>
-                <param name="max">pi/2</param>
+                <param name="min">-pi/4</param>
+                <param name="max">pi/4</param>
             </command_interface>
             <state_interface name="position">
@@ -31,4 +37,5 @@
             </state_interface>
             <state_interface name="velocity"/>
+            <state_interface name="effort"/>
         </joint>
     </ros2_control>

File: ros_ws/src/pipe_swarm/urdf/gazebo/wheels.xacro (robot description, xacro)
@@ -10,5 +10,5 @@
             <right_joint>${agent_namespace}_base_wheel_back_right_joint</right_joint>
             <left_joint>${agent_namespace}_base_wheel_back_left_joint</left_joint>
-            <wheel_separation>${base_l + wheel_l}</wheel_separation>
+            <wheel_separation>${base_l + wheel_l+ 2*wheel_y_offset}</wheel_separation>
             <wheel_diameter>${wheel_r*2}</wheel_diameter>
             <max_wheel_torque>20</max_wheel_torque>
@@ -16,5 +16,5 @@
             <command_topic>cmd_vel</command_topic>
             <odometry_frame>odom</odometry_frame>
-            <robot_base_frame>${base_agent}_footprint_link</robot_base_frame>
+            <robot_base_frame>${agent_namespace}_footprint_link</robot_base_frame>
             <odometry_topic>odom</odometry_topic>
             <publish_odom>true</publish_odom>
@@ -31,5 +31,5 @@
             <right_joint>${agent_namespace}_base_wheel_front_right_joint</right_joint>
             <left_joint>${agent_namespace}_base_wheel_front_left_joint</left_joint>
-            <wheel_separation>${base_l + wheel_l}</wheel_separation>
+            <wheel_separation>${base_l + wheel_l+ 2*wheel_y_offset}</wheel_separation>
             <wheel_diameter>${wheel_r*2}</wheel_diameter>
             <max_wheel_torque>20</max_wheel_torque>
@@ -37,5 +37,5 @@
             <command_topic>cmd_vel</command_topic>
             <odometry_frame>odom</odometry_frame>
-            <robot_base_frame>${base_agent}_footprint_link</robot_base_frame>
+            <robot_base_frame>${agent_namespace}_footprint_link</robot_base_frame>
             <odometry_topic>odom</odometry_topic>
             <publish_odom>true</publish_odom>

File: ros_ws/src/pipe_swarm/urdf/linkage.xacro (robot description, xacro)
@@ -123,5 +123,5 @@
         <child link="${agent_namespace}_pivot_link"/>
         <axis xyz="0 1 0"/>
-        <limit lower="${-pi/2}" upper="${pi/2}" effort="1.0" velocity="1.0"/>
+        <limit lower="${-pi/4}" upper="${pi/4}" effort="1.0" velocity="1.0"/>
     </joint>
     <!-- <joint name="${agent_namespace}_footprint_base_joint" type="fixed">
@@ -135,42 +135,3 @@
         <child link="${agent_namespace}_female_link"/>
     </joint>
-    <!-- GAZEBO -->
-    <gazebo reference="${agent_namespace}_female_link">
-        <material>Gazebo/White</material>
-    </gazebo>
-    <gazebo reference="${agent_namespace}_male_link">
-        <material>Gazebo/White</material>
-    </gazebo>
-    <gazebo reference="${agent_namespace}_pivot_link">
-        <material>Gazebo/White</material>
-    </gazebo>
-        <gazebo reference="${agent_namespace}_neutral_link">
-        <material>Gazebo/White</material>
-    </gazebo>
-    <gazebo>
-        <plugin name="${agent_namespace}_control" filename="libgazebo_ros2_control.so">
-            <robot_param_node>/${agent_namespace}/robot_state_publisher</robot_param_node>
-            <parameters>$(find pipe_swarm)/config/robot_controllers_sim.yaml</parameters>
-            <ros>
-                <namespace>${agent_namespace}</namespace>
-            </ros>
-        </plugin>
-    </gazebo>
-    <!-- ros2_control Plugin -->
-    <ros2_control name="GazeboSystem" type="system">
-        <hardware>
-            <plugin>gazebo_ros2_control/GazeboSystem</plugin>
-        </hardware>
-        <joint name="base_female_joint">
-            <command_interface name="position">
-                <param name="min">-pi/2</param>
-                <param name="max">pi/2</param>
-            </command_interface>
-            <state_interface name="position">
-                <param name="initial_value">0.0</param>
-            </state_interface>
-            <state_interface name="velocity"/>
-            <state_interface name="effort"/>
-        </joint>
-    </ros2_control>
 </robot>

File: ros_ws/src/pipe_swarm/urdf/wheels.xacro (robot description, xacro)
@@ -79,112 +79,3 @@
         <!-- <mimic joint="${agent_namespace}_base_wheel_front_left_joint" multiplier="1.0"/> -->
     </joint>
-    <!-- GAZEBO -->
-    <gazebo>
-        <plugin name="${agent_namespace}_diff_drive" filename="libgazebo_ros_diff_drive.so">
-            <ros>
-                <namespace>${agent_namespace}</namespace>
-            </ros>
-            <update_rate>50</update_rate>
-            <right_joint>base_wheel_back_right_joint</right_joint>
-            <left_joint>base_wheel_back_left_joint</left_joint>
-            <wheel_separation>${base_l + wheel_l+ 2*wheel_y_offset}</wheel_separation>
-            <wheel_diameter>${wheel_r*2}</wheel_diameter>
-            <max_wheel_torque>20</max_wheel_torque>
-            <max_wheel_acceleration>1</max_wheel_acceleration>
-            <command_topic>cmd_vel</command_topic>
-            <odometry_frame>odom</odometry_frame>
-            <robot_base_frame>${agent_namespace}_footprint_link</robot_base_frame>
-            <odometry_topic>odom</odometry_topic>
-            <publish_odom>true</publish_odom>
-            <publish_odom_tf>true</publish_odom_tf>
-            <publish_wheel_tf>true</publish_wheel_tf>
-        </plugin>
-    </gazebo>
-    <gazebo>
-        <plugin name="${agent_namespace}_diff_drive_2" filename="libgazebo_ros_diff_drive.so">
-            <ros>
-                <namespace>${agent_namespace}</namespace>
-            </ros>
-            <update_rate>50</update_rate>
-            <right_joint>base_wheel_front_right_joint</right_joint>
-            <left_joint>base_wheel_front_left_joint</left_joint>
-            <wheel_separation>${base_l + wheel_l+ 2*wheel_y_offset}</wheel_separation>
-            <wheel_diameter>${wheel_r*2}</wheel_diameter>
-            <max_wheel_torque>20</max_wheel_torque>
-            <max_wheel_acceleration>1</max_wheel_acceleration>
-            <command_topic>cmd_vel</command_topic>
-            <odometry_frame>odom</odometry_frame>
-            <robot_base_frame>${agent_namespace}_footprint_link</robot_base_frame>
-            <odometry_topic>odom</odometry_topic>
-            <publish_odom>true</publish_odom>
-            <publish_odom_tf>true</publish_odom_tf>
-            <publish_wheel_tf>true</publish_wheel_tf>
-        </plugin>
-    </gazebo>
-    <!-- <gazebo>
-        <plugin name="${agent_namespace}_control" filename="libgazebo_ros2_control.so">
-            <robot_param_node>/${agent_namespace}/robot_state_publisher</robot_param_node>
-            <parameters>$(find pipe_swarm)/config/robot_controllers_sim.yaml</parameters>
-            <ros>
-                <namespace>${agent_namespace}</namespace>
-            </ros>
-        </plugin>
-    </gazebo>
-    <ros2_control name="GazeboSystem" type="system">
-        <hardware>
-            <plugin>gazebo_ros2_control/GazeboSystem</plugin>
-        </hardware>
-        <joint name="base_wheel_front_right_joint">
-            <command_interface name="velocity">
-                <param name="min">-2</param>
-                <param name="max">2</param>
-            </command_interface>
-            <state_interface name="position"/>
-            <state_interface name="velocity"/>
-        </joint>
-        <joint name="base_wheel_front_left_joint">
-            <command_interface name="velocity">
-                <param name="min">-2</param>
-                <param name="max">2</param>
-            </command_interface>
-            <state_interface name="position"/>
-            <state_interface name="velocity"/>
-        </joint>
-        <joint name="base_wheel_back_right_joint">
-            <command_interface name="velocity">
-                <param name="min">-2</param>
-                <param name="max">2</param>
-            </command_interface>
-            <state_interface name="position"/>
-            <state_interface name="velocity"/>
-        </joint>
-        <joint name="base_wheel_back_left_joint">
-            <command_interface name="velocity">
-                <param name="min">-2</param>
-                <param name="max">2</param>
-            </command_interface>
-            <state_interface name="position"/>
-            <state_interface name="velocity"/>
-        </joint>
-    </ros2_control> -->
-    <gazebo reference="${agent_namespace}_wheel_front_right_link">
-        <material>Gazebo/Black</material>
-        <mu1 value="1.0"/>
-        <mu2 value="1.0"/>
-    </gazebo>
-    <gazebo reference="${agent_namespace}_wheel_front_left_link">
-        <material>Gazebo/Black</material>
-        <mu1 value="1.0"/>
-        <mu2 value="1.0"/>
-    </gazebo>
-    <gazebo reference="${agent_namespace}_wheel_back_right_link">
-        <material>Gazebo/Black</material>
-        <mu1 value="1.0"/>
-        <mu2 value="1.0"/>
-    </gazebo>
-    <gazebo reference="${agent_namespace}_wheel_back_left_link">
-        <material>Gazebo/Black</material>
-        <mu1 value="1.0"/>
-        <mu2 value="1.0"/>
-    </gazebo>
 </robot>

Commit message: updating pipe_swarm masses

File: ros_ws/src/pipe_swarm/urdf/camera.xacro (robot description, xacro)
@@ -1,5 +1,5 @@
 <?xml version="1.0"?>
 <robot name="camera" xmlns:xacro="http://www.ros.org/wiki/xacro">
-    <xacro:property name="camera_m" value="0.1" />  <!-- mass /kg -->
+    <xacro:property name="camera_m" value="0.001" />  <!-- mass /kg -->
     <xacro:property name="camera_w" value="0.01" />  <!-- width /m -->
     <xacro:property name="camera_l" value="0.01" />  <!-- length /m -->

File: ros_ws/src/pipe_swarm/urdf/detection_object.xacro (robot description, xacro)
@@ -1,5 +1,5 @@
 <?xml version="1.0"?>
 <robot name="obstacle" xmlns:xacro="http://www.ros.org/wiki/xacro">
-    <xacro:property name="obstacle_m" value="0.1" />  <!-- mass /kg -->
+    <xacro:property name="obstacle_m" value="0.001" />  <!-- mass /kg -->
     <xacro:property name="obstacle_w" value="0.01" />  <!-- width /m -->
     <xacro:property name="obstacle_l" value="0.01" />  <!-- length /m -->

File: ros_ws/src/pipe_swarm/urdf/front_tof.xacro (robot description, xacro)
@@ -1,5 +1,5 @@
 <?xml version="1.0"?>
 <robot name="front_tof" xmlns:xacro="http://www.ros.org/wiki/xacro">
-    <xacro:property name="front_tof_m" value="0.1" />  <!-- mass /kg -->
+    <xacro:property name="front_tof_m" value="0.001" />  <!-- mass /kg -->
     <xacro:property name="front_tof_w" value="0.01" />  <!-- width /m -->
     <xacro:property name="front_tof_l" value="0.01" />  <!-- length /m -->

File: ros_ws/src/pipe_swarm/urdf/imu.xacro (robot description, xacro)
@@ -1,5 +1,5 @@
 <?xml version="1.0"?>
 <robot name="imu" xmlns:xacro="http://www.ros.org/wiki/xacro">
-    <xacro:property name="imu_m" value="0.1" />  <!-- mass /kg -->
+    <xacro:property name="imu_m" value="0.001" />  <!-- mass /kg -->
     <xacro:property name="imu_w" value="0.01" />  <!-- width /m -->
     <xacro:property name="imu_l" value="0.01" />  <!-- length /m -->

File: ros_ws/src/pipe_swarm/urdf/lidar.xacro (robot description, xacro)
@@ -1,5 +1,5 @@
 <?xml version="1.0"?>
 <robot name="lidar" xmlns:xacro="http://www.ros.org/wiki/xacro">
-    <xacro:property name="lidar_m" value="0.1" />  <!-- mass /kg -->
+    <xacro:property name="lidar_m" value="0.001" />  <!-- mass /kg -->
     <xacro:property name="lidar_w" value="0.01" />  <!-- width /m -->
     <xacro:property name="lidar_l" value="0.01" />  <!-- length /m -->

File: ros_ws/src/pipe_swarm/urdf/linkage.xacro (robot description, xacro)
@@ -1,5 +1,5 @@
 <?xml version="1.0"?>
 <robot name="linkage" xmlns:xacro="http://www.ros.org/wiki/xacro">
-    <xacro:property name="cover_m" value="0.1" />  <!-- mass /kg -->
+    <xacro:property name="cover_m" value="0.02" />  <!-- mass /kg -->
     <xacro:property name="cover_w" value="0.029" />  <!-- width /m -->
     <xacro:property name="cover_h" value="0.024" />  <!-- height /m -->
@@ -7,15 +7,15 @@
     <xacro:property name="cover_o" value="0.0045" />  <!-- offset /m -->
     <xacro:property name="cover_out" value="0.0015" />  <!-- extruded cover /m -->
-    <xacro:property name="male_m" value="0.1" />  <!-- mass /kg -->
+    <xacro:property name="male_m" value="0.0065" />  <!-- mass /kg -->
     <xacro:property name="male_w" value="0.014" />  <!-- width /m -->
     <xacro:property name="male_h" value="0.0128" />  <!-- length /m -->
     <xacro:property name="male_l" value="0.0054" />  <!-- height /m -->
     <xacro:property name="male_o" value="0.007" />  <!-- offset /m -->
-    <xacro:property name="pivot_m" value="0.1" />  <!-- mass /kg -->
+    <xacro:property name="pivot_m" value="0.014" />  <!-- mass /kg -->
     <xacro:property name="pivot_w" value="0.035" />  <!-- width /m -->
     <xacro:property name="pivot_h" value="0.024" />  <!-- height /m -->
     <xacro:property name="pivot_l" value="0.055" />   <!-- length /m -->
     <xacro:property name="pivot_o" value="0.0075" />  <!-- offset /m -->
-    <xacro:property name="female_m" value="0.1" />  <!-- mass /kg -->
+    <xacro:property name="female_m" value="0.00825" />  <!-- mass /kg -->
     <xacro:property name="female_w" value="0.02" />  <!-- width /m -->
     <xacro:property name="female_h" value="0.024" />  <!-- height /m -->

File: ros_ws/src/pipe_swarm/urdf/mobile_base.xacro (robot description, xacro)
@@ -1,5 +1,5 @@
 <?xml version="1.0" ?>
 <robot name="mobile_base" xmlns:xacro="http://www.ros.org/wiki/xacro">
-    <xacro:property name="base_m" value="1" />  <!-- mass /kg -->
+    <xacro:property name="base_m" value="0.25" />  <!-- mass /kg -->
     <xacro:property name="base_w" value="0.1045" />  <!-- width /m -->
     <xacro:property name="base_w_offset" value="0.05" />  <!-- offset /m -->

File: ros_ws/src/pipe_swarm/urdf/tof.xacro (robot description, xacro)
@@ -1,5 +1,5 @@
 <?xml version="1.0"?>
 <robot name="tof" xmlns:xacro="http://www.ros.org/wiki/xacro">
-    <xacro:property name="tof_m" value="0.1" />  <!-- mass /kg -->
+    <xacro:property name="tof_m" value="0.001" />  <!-- mass /kg -->
     <xacro:property name="tof_w" value="0.01" />  <!-- width /m -->
     <xacro:property name="tof_l" value="0.01" />  <!-- length /m -->

File: ros_ws/src/pipe_swarm/urdf/tof_lidar.xacro (robot description, xacro)
@@ -1,5 +1,5 @@
 <?xml version="1.0"?>
 <robot name="tof_lidar" xmlns:xacro="http://www.ros.org/wiki/xacro">
-    <xacro:property name="tof_lidar_m" value="0.1" />  <!-- mass /kg -->
+    <xacro:property name="tof_lidar_m" value="0.001" />  <!-- mass /kg -->
     <xacro:property name="tof_lidar_w" value="0.01" />  <!-- width /m -->
     <xacro:property name="tof_lidar_l" value="0.01" />  <!-- length /m -->

File: ros_ws/src/pipe_swarm/urdf/wheels.xacro (robot description, xacro)
@@ -1,5 +1,5 @@
 <?xml version="1.0"?>
 <robot name="wheels" xmlns:xacro="http://www.ros.org/wiki/xacro">
-    <xacro:property name="wheel_m" value="0.1" />  <!-- mass /kg -->
+    <xacro:property name="wheel_m" value="0.005" />  <!-- mass /kg -->
     <xacro:property name="wheel_r" value="0.015" />  <!-- radius /m -->
     <xacro:property name="wheel_l" value="0.008" />  <!-- length /m 8 or 3 -->
