Commit message: adding modularity between gazebo and modular robot

File: ros_ws/src/pipe_swarm/urdf/gazebo/linkage.xacro (robot description, xacro)
@@ -8,5 +8,5 @@
         <material>Gazebo/White</material>
     </gazebo>
-    <gazebo>
+    <!-- <gazebo>
         <plugin name="${agent_namespace}_control" filename="libgazebo_ros2_control.so">
             <robot_param_node>/${agent_namespace}/robot_state_publisher</robot_param_node>
@@ -16,11 +16,11 @@
             </ros>
         </plugin>
-    </gazebo>
+    </gazebo> -->
     <!-- ros2_control Plugin -->
-    <ros2_control name="GazeboSystem" type="system">
+    <!-- <ros2_control name="GazeboSystem" type="system">
         <hardware>
             <plugin>gazebo_ros2_control/GazeboSystem</plugin>
         </hardware>
-        <joint name="base_female_joint">
+        <joint name="${agent_namespace}_base_female_joint">
             <command_interface name="position">
                 <param name="min">-pi/2</param>
@@ -33,4 +33,4 @@
             <state_interface name="effort"/>
         </joint>
-    </ros2_control>
+    </ros2_control> -->
 </robot>

File: ros_ws/src/pipe_swarm/urdf/gazebo/pipe_robot.xacro (robot description, xacro)
@@ -7,6 +7,6 @@
         <xacro:include filename="tof.xacro"/>
         <xacro:include filename="camera.xacro"/>
+        <xacro:include filename="linkage.xacro"/>
         <xacro:include filename="wheels.xacro"/>
-        <xacro:include filename="linkage.xacro"/>
     </xacro:macro>
     <xacro:gazebo_pipe_robot namespace="${agent_namespace}" />

File: ros_ws/src/pipe_swarm/urdf/gazebo/wheels.xacro (robot description, xacro)
@@ -8,6 +8,6 @@
             </ros>
             <update_rate>50</update_rate>
-            <right_joint>base_wheel_back_right_joint</right_joint>
-            <left_joint>base_wheel_back_left_joint</left_joint>
+            <right_joint>${agent_namespace}_base_wheel_back_right_joint</right_joint>
+            <left_joint>${agent_namespace}_base_wheel_back_left_joint</left_joint>
             <wheel_separation>${base_l + wheel_l}</wheel_separation>
             <wheel_diameter>${wheel_r*2}</wheel_diameter>
@@ -16,5 +16,5 @@
             <command_topic>cmd_vel</command_topic>
             <odometry_frame>odom</odometry_frame>
-            <robot_base_frame>${agent_namespace}_footprint_link</robot_base_frame>
+            <robot_base_frame>${base_agent}_footprint</robot_base_frame>
             <odometry_topic>odom</odometry_topic>
             <publish_odom>true</publish_odom>
@@ -29,6 +29,6 @@
             </ros>
             <update_rate>50</update_rate>
-            <right_joint>base_wheel_front_right_joint</right_joint>
-            <left_joint>base_wheel_front_left_joint</left_joint>
+            <right_joint>${agent_namespace}_base_wheel_front_right_joint</right_joint>
+            <left_joint>${agent_namespace}_base_wheel_front_left_joint</left_joint>
             <wheel_separation>${base_l + wheel_l}</wheel_separation>
             <wheel_diameter>${wheel_r*2}</wheel_diameter>
@@ -37,5 +37,5 @@
             <command_topic>cmd_vel</command_topic>
             <odometry_frame>odom</odometry_frame>
-            <robot_base_frame>${agent_namespace}_footprint_link</robot_base_frame>
+            <robot_base_frame>${base_agent}_footprint</robot_base_frame>
             <odometry_topic>odom</odometry_topic>
             <publish_odom>true</publish_odom>

File: ros_ws/src/pipe_swarm/urdf/linkage.xacro (robot description, xacro)
@@ -117,10 +117,15 @@
         <child link="${agent_namespace}_male_link"/>
     </joint>
-    <joint name="base_female_joint" type="revolute">
-        <origin xyz="${-(base_w*0.5) + female_diameter/2} 0 0" rpy="0 0 0"/>
-        <parent link="${agent_namespace}_base_link"/>
-        <child link="${agent_namespace}_female_link"/>
-        <axis xyz="0 1 0"/>
-        <limit lower="${-pi/2}" upper="${pi/2}" effort="1.0" velocity="1.0"/>
+    <joint name="${agent_namespace}_female_footprint_joint" type="fixed">
+        <origin xyz="0 0 0" rpy="0 0 0"/>
+        <parent link="${agent_namespace}_female_link"/>
+        <child link="${agent_namespace}_footprint_link"/>
+        <!-- <axis xyz="0 1 0"/>
+        <limit lower="${-pi/2}" upper="${pi/2}" effort="1.0" velocity="1.0"/> -->
+    </joint>
+    <joint name="${agent_namespace}_footprint_base_joint" type="fixed">
+        <origin xyz="${(base_w*0.5) - female_diameter/2} 0 0" rpy="0 0 0"/>
+        <parent link="${agent_namespace}_footprint_link"/>
+        <child link="${agent_namespace}_base_link"/>
     </joint>
 </robot>

File: ros_ws/src/pipe_swarm/urdf/mobile_base.xacro (robot description, xacro)
@@ -25,8 +25,8 @@
     </link>
     <!-- JOINTS -->
-    <joint name="${agent_namespace}_base_footprint" type="fixed">
+    <!-- <joint name="${agent_namespace}_base_footprint" type="fixed">
         <origin xyz="0 0 0.035" rpy="0 0 0"/>
         <parent link="${agent_namespace}_footprint_link"/>
         <child link="${agent_namespace}_base_link"/>
-    </joint>
+    </joint> -->
 </robot>

File: ros_ws/src/pipe_swarm/urdf/pipe_agent.urdf.xacro (robot description, xacro)
@@ -5,4 +5,9 @@
     <xacro:include filename="pipe_robot.xacro"/>
     <!-- Call pipe_robot with agent_namespace -->
-    <xacro:pipe_robot namespace="${agent_namespace}" include_gazebo="true"/>
+    <xacro:pipe_robot namespace="${agent_namespace}" base_agent="${agent_namespace}" include_gazebo="true"/>
+    <link name="${agent_namespace}_footprint" />
+    <joint name="${agent_namespace}_footprint_joint" type="fixed">
+        <parent link="${agent_namespace}_footprint"/>
+        <child link="${agent_namespace}_female_link"/>
+    </joint>
 </robot>

File: ros_ws/src/pipe_swarm/urdf/pipe_robot.xacro (robot description, xacro)
@@ -1,5 +1,5 @@
 <?xml version="1.0"?>
 <robot name="pipe_robot" xmlns:xacro="http://www.ros.org/wiki/xacro">
-    <xacro:macro name="pipe_robot" params="namespace include_gazebo">
+    <xacro:macro name="pipe_robot" params="namespace base_agent include_gazebo">
         <xacro:property name="agent_namespace" value="${namespace}" />
         <!-- Include shared components -->
@@ -9,6 +9,6 @@
         <xacro:include filename="tof.xacro"/>
         <xacro:include filename="camera.xacro"/>
+        <xacro:include filename="linkage.xacro"/>
         <xacro:include filename="wheels.xacro"/>
-        <xacro:include filename="linkage.xacro"/>
         <xacro:if value="${include_gazebo}">
             <xacro:include filename="gazebo/pipe_robot.xacro"/>

File: ros_ws/src/pipe_swarm/urdf/wheels.xacro (robot description, xacro)
@@ -30,5 +30,5 @@
     <xacro:wheel_link prefix="back_left" />
     <!-- JOINTS -->
-    <joint name="base_wheel_front_right_joint" type="continuous">
+    <joint name="${agent_namespace}_base_wheel_front_right_joint" type="continuous">
         <origin xyz="${(base_w)/2 - wheel_r} ${-((base_l/2) + (wheel_l/2))} ${-base_h/2}" rpy="${-pi/2} 0 0"/>
         <parent link="${agent_namespace}_base_link"/>
@@ -36,5 +36,5 @@
         <axis xyz="0 0 1"/>
     </joint>
-    <joint name="base_wheel_front_left_joint" type="continuous">
+    <joint name="${agent_namespace}_base_wheel_front_left_joint" type="continuous">
         <origin xyz="${(base_w)/2 - wheel_r} ${(base_l/2) + (wheel_l/2)} ${-base_h/2}" rpy="${-pi/2} 0 0"/>
         <parent link="${agent_namespace}_base_link"/>
@@ -42,17 +42,17 @@
         <axis xyz="0 0 1"/>
     </joint>
-    <joint name="base_wheel_back_right_joint" type="continuous">
+    <joint name="${agent_namespace}_base_wheel_back_right_joint" type="continuous">
         <origin xyz="${-((base_w)/2 - wheel_r)} ${-((base_l/2) + (wheel_l/2))} ${-base_h/2}" rpy="${-pi/2} 0 0"/>
         <parent link="${agent_namespace}_base_link"/>
         <child link="${agent_namespace}_wheel_back_right_link"/>
         <axis xyz="0 0 1"/>
-        <!-- <mimic joint="base_wheel_front_right_joint" multiplier="1.0"/> -->
+        <!-- <mimic joint="${agent_namespace}_base_wheel_front_right_joint" multiplier="1.0"/> -->
     </joint>
-    <joint name="base_wheel_back_left_joint" type="continuous">
+    <joint name="${agent_namespace}_base_wheel_back_left_joint" type="continuous">
         <origin xyz="${-((base_w)/2 - wheel_r)} ${(base_l/2) + (wheel_l/2)} ${-base_h/2}" rpy="${-pi/2} 0 0"/>
         <parent link="${agent_namespace}_base_link"/>
         <child link="${agent_namespace}_wheel_back_left_link"/>
         <axis xyz="0 0 1"/>
-        <!-- <mimic joint="base_wheel_front_left_joint" multiplier="1.0"/> -->
+        <!-- <mimic joint="${agent_namespace}_base_wheel_front_left_joint" multiplier="1.0"/> -->
     </joint>
 </robot>

Commit message: reverting tf tree to original

File: ros_ws/src/pipe_swarm/urdf/gazebo/linkage.xacro (robot description, xacro)
@@ -8,5 +8,5 @@
         <material>Gazebo/White</material>
     </gazebo>
-    <!-- <gazebo>
+    <gazebo>
         <plugin name="${agent_namespace}_control" filename="libgazebo_ros2_control.so">
             <robot_param_node>/${agent_namespace}/robot_state_publisher</robot_param_node>
@@ -16,11 +16,11 @@
             </ros>
         </plugin>
-    </gazebo> -->
+    </gazebo>
     <!-- ros2_control Plugin -->
-    <!-- <ros2_control name="GazeboSystem" type="system">
+    <ros2_control name="GazeboSystem" type="system">
         <hardware>
             <plugin>gazebo_ros2_control/GazeboSystem</plugin>
         </hardware>
-        <joint name="${agent_namespace}_base_female_joint">
+        <joint name="base_female_joint">
             <command_interface name="position">
                 <param name="min">-pi/2</param>
@@ -33,4 +33,4 @@
             <state_interface name="effort"/>
         </joint>
-    </ros2_control> -->
+    </ros2_control>
 </robot>

File: ros_ws/src/pipe_swarm/urdf/gazebo/wheels.xacro (robot description, xacro)
@@ -16,5 +16,5 @@
             <command_topic>cmd_vel</command_topic>
             <odometry_frame>odom</odometry_frame>
-            <robot_base_frame>${base_agent}_footprint</robot_base_frame>
+            <robot_base_frame>${base_agent}_footprint_link</robot_base_frame>
             <odometry_topic>odom</odometry_topic>
             <publish_odom>true</publish_odom>
@@ -37,5 +37,5 @@
             <command_topic>cmd_vel</command_topic>
             <odometry_frame>odom</odometry_frame>
-            <robot_base_frame>${base_agent}_footprint</robot_base_frame>
+            <robot_base_frame>${base_agent}_footprint_link</robot_base_frame>
             <odometry_topic>odom</odometry_topic>
             <publish_odom>true</publish_odom>

File: ros_ws/src/pipe_swarm/urdf/linkage.xacro (robot description, xacro)
@@ -117,15 +117,15 @@
         <child link="${agent_namespace}_male_link"/>
     </joint>
-    <joint name="${agent_namespace}_female_footprint_joint" type="fixed">
-        <origin xyz="0 0 0" rpy="0 0 0"/>
-        <parent link="${agent_namespace}_female_link"/>
-        <child link="${agent_namespace}_footprint_link"/>
-        <!-- <axis xyz="0 1 0"/>
-        <limit lower="${-pi/2}" upper="${pi/2}" effort="1.0" velocity="1.0"/> -->
+    <joint name="base_female_joint" type="revolute">
+        <origin xyz="${-(base_w*0.5) + female_diameter/2} 0 0" rpy="0 0 0"/>
+        <parent link="${agent_namespace}_base_link"/>
+        <child link="${agent_namespace}_female_link"/>
+        <axis xyz="0 1 0"/>
+        <limit lower="${-pi/2}" upper="${pi/2}" effort="1.0" velocity="1.0"/>
     </joint>
-    <joint name="${agent_namespace}_footprint_base_joint" type="fixed">
+    <!-- <joint name="${agent_namespace}_footprint_base_joint" type="fixed">
         <origin xyz="${(base_w*0.5) - female_diameter/2} 0 0" rpy="0 0 0"/>
         <parent link="${agent_namespace}_footprint_link"/>
         <child link="${agent_namespace}_base_link"/>
-    </joint>
+    </joint> -->
 </robot>

File: ros_ws/src/pipe_swarm/urdf/mobile_base.xacro (robot description, xacro)
@@ -25,8 +25,8 @@
     </link>
     <!-- JOINTS -->
-    <!-- <joint name="${agent_namespace}_base_footprint" type="fixed">
+    <joint name="${agent_namespace}_base_footprint" type="fixed">
         <origin xyz="0 0 0.035" rpy="0 0 0"/>
         <parent link="${agent_namespace}_footprint_link"/>
         <child link="${agent_namespace}_base_link"/>
-    </joint> -->
+    </joint>
 </robot>

File: ros_ws/src/pipe_swarm/urdf/pipe_agent.urdf.xacro (robot description, xacro)
@@ -6,8 +6,9 @@
     <!-- Call pipe_robot with agent_namespace -->
     <xacro:pipe_robot namespace="${agent_namespace}" base_agent="${agent_namespace}" include_gazebo="true"/>
-    <link name="${agent_namespace}_footprint" />
+    <!-- <link name="${agent_namespace}_footprint" /> -->
+<!--
     <joint name="${agent_namespace}_footprint_joint" type="fixed">
         <parent link="${agent_namespace}_footprint"/>
         <child link="${agent_namespace}_female_link"/>
-    </joint>
+    </joint> -->
 </robot>
