Commit message: isolating imu sensor

File: ros_ws/src/pipe_swarm/urdf/gazebo/pipe_robot.xacro (robot description, xacro)
@@ -4,5 +4,6 @@
         <!-- Include shared components -->
         <xacro:include filename="mobile_base.xacro"/>
-        <xacro:include filename="lidar.xacro"/>
+        <!-- <xacro:include filename="lidar.xacro"/> -->
+        <xacro:include filename="imu.xacro"/>
         <xacro:include filename="tof.xacro"/>
         <xacro:include filename="camera.xacro"/>

File: ros_ws/src/pipe_swarm/urdf/imu.xacro (robot description, xacro)
@@ -29,25 +29,3 @@
         <child link="${agent_namespace}_imu_link"/>
     </joint>
-    <!-- GAZEBO -->
-    <gazebo reference="${agent_namespace}_imu_link">
-        <material>Gazebo/Red</material>
-        <sensor name="${agent_namespace}_imu_sensor" type="imu">
-            <always_on>true</always_on>
-            <visualize>true</visualize>
-            <update_rate>100</update_rate>
-            <topic>__default_topic__</topic>
-            <plugin name="imu" filename="libgazebo_ros_imu_sensor.so">
-                <topicName>imu</topicName>
-                <serviceName>imu_service</serviceName>
-                <bodyName>${agent_namespace}_imu_link</bodyName>
-                <updateRateHZ>10.0</updateRateHZ>
-                <gaussianNoise>0.0</gaussianNoise>
-                <xyzOffset>0 0 0</xyzOffset>
-                <rpyOffset>0 0 0</rpyOffset>
-                <frameName>${agent_namespace}_imu_link</frameName>
-                <initialOrientationAsReference>false</initialOrientationAsReference>
-            </plugin>
-            <pose>0 0 0 0 0 0</pose>
-        </sensor>
-    </gazebo>
 </robot>

File: ros_ws/src/pipe_swarm/urdf/pipe_robot.xacro (robot description, xacro)
@@ -6,5 +6,6 @@
         <xacro:include filename="common.xacro"/>
         <xacro:include filename="mobile_base.xacro"/>
-        <xacro:include filename="lidar.xacro"/>
+        <!-- <xacro:include filename="lidar.xacro"/> -->
+        <xacro:include filename="imu.xacro"/>
         <xacro:include filename="tof.xacro"/>
         <xacro:include filename="camera.xacro"/>

Commit message: adding tof_lidar plugin

File: ros_ws/src/pipe_swarm/urdf/gazebo/pipe_robot.xacro (robot description, xacro)
@@ -6,4 +6,5 @@
         <!-- <xacro:include filename="lidar.xacro"/> -->
         <xacro:include filename="imu.xacro"/>
+        <xacro:include filename="tof_lidar.xacro"/>
         <xacro:include filename="tof.xacro"/>
         <xacro:include filename="camera.xacro"/>

File: ros_ws/src/pipe_swarm/urdf/pipe_robot.xacro (robot description, xacro)
@@ -8,4 +8,5 @@
         <!-- <xacro:include filename="lidar.xacro"/> -->
         <xacro:include filename="imu.xacro"/>
+        <xacro:include filename="tof_lidar.xacro"/>
         <xacro:include filename="tof.xacro"/>
         <xacro:include filename="camera.xacro"/>

File: ros_ws/src/pipe_swarm/urdf/tof_lidar.xacro (robot description, xacro)
@@ -29,34 +29,3 @@
         <child link="${agent_namespace}_lidar_link"/>
     </joint>
-    <!-- GAZEBO -->
-    <gazebo reference="${agent_namespace}_lidar_link">
-        <material>Gazebo/Green</material>
-        <sensor name="lidar_sensor" type="lidar">
-            <pose>0 0 0 0 0 0</pose>
-            <visualize>true</visualize>
-            <update_rate>10.0</update_rate>
-            <ray>
-                <scan>
-                    <horizontal>
-                        <samples>3</samples>
-                        <min_angle>${pi/6}</min_angle>
-                        <max_angle>${-pi/6}</max_angle>
-                    </horizontal>
-                </scan>
-                <range>
-                    <min>0.1</min>
-                    <max>1</max>
-                </range>
-            </ray>
-            <plugin name="lidar_controller" filename="libgazebo_ros_ray_sensor.so">
-                <ros>
-                    <namespace>${agent_namespace}</namespace>
-                    <remapping>~/out:=laserscan</remapping>
-                </ros>
-                <output_type>sensor_msgs/LaserScan</output_type>
-                <min_intensity>100.0</min_intensity>
-                <frame_name>${agent_namespace}_lidar_link</frame_name>
-            </plugin>
-        </sensor>
-    </gazebo>
 </robot>
