Commit message: renaming tof_lidar link

File: ros_ws/src/pipe_swarm/urdf/gazebo/tof_lidar.xacro (robot description, xacro)
@@ -2,7 +2,7 @@
 <robot name="gazebo_tof_lidar" xmlns:xacro="http://www.ros.org/wiki/xacro">
     <!-- GAZEBO -->
-    <gazebo reference="${agent_namespace}_lidar_link">
+    <gazebo reference="${agent_namespace}_tof_lidar_link">
         <material>Gazebo/Green</material>
-        <sensor name="${agent_namespace}_lidar_sensor" type="lidar">
+        <sensor name="${agent_namespace}_tof_lidar_sensor" type="lidar">
             <pose>0 0 0 0 0 0</pose>
             <visualize>true</visualize>
@@ -21,5 +21,5 @@
                 </range>
             </ray>
-            <plugin name="${agent_namespace}_lidar_controller" filename="libgazebo_ros_ray_sensor.so">
+            <plugin name="${agent_namespace}_tof_lidar_controller" filename="libgazebo_ros_ray_sensor.so">
                 <ros>
                     <namespace>${agent_namespace}</namespace>
@@ -28,5 +28,5 @@
                 <output_type>sensor_msgs/LaserScan</output_type>
                 <min_intensity>100.0</min_intensity>
-                <frame_name>${agent_namespace}_lidar_link</frame_name>
+                <frame_name>${agent_namespace}_tof_lidar_link</frame_name>
             </plugin>
         </sensor>

File: ros_ws/src/pipe_swarm/urdf/tof_lidar.xacro (robot description, xacro)
@@ -1,14 +1,14 @@
 <?xml version="1.0"?>
 <robot name="tof_lidar" xmlns:xacro="http://www.ros.org/wiki/xacro">
-    <xacro:property name="lidar_m" value="0.1" />  <!-- mass /kg -->
-    <xacro:property name="lidar_w" value="0.01" />  <!-- width /m -->
-    <xacro:property name="lidar_l" value="0.01" />  <!-- length /m -->
-    <xacro:property name="lidar_h" value="0.01" />  <!-- height /m -->
+    <xacro:property name="tof_lidar_m" value="0.1" />  <!-- mass /kg -->
+    <xacro:property name="tof_lidar_w" value="0.01" />  <!-- width /m -->
+    <xacro:property name="tof_lidar_l" value="0.01" />  <!-- length /m -->
+    <xacro:property name="tof_lidar_h" value="0.01" />  <!-- height /m -->
     <!-- LINKS -->
-    <link name="${agent_namespace}_lidar_link">
+    <link name="${agent_namespace}_tof_lidar_link">
         <visual>
             <origin xyz="0.0 0.0 0.0" rpy="0.0 0.0 0.0"/>
             <geometry>
-                <box size="${lidar_w} ${lidar_l} ${lidar_h}"/>
+                <box size="${tof_lidar_w} ${tof_lidar_l} ${tof_lidar_h}"/>
             </geometry>
             <material name="red">
@@ -18,14 +18,14 @@
         <collision>
             <geometry>
-                <box size="${lidar_w} ${lidar_l} ${lidar_h}"/>
+                <box size="${tof_lidar_w} ${tof_lidar_l} ${tof_lidar_h}"/>
             </geometry>
         </collision>
-        <xacro:box_inertial m="${lidar_m}" w="${lidar_w}" l="${lidar_l}" h="${lidar_h}" xyz="0 0 0 " rpy="0 0 0"/>
+        <xacro:box_inertial m="${tof_lidar_m}" w="${tof_lidar_w}" l="${tof_lidar_l}" h="${tof_lidar_h}" xyz="0 0 0 " rpy="0 0 0"/>
     </link>
     <!-- JOINTS -->
-    <joint name="${agent_namespace}_base_lidar_joint" type="fixed">
-        <origin xyz="${(base_w*0.5)} ${-(base_l*0.5 - lidar_l*0.5)} ${(base_h*0.5)}" rpy="${pi/2} 0 0"/>
+    <joint name="${agent_namespace}_base_tof_lidar_joint" type="fixed">
+        <origin xyz="${(base_w*0.5)} ${-(base_l*0.5 - tof_lidar_l*0.5)} ${(base_h*0.5)}" rpy="${pi/2} 0 0"/>
         <parent link="${agent_namespace}_base_link"/>
-        <child link="${agent_namespace}_lidar_link"/>
+        <child link="${agent_namespace}_tof_lidar_link"/>
     </joint>
 </robot>
