Commit message: wheel update

File: ros_ws/src/pipe_swarm/urdf/gazebo/wheels.xacro (robot description, xacro)
@@ -92,21 +92,21 @@
     <gazebo reference="${agent_namespace}_wheel_front_right_link">
         <material>Gazebo/Black</material>
-        <mu1 value="1.0"/>
-        <mu2 value="1.0"/>
+        <mu1 value="2.0"/>
+        <mu2 value="2.0"/>
     </gazebo>
     <gazebo reference="${agent_namespace}_wheel_front_left_link">
         <material>Gazebo/Black</material>
-        <mu1 value="1.0"/>
-        <mu2 value="1.0"/>
+        <mu1 value="2.0"/>
+        <mu2 value="2.0"/>
     </gazebo>
     <gazebo reference="${agent_namespace}_wheel_back_right_link">
         <material>Gazebo/Black</material>
-        <mu1 value="1.0"/>
-        <mu2 value="1.0"/>
+        <mu1 value="2.0"/>
+        <mu2 value="2.0"/>
     </gazebo>
     <gazebo reference="${agent_namespace}_wheel_back_left_link">
         <material>Gazebo/Black</material>
-        <mu1 value="1.0"/>
-        <mu2 value="1.0"/>
+        <mu1 value="2.0"/>
+        <mu2 value="2.0"/>
     </gazebo>
 </robot>

File: ros_ws/src/pipe_swarm/urdf/wheels.xacro (robot description, xacro)
@@ -10,8 +10,8 @@
         <link name="${agent_namespace}_wheel_${prefix}_left_link">
             <visual>
-                <origin xyz="${-wheel_r} ${-wheel_r} ${-wheel_l/2}" rpy="0 0 0"/>
+                <origin xyz="0 0 0" rpy="0 0 0"/>
                 <geometry>
-                    <mesh filename="package://pipe_swarm/models/hollow_pipe/meshes/wheel.stl" scale="0.001 0.001 0.001"/>
-                    <!-- <cylinder radius="${wheel_r}" length="${wheel_l}"/> -->
+                    <!-- <mesh filename="package://pipe_swarm/models/hollow_pipe/meshes/wheel.stl" scale="0.001 0.001 0.001"/> -->
+                    <cylinder radius="${wheel_r}" length="${wheel_l}"/>
                 </geometry>
                 <material name="wheel">
@@ -20,8 +20,8 @@
             </visual>
             <collision>
-                <origin xyz="${-wheel_r} ${-wheel_r} ${-wheel_l/2}" rpy="0 0 0"/>
+                <origin xyz="0 0 0 " rpy="0 0 0"/>
                 <geometry>
-                    <mesh filename="package://pipe_swarm/models/hollow_pipe/meshes/wheel.stl" scale="0.001 0.001 0.001"/>
-                    <!-- <cylinder radius="${wheel_r}" length="${wheel_l}"/> -->
+                    <!-- <mesh filename="package://pipe_swarm/models/hollow_pipe/meshes/wheel.stl" scale="0.001 0.001 0.001"/> -->
+                    <cylinder radius="${wheel_r}" length="${wheel_l}"/>
                 </geometry>
             </collision>
@@ -30,8 +30,8 @@
         <link name="${agent_namespace}_wheel_${prefix}_right_link">
             <visual>
-                <origin xyz="${-wheel_r} ${-wheel_r} ${-wheel_l/2}" rpy="0 0 0"/>
+                <origin xyz="0 0 0" rpy="0 0 0"/>
                 <geometry>
-                    <mesh filename="package://pipe_swarm/models/hollow_pipe/meshes/wheel.stl" scale="0.001 0.001 0.001"/>
-                    <!-- <cylinder radius="${wheel_r}" length="${wheel_l}"/> -->
+                    <!-- <mesh filename="package://pipe_swarm/models/hollow_pipe/meshes/wheel.stl" scale="0.001 0.001 0.001"/> -->
+                    <cylinder radius="${wheel_r}" length="${wheel_l}"/>
                 </geometry>
                 <material name="wheel">
@@ -40,8 +40,8 @@
             </visual>
             <collision>
-                <origin xyz="${-wheel_r} ${-wheel_r} ${-wheel_l/2}" rpy="0 0 0"/>
+                <origin xyz="0 0 0" rpy="0 0 0"/>
                 <geometry>
-                    <mesh filename="package://pipe_swarm/models/hollow_pipe/meshes/wheel.stl" scale="0.001 0.001 0.001"/>
-                    <!-- <cylinder radius="${wheel_r}" length="${wheel_l}"/> -->
+                    <!-- <mesh filename="package://pipe_swarm/models/hollow_pipe/meshes/wheel.stl" scale="0.001 0.001 0.001"/> -->
+                    <cylinder radius="${wheel_r}" length="${wheel_l}"/>
                 </geometry>
             </collision>
@@ -54,28 +54,32 @@
     <!-- JOINTS -->
     <joint name="${agent_namespace}_base_wheel_front_right_joint" type="continuous">
-        <origin xyz="${(base_w)/2 - wheel_x_offset_front} ${-((base_l/2) + (wheel_l/2) + wheel_y_offset)} ${-base_h/2}" rpy="${-pi/2} 0 0"/>
+        <origin xyz="${(base_w)/2 - wheel_x_offset_front} ${-((base_l/2) + (wheel_l/2) + wheel_y_offset)} ${-base_h/2}" rpy="${-pi/2- 0.1745} 0 0"/>
         <parent link="${agent_namespace}_base_link"/>
         <child link="${agent_namespace}_wheel_front_right_link"/>
         <axis xyz="0 0 1"/>
+        <dynamics damping="0.8"/>
     </joint>
     <joint name="${agent_namespace}_base_wheel_front_left_joint" type="continuous">
-        <origin xyz="${(base_w)/2 - wheel_x_offset_front} ${(base_l/2) + (wheel_l/2) + wheel_y_offset} ${-base_h/2}" rpy="${pi/2} 0 0"/>
+        <origin xyz="${(base_w)/2 - wheel_x_offset_front} ${(base_l/2) + (wheel_l/2) + wheel_y_offset} ${-base_h/2}" rpy="${pi/2+ 0.1745} 0 0"/>
         <parent link="${agent_namespace}_base_link"/>
         <child link="${agent_namespace}_wheel_front_left_link"/>
         <axis xyz="0 0 -1"/>
+        <dynamics damping="0.8"/>
     </joint>
     <joint name="${agent_namespace}_base_wheel_back_right_joint" type="continuous">
-        <origin xyz="${-((base_w)/2 - wheel_x_offset_back)} ${-((base_l/2) + (wheel_l/2) + wheel_y_offset)} ${-base_h/2}" rpy="${-pi/2} 0 0"/>
+        <origin xyz="${-((base_w)/2 - wheel_x_offset_back)} ${-((base_l/2) + (wheel_l/2) + wheel_y_offset)} ${-base_h/2}" rpy="${-pi/2- 0.1745} 0 0"/>
         <parent link="${agent_namespace}_base_link"/>
         <child link="${agent_namespace}_wheel_back_right_link"/>
         <axis xyz="0 0 1"/>
         <!-- <mimic joint="${agent_namespace}_base_wheel_front_right_joint" multiplier="1.0"/> -->
+        <dynamics damping="0.8"/>
     </joint>
     <joint name="${agent_namespace}_base_wheel_back_left_joint" type="continuous">
-        <origin xyz="${-((base_w)/2 - wheel_x_offset_back)} ${(base_l/2) + (wheel_l/2) + wheel_y_offset} ${-base_h/2}" rpy="${pi/2} 0 0"/>
+        <origin xyz="${-((base_w)/2 - wheel_x_offset_back)} ${(base_l/2) + (wheel_l/2) + wheel_y_offset} ${-base_h/2}" rpy="${pi/2+ 0.1745} 0 0"/>
         <parent link="${agent_namespace}_base_link"/>
         <child link="${agent_namespace}_wheel_back_left_link"/>
         <axis xyz="0 0 -1"/>
         <!-- <mimic joint="${agent_namespace}_base_wheel_front_left_joint" multiplier="1.0"/> -->
+        <dynamics damping="0.8"/>
     </joint>
 </robot>
