Commit message: making female link parent of base link

File: ros_ws/src/modular_robot/urdf/gazebo/linkage.xacro (robot description, xacro)
@@ -19,5 +19,5 @@
             <plugin>gazebo_ros2_control/GazeboSystem</plugin>
         </hardware>
-        <joint name="base_female_joint">
+        <joint name="female_base_joint">
             <command_interface name="position">
                 <param name="min">-pi/2</param>
@@ -31,3 +31,16 @@
         </joint>
     </ros2_control>
+    <!-- <gazebo>
+        <plugin name="joint_state_publisher" filename="libgazebo_ros_joint_state_publisher.so">
+            <ros>
+                <namespace>${agent_namespace}</namespace>
+            </ros>
+            <update_rate>50</update_rate>
+            <joint_name>female_base_joint</joint_name>
+        </plugin>
+    </gazebo>
+    <gazebo>
+        <plugin name="${agent_namespace}_control" filename="libgazebo_ros_control.so">
+        </plugin>
+    </gazebo> -->
 </robot>

File: ros_ws/src/modular_robot/urdf/linkage.xacro (robot description, xacro)
@@ -1,5 +1,5 @@
 <?xml version="1.0"?>
 <robot name="linkage" xmlns:xacro="http://www.ros.org/wiki/xacro">
-    <xacro:property name="male_m" value="0.1" />  <!-- mass /kg -->
+    <xacro:property name="male_m" value="0.3" />  <!-- mass /kg -->
     <xacro:property name="male_w" value="0.04" />  <!-- width /m -->
     <xacro:property name="male_h" value="0.01" />  <!-- height /m -->
@@ -113,14 +113,15 @@
     <!-- JOINTS -->
     <joint name="${agent_namespace}_base_male_joint" type="fixed">
-        <origin xyz="${(base_w*0.5) + (male_w*0.5)} 0 0" rpy="0 0 0"/>
+        <origin xyz="${(base_w - 0.02) + (male_w*0.5) } 0 0" rpy="0 0 0"/>
         <parent link="${agent_namespace}_base_link"/>
         <child link="${agent_namespace}_male_link"/>
     </joint>
-    <joint name="base_female_joint" type="revolute">
-        <origin xyz="${-(base_w*0.5) + female_diameter/2} 0 0" rpy="0 0 0"/>
-        <parent link="${agent_namespace}_base_link"/>
-        <child link="${agent_namespace}_female_link"/>
+    <joint name="female_base_joint" type="revolute">
+        <origin xyz="0 0 0" rpy="0 0 0"/>
+        <parent link="${agent_namespace}_female_link"/>
+        <child link="${agent_namespace}_base_link"/>
         <axis xyz="0 1 0"/>
         <limit lower="${-pi/2}" upper="${pi/2}" effort="1.0" velocity="1.0"/>
+        <dynamics damping="0.3" friction="0.5"/>  <!-- Add damping -->
     </joint>
     <!-- <joint name="${agent_namespace}_footprint_base_joint" type="fixed">

File: ros_ws/src/modular_robot/urdf/mobile_base.xacro (robot description, xacro)
@@ -1,13 +1,13 @@
 <?xml version="1.0" ?>
 <robot name="mobile_base" xmlns:xacro="http://www.ros.org/wiki/xacro">
-    <xacro:property name="base_m" value="1" />  <!-- mass /kg -->
+    <xacro:property name="base_m" value="0.5" />  <!-- mass /kg -->
     <xacro:property name="base_w" value="0.15" />  <!-- width /m -->
     <xacro:property name="base_l" value="0.05" />  <!-- length /m -->
     <xacro:property name="base_h" value="0.045" />  <!-- height /m -->
     <!-- LINKS -->
-    <link name="${agent_namespace}_footprint_link" />
+    <!-- <link name="${agent_namespace}_footprint_link" /> -->
     <link name="${agent_namespace}_base_link">
         <visual>
-            <origin xyz="0.0 0.0 0.0" rpy="0.0 0.0 0.0"/>
+            <origin xyz="${(base_w*0.5) - 0.02} 0.0 0.0" rpy="0.0 0.0 0.0"/>
             <geometry>
                 <box size="${base_w} ${base_l} ${base_h}"/>
@@ -18,4 +18,5 @@
         </visual>
         <collision>
+            <origin xyz="${(base_w*0.5) - 0.02} 0.0 0.0" rpy="0.0 0.0 0.0"/>
             <geometry>
                 <box size="${base_w} ${base_l} ${base_h}"/>
@@ -25,8 +26,8 @@
     </link>
     <!-- JOINTS -->
-    <joint name="${agent_namespace}_base_footprint" type="fixed">
+    <!-- <joint name="${agent_namespace}_base_footprint" type="fixed">
         <origin xyz="0 0 0.035" rpy="0 0 0"/>
         <parent link="${agent_namespace}_footprint_link"/>
         <child link="${agent_namespace}_base_link"/>
-    </joint>
+    </joint> -->
 </robot>

Commit message: isolating ros2 control with hardcoded joints

File: ros_ws/src/modular_robot/urdf/gazebo/linkage.xacro (robot description, xacro)
@@ -8,39 +8,3 @@
         <material>Gazebo/White</material>
     </gazebo>
-    <gazebo>
-        <plugin name="${agent_namespace}_control" filename="libgazebo_ros2_control.so">
-            <robot_param_node>robot_state_publisher</robot_param_node>
-            <parameters>$(find modular_robot)/config/modular_controller.yaml</parameters>
-        </plugin>
-    </gazebo>
-    <!-- ros2_control Plugin -->
-    <ros2_control name="GazeboSystem" type="system">
-        <hardware>
-            <plugin>gazebo_ros2_control/GazeboSystem</plugin>
-        </hardware>
-        <joint name="female_base_joint">
-            <command_interface name="position">
-                <param name="min">-pi/2</param>
-                <param name="max">pi/2</param>
-            </command_interface>
-            <state_interface name="position">
-                <param name="initial_value">0.0</param>
-            </state_interface>
-            <state_interface name="velocity"/>
-            <state_interface name="effort"/>
-        </joint>
-    </ros2_control>
-    <!-- <gazebo>
-        <plugin name="joint_state_publisher" filename="libgazebo_ros_joint_state_publisher.so">
-            <ros>
-                <namespace>${agent_namespace}</namespace>
-            </ros>
-            <update_rate>50</update_rate>
-            <joint_name>female_base_joint</joint_name>
-        </plugin>
-    </gazebo>
-    <gazebo>
-        <plugin name="${agent_namespace}_control" filename="libgazebo_ros_control.so">
-        </plugin>
-    </gazebo> -->
 </robot>

File: ros_ws/src/modular_robot/urdf/linkage.xacro (robot description, xacro)
@@ -117,5 +117,5 @@
         <child link="${agent_namespace}_male_link"/>
     </joint>
-    <joint name="female_base_joint" type="revolute">
+    <joint name="${agent_namespace}_female_base_joint" type="revolute">
         <origin xyz="0 0 0" rpy="0 0 0"/>
         <parent link="${agent_namespace}_female_link"/>

File: ros_ws/src/modular_robot/urdf/modular_robot.urdf.xacro (robot description, xacro)
@@ -5,9 +5,61 @@
     <!-- Call pipe_robot with agent_namespace -->
     <xacro:pipe_robot agent_namespace="agent_n" include_gazebo="true"/>
+    <xacro:pipe_robot agent_namespace="agent_n2" include_gazebo="true"/>
+    <xacro:pipe_robot agent_namespace="agent_n3" include_gazebo="true"/>
     <!-- <link name="${agent_namespace}_footprint" /> -->
-<!--
-    <joint name="${agent_namespace}_footprint_joint" type="fixed">
-        <parent link="${agent_namespace}_footprint"/>
-        <child link="${agent_namespace}_female_link"/>
-    </joint> -->
+    <joint name="agent_n_agent_n2_joint" type="fixed">
+        <origin xyz="${(0.05+0.02)} 0 0" rpy="0 0 0"/>
+        <parent link="agent_n_male_link"/>
+        <child link="agent_n2_female_link"/>
+    </joint>
+    <joint name="agent_n2_agent_n3_joint" type="fixed">
+        <origin xyz="${(0.05+0.02)} 0 0" rpy="0 0 0"/>
+        <parent link="agent_n2_male_link"/>
+        <child link="agent_n3_female_link"/>
+    </joint>
+    <gazebo>
+        <plugin name="ros_control" filename="libgazebo_ros2_control.so">
+            <robot_param_node>robot_state_publisher</robot_param_node>
+            <parameters>$(find modular_robot)/config/modular_controller.yaml</parameters>
+        </plugin>
+    </gazebo>
+    <!-- ros2_control Plugin -->
+    <ros2_control name="GazeboSystem" type="system">
+        <hardware>
+            <plugin>gazebo_ros2_control/GazeboSystem</plugin>
+        </hardware>
+        <joint name="agent_n_female_base_joint">
+            <command_interface name="position">
+                <param name="min">-pi/2</param>
+                <param name="max">pi/2</param>
+            </command_interface>
+            <state_interface name="position">
+                <param name="initial_value">0.0</param>
+            </state_interface>
+            <state_interface name="velocity"/>
+            <state_interface name="effort"/>
+        </joint>
+        <joint name="agent_n2_female_base_joint">
+            <command_interface name="position">
+                <param name="min">-pi/2</param>
+                <param name="max">pi/2</param>
+            </command_interface>
+            <state_interface name="position">
+                <param name="initial_value">0.0</param>
+            </state_interface>
+            <state_interface name="velocity"/>
+            <state_interface name="effort"/>
+        </joint>
+        <joint name="agent_n3_female_base_joint">
+            <command_interface name="position">
+                <param name="min">-pi/2</param>
+                <param name="max">pi/2</param>
+            </command_interface>
+            <state_interface name="position">
+                <param name="initial_value">0.0</param>
+            </state_interface>
+            <state_interface name="velocity"/>
+            <state_interface name="effort"/>
+        </joint>
+    </ros2_control>
 </robot>
