Commit message: adding joint_trajectory_controller

File: ros_ws/src/modular_robot/urdf/mobile_base.xacro (robot description, xacro)
@@ -6,5 +6,4 @@
     <xacro:property name="base_h" value="0.045" />  <!-- height /m -->
     <!-- LINKS -->
-    <!-- <link name="${agent_namespace}_footprint_link" /> -->
     <link name="${agent_namespace}_base_link">
         <visual>

File: ros_ws/src/modular_robot/urdf/modular_robot.urdf.xacro (robot description, xacro)
@@ -3,9 +3,15 @@
     <!-- Correct include syntax -->
     <xacro:include filename="pipe_robot.xacro"/>
+    <link name="footprint_link" />
     <!-- Call pipe_robot with agent_namespace -->
     <xacro:pipe_robot agent_namespace="agent_n" include_gazebo="true"/>
     <xacro:pipe_robot agent_namespace="agent_n2" include_gazebo="true"/>
     <xacro:pipe_robot agent_namespace="agent_n3" include_gazebo="true"/>
-    <!-- <link name="${agent_namespace}_footprint" /> -->
+    <xacro:pipe_robot agent_namespace="agent_n4" include_gazebo="true"/>
+    <joint name="footprint_agent_n2_joint" type="fixed">
+        <origin xyz="0 0 0" rpy="0 0 0"/>
+        <child link="agent_n_female_link"/>
+        <parent link="footprint_link"/>
+    </joint>
     <joint name="agent_n_agent_n2_joint" type="fixed">
         <origin xyz="${(0.05+0.02)} 0 0" rpy="0 0 0"/>
@@ -17,4 +23,9 @@
         <parent link="agent_n2_male_link"/>
         <child link="agent_n3_female_link"/>
+    </joint>
+    <joint name="agent_n3_agent_n4_joint" type="fixed">
+        <origin xyz="${(0.05+0.02)} 0 0" rpy="0 0 0"/>
+        <parent link="agent_n3_male_link"/>
+        <child link="agent_n4_female_link"/>
     </joint>
     <gazebo>
@@ -62,4 +73,15 @@
             <state_interface name="effort"/>
         </joint>
+        <joint name="agent_n4_female_base_joint">
+            <command_interface name="position">
+                <param name="min">-pi/2</param>
+                <param name="max">pi/2</param>
+            </command_interface>
+            <state_interface name="position">
+                <param name="initial_value">0.0</param>
+            </state_interface>
+            <state_interface name="velocity"/>
+            <state_interface name="effort"/>
+        </joint>
     </ros2_control>
 </robot>

Commit message: changing base link colour to grey to match model

File: ros_ws/src/modular_robot/urdf/mobile_base.xacro (robot description, xacro)
@@ -13,5 +13,5 @@
             </geometry>
             <material name="blue">
-                <color rgba="0 0 1 1"/>
+                <color rgba="0.86 0.86 0.86 1"/>
             </material>
         </visual>
@@ -24,9 +24,3 @@
         <xacro:box_inertial m="${base_m}" w="${base_w}" l="${base_l}" h="${base_h}" xyz="0 0 0 " rpy="0 0 0"/>
     </link>
-    <!-- JOINTS -->
-    <!-- <joint name="${agent_namespace}_base_footprint" type="fixed">
-        <origin xyz="0 0 0.035" rpy="0 0 0"/>
-        <parent link="${agent_namespace}_footprint_link"/>
-        <child link="${agent_namespace}_base_link"/>
-    </joint> -->
 </robot>

File: ros_ws/src/pipe_swarm/urdf/mobile_base.xacro (robot description, xacro)
@@ -16,6 +16,6 @@
                 <box size="${base_w_main} ${base_l} ${base_h}"/>
             </geometry>
-            <material name="blue">
-                <color rgba="0 0 1 1"/>
+            <material name="grey">
+                <color rgba="0.86 0.86 0.86 1"/>
             </material>
         </visual>
@@ -25,7 +25,5 @@
                 <box size="${base_w_offset} ${base_l_offset} ${base_h}"/>
             </geometry>
-            <material name="blue">
-                <color rgba="0 0 1 1"/>
-            </material>
+            <material name="grey">
         </visual>
         <visual>
@@ -34,7 +32,5 @@
                 <box size="${base_w_offset} ${base_l_offset} ${base_h}"/>
             </geometry>
-            <material name="blue">
-                <color rgba="0 0 1 1"/>
-            </material>
+            <material name="grey">
         </visual>
         <visual>
@@ -43,7 +39,5 @@
                 <box size="${base_w_offset} ${base_l} ${base_l_offset}"/>
             </geometry>
-            <material name="blue">
-                <color rgba="0 0 1 1"/>
-            </material>
+            <material name="grey">
         </visual>
         <visual>
@@ -52,7 +46,5 @@
                 <box size="${base_w_offset} ${base_l} ${base_l_offset}"/>
             </geometry>
-            <material name="blue">
-                <color rgba="0 0 1 1"/>
-            </material>
+            <material name="grey">
         </visual>
         <collision>
