Commit message: adding stl wheels to modular robot

File: ros_ws/src/modular_robot/urdf/wheels.xacro (robot description, xacro)
@@ -4,10 +4,14 @@
     <xacro:property name="wheel_r" value="0.0175" />  <!-- radius /m -->
     <xacro:property name="wheel_l" value="0.01" />  <!-- length /m -->
+    <xacro:property name="wheel_y_offset" value="0.002" />  <!-- length /m -->
+    <xacro:property name="wheel_x_offset_front" value="0.008" />  <!-- length /m -->
+    <xacro:property name="wheel_x_offset_back" value="0.012" />  <!-- length /m -->
     <xacro:macro name="wheel_link" params="prefix">
-        <link name="${agent_namespace}_wheel_${prefix}_link">
+        <link name="${agent_namespace}_wheel_${prefix}_left_link">
             <visual>
                 <origin xyz="0.0 0.0 0.0" rpy="0 0.0 0.0"/>
                 <geometry>
-                    <cylinder radius="${wheel_r}" length="${wheel_l}"/>
+                    <mesh filename="package://modular_robot/meshes/wheel_right.stl" scale="0.001 0.001 0.001"/>
+                    <!-- <cylinder radius="${wheel_r}" length="${wheel_l}"/> -->
                 </geometry>
                 <material name="wheel">
@@ -18,5 +22,26 @@
                 <origin xyz="0.0 0.0 0.0" rpy="0 0.0 0.0"/>
                 <geometry>
-                    <cylinder radius="${wheel_r}" length="${wheel_l}"/>
+                    <mesh filename="package://modular_robot/meshes/wheel_right.stl" scale="0.001 0.001 0.001"/>
+                    <!-- <cylinder radius="${wheel_r}" length="${wheel_l}"/> -->
+                </geometry>
+            </collision>
+            <xacro:cylinder_solid_inertial m="${wheel_m}" r="${wheel_r}" l="${wheel_l}" xyz="0 0 0 " rpy="0 0 0"/>
+        </link>
+        <link name="${agent_namespace}_wheel_${prefix}_right_link">
+            <visual>
+                <origin xyz="0.0 0.0 0.0" rpy="0 0.0 0.0"/>
+                <geometry>
+                    <mesh filename="package://modular_robot/meshes/wheel.stl" scale="0.001 0.001 0.001"/>
+                    <!-- <cylinder radius="${wheel_r}" length="${wheel_l}"/> -->
+                </geometry>
+                <material name="wheel">
+                    <color rgba="0 0 0 1.0"/>
+                </material>
+            </visual>
+            <collision>
+                <origin xyz="0.0 0.0 0.0" rpy="0 0.0 0.0"/>
+                <geometry>
+                    <mesh filename="package://modular_robot/meshes/wheel.stl" scale="0.001 0.001 0.001"/>
+                    <!-- <cylinder radius="${wheel_r}" length="${wheel_l}"/> -->
                 </geometry>
             </collision>
@@ -25,11 +50,9 @@
     </xacro:macro>
     <!-- LINKS -->
-    <xacro:wheel_link prefix="front_right" />
-    <xacro:wheel_link prefix="front_left" />
-    <xacro:wheel_link prefix="back_right" />
-    <xacro:wheel_link prefix="back_left" />
+    <xacro:wheel_link prefix="front" />
+    <xacro:wheel_link prefix="back" />
     <!-- JOINTS -->
     <joint name="${agent_namespace}_base_wheel_front_right_joint" type="fixed">
-        <origin xyz="${base_w - wheel_r - 0.02} ${-((base_l/2) + (wheel_l/2))} ${-base_h/2}" rpy="${-pi/2} 0 0"/>
+        <origin xyz="${base_w - wheel_x_offset_front - 0.02} ${-((base_l/2) + wheel_y_offset)} ${-base_h/2}" rpy="${-pi/2} 0 0"/>
         <parent link="${agent_namespace}_base_link"/>
         <child link="${agent_namespace}_wheel_front_right_link"/>
@@ -37,5 +60,5 @@
     </joint>
     <joint name="${agent_namespace}_base_wheel_front_left_joint" type="fixed">
-        <origin xyz="${base_w - wheel_r - 0.02} ${(base_l/2) + (wheel_l/2)} ${-base_h/2}" rpy="${-pi/2} 0 0"/>
+        <origin xyz="${base_w - wheel_x_offset_front - 0.02} ${(base_l/2) + wheel_y_offset} ${-base_h/2}" rpy="${-pi/2} 0 0"/>
         <parent link="${agent_namespace}_base_link"/>
         <child link="${agent_namespace}_wheel_front_left_link"/>
@@ -43,5 +66,5 @@
     </joint>
     <joint name="${agent_namespace}_base_wheel_back_right_joint" type="fixed">
-        <origin xyz="${wheel_r - 0.02} ${-((base_l/2) + (wheel_l/2))} ${-base_h/2}" rpy="${-pi/2} 0 0"/>
+        <origin xyz="${wheel_x_offset_back - 0.02} ${-((base_l/2) + wheel_y_offset)} ${-base_h/2}" rpy="${-pi/2} 0 0"/>
         <parent link="${agent_namespace}_base_link"/>
         <child link="${agent_namespace}_wheel_back_right_link"/>
@@ -50,5 +73,5 @@
     </joint>
     <joint name="${agent_namespace}_base_wheel_back_left_joint" type="fixed">
-        <origin xyz="${wheel_r - 0.02} ${(base_l/2) + (wheel_l/2)} ${-base_h/2}" rpy="${-pi/2} 0 0"/>
+        <origin xyz="${wheel_x_offset_back - 0.02} ${(base_l/2) + wheel_y_offset} ${-base_h/2}" rpy="${-pi/2} 0 0"/>
         <parent link="${agent_namespace}_base_link"/>
         <child link="${agent_namespace}_wheel_back_left_link"/>

Commit message: modifying wheels of modular robot

File: ros_ws/src/modular_robot/urdf/wheels.xacro (robot description, xacro)
@@ -2,6 +2,6 @@
 <robot name="wheels" xmlns:xacro="http://www.ros.org/wiki/xacro">
     <xacro:property name="wheel_m" value="0.1" />  <!-- mass /kg -->
-    <xacro:property name="wheel_r" value="0.0175" />  <!-- radius /m -->
-    <xacro:property name="wheel_l" value="0.01" />  <!-- length /m -->
+    <xacro:property name="wheel_r" value="0.015" />  <!-- radius /m -->
+    <xacro:property name="wheel_l" value="0.008" />  <!-- length /m 8 or 3 -->
     <xacro:property name="wheel_y_offset" value="0.002" />  <!-- length /m -->
     <xacro:property name="wheel_x_offset_front" value="0.012" />  <!-- length /m -->
@@ -10,5 +10,5 @@
         <link name="${agent_namespace}_wheel_${prefix}_left_link">
             <visual>
-                <origin xyz="0.0 0.0 0.0" rpy="0 0.0 0.0"/>
+                <origin xyz="${-wheel_r} ${-wheel_r} ${-wheel_l/2}" rpy="0 0 0"/>
                 <geometry>
                     <mesh filename="package://modular_robot/meshes/wheel.stl" scale="0.001 0.001 0.001"/>
@@ -20,5 +20,5 @@
             </visual>
             <collision>
-                <origin xyz="0.0 0.0 0.0" rpy="0 0.0 0.0"/>
+                <origin xyz="${-wheel_r} ${-wheel_r} ${-wheel_l/2}" rpy="0 0 0"/>
                 <geometry>
                     <mesh filename="package://modular_robot/meshes/wheel.stl" scale="0.001 0.001 0.001"/>
@@ -30,5 +30,5 @@
         <link name="${agent_namespace}_wheel_${prefix}_right_link">
             <visual>
-                <origin xyz="0.0 0.0 0.0" rpy="0 0.0 0.0"/>
+                <origin xyz="${-wheel_r} ${-wheel_r} ${-wheel_l/2}" rpy="0 0 0"/>
                 <geometry>
                     <mesh filename="package://modular_robot/meshes/wheel.stl" scale="0.001 0.001 0.001"/>
@@ -40,5 +40,5 @@
             </visual>
             <collision>
-                <origin xyz="0.0 0.0 0.0" rpy="0 0.0 0.0"/>
+                <origin xyz="${-wheel_r} ${-wheel_r} ${-wheel_l/2}" rpy="0 0 0"/>
                 <geometry>
                     <mesh filename="package://modular_robot/meshes/wheel.stl" scale="0.001 0.001 0.001"/>
@@ -54,11 +54,11 @@
     <!-- JOINTS -->
     <joint name="${agent_namespace}_base_wheel_front_right_joint" type="fixed">
-        <origin xyz="${base_w - wheel_x_offset_front - 0.02} ${-((base_l/2) + wheel_y_offset)} ${-base_h/2}" rpy="${-pi/2} 0 0"/>
+        <origin xyz="${base_w - wheel_x_offset_front - 0.02} ${-((base_l/2) + (wheel_l/2) + wheel_y_offset)} ${-base_h/2}" rpy="${-pi/2} 0 0"/>
         <parent link="${agent_namespace}_base_link"/>
         <child link="${agent_namespace}_wheel_front_right_link"/>
-        <!-- <axis xyz="0 0 1"/> -->
+        <axis xyz="0 0 1"/>
     </joint>
     <joint name="${agent_namespace}_base_wheel_front_left_joint" type="fixed">
-        <origin xyz="${base_w - wheel_x_offset_front - 0.02} ${(base_l/2) + wheel_y_offset} ${-base_h/2}" rpy="${pi/2} 0 0"/>
+        <origin xyz="${base_w - wheel_x_offset_front - 0.02} ${(base_l/2) + (wheel_l/2) + wheel_y_offset} ${-base_h/2}" rpy="${pi/2} 0 0"/>
         <parent link="${agent_namespace}_base_link"/>
         <child link="${agent_namespace}_wheel_front_left_link"/>
@@ -66,5 +66,5 @@
     </joint>
     <joint name="${agent_namespace}_base_wheel_back_right_joint" type="fixed">
-        <origin xyz="${wheel_x_offset_back - 0.02} ${-((base_l/2) + wheel_y_offset)} ${-base_h/2}" rpy="${-pi/2} 0 0"/>
+        <origin xyz="${wheel_x_offset_back - 0.02} ${-((base_l/2) + (wheel_l/2) + wheel_y_offset)} ${-base_h/2}" rpy="${-pi/2} 0 0"/>
         <parent link="${agent_namespace}_base_link"/>
         <child link="${agent_namespace}_wheel_back_right_link"/>
@@ -73,5 +73,5 @@
     </joint>
     <joint name="${agent_namespace}_base_wheel_back_left_joint" type="fixed">
-        <origin xyz="${wheel_x_offset_back - 0.02} ${(base_l/2) + wheel_y_offset} ${-base_h/2}" rpy="${pi/2} 0 0"/>
+        <origin xyz="${wheel_x_offset_back - 0.02} ${(base_l/2) + (wheel_l/2) + wheel_y_offset} ${-base_h/2}" rpy="${pi/2} 0 0"/>
         <parent link="${agent_namespace}_base_link"/>
         <child link="${agent_namespace}_wheel_back_left_link"/>

Commit message: removing unused wheel axis

File: ros_ws/src/modular_robot/urdf/wheels.xacro (robot description, xacro)
@@ -57,5 +57,5 @@
         <parent link="${agent_namespace}_base_link"/>
         <child link="${agent_namespace}_wheel_front_right_link"/>
-        <axis xyz="0 0 1"/>
+        <!-- <axis xyz="0 0 1"/> -->
     </joint>
     <joint name="${agent_namespace}_base_wheel_front_left_joint" type="fixed">

Commit message: removing wheel y offset

File: ros_ws/src/modular_robot/urdf/wheels.xacro (robot description, xacro)
@@ -4,5 +4,4 @@
     <xacro:property name="wheel_r" value="0.015" />  <!-- radius /m -->
     <xacro:property name="wheel_l" value="0.008" />  <!-- length /m 8 or 3 -->
-    <xacro:property name="wheel_y_offset" value="0.002" />  <!-- length /m -->
     <xacro:property name="wheel_x_offset_front" value="0.012" />  <!-- length /m -->
     <xacro:property name="wheel_x_offset_back" value="0.008" />  <!-- length /m -->
@@ -54,5 +53,5 @@
     <!-- JOINTS -->
     <joint name="${agent_namespace}_base_wheel_front_right_joint" type="fixed">
-        <origin xyz="${base_w - wheel_x_offset_front - 0.02} ${-((base_l/2) + (wheel_l/2) + wheel_y_offset)} ${-base_h/2}" rpy="${-pi/2} 0 0"/>
+        <origin xyz="${base_w - wheel_x_offset_front - 0.02} ${-((base_l/2) + (wheel_l/2))} ${-base_h/2}" rpy="${-pi/2} 0 0"/>
         <parent link="${agent_namespace}_base_link"/>
         <child link="${agent_namespace}_wheel_front_right_link"/>
@@ -60,5 +59,5 @@
     </joint>
     <joint name="${agent_namespace}_base_wheel_front_left_joint" type="fixed">
-        <origin xyz="${base_w - wheel_x_offset_front - 0.02} ${(base_l/2) + (wheel_l/2) + wheel_y_offset} ${-base_h/2}" rpy="${pi/2} 0 0"/>
+        <origin xyz="${base_w - wheel_x_offset_front - 0.02} ${(base_l/2) + (wheel_l/2)} ${-base_h/2}" rpy="${pi/2} 0 0"/>
         <parent link="${agent_namespace}_base_link"/>
         <child link="${agent_namespace}_wheel_front_left_link"/>
@@ -66,5 +65,5 @@
     </joint>
     <joint name="${agent_namespace}_base_wheel_back_right_joint" type="fixed">
-        <origin xyz="${wheel_x_offset_back - 0.02} ${-((base_l/2) + (wheel_l/2) + wheel_y_offset)} ${-base_h/2}" rpy="${-pi/2} 0 0"/>
+        <origin xyz="${wheel_x_offset_back - 0.02} ${-((base_l/2) + (wheel_l/2))} ${-base_h/2}" rpy="${-pi/2} 0 0"/>
         <parent link="${agent_namespace}_base_link"/>
         <child link="${agent_namespace}_wheel_back_right_link"/>
@@ -73,5 +72,5 @@
     </joint>
     <joint name="${agent_namespace}_base_wheel_back_left_joint" type="fixed">
-        <origin xyz="${wheel_x_offset_back - 0.02} ${(base_l/2) + (wheel_l/2) + wheel_y_offset} ${-base_h/2}" rpy="${pi/2} 0 0"/>
+        <origin xyz="${wheel_x_offset_back - 0.02} ${(base_l/2) + (wheel_l/2)} ${-base_h/2}" rpy="${pi/2} 0 0"/>
         <parent link="${agent_namespace}_base_link"/>
         <child link="${agent_namespace}_wheel_back_left_link"/>
