Commit message: editing linkage size parameters

File: ros_ws/src/modular_robot/urdf/linkage.xacro (robot description, xacro)
@@ -3,6 +3,6 @@
     <xacro:property name="male_m" value="0.3" />  <!-- mass /kg -->
     <xacro:property name="male_w" value="0.04" />  <!-- width /m -->
-    <xacro:property name="male_h" value="0.01" />  <!-- height /m -->
-    <xacro:property name="male_l" value="0.01" />  <!-- length /m -->
+    <xacro:property name="male_h" value="0.005" />  <!-- height /m -->
+    <xacro:property name="male_l" value="0.005" />  <!-- length /m -->
     <xacro:property name="female_diameter" value="0.04" />  <!-- /m -->
     <xacro:property name="female_stopper_width" value="0.05" />  <!-- /m -->

Commit message: editing male linkage to use stl

File: ros_ws/src/modular_robot/urdf/linkage.xacro (robot description, xacro)
@@ -5,4 +5,5 @@
     <xacro:property name="male_h" value="0.005" />  <!-- height /m -->
     <xacro:property name="male_l" value="0.005" />  <!-- length /m -->
+    <xacro:property name="male_o" value="0.007" />  <!-- offset /m -->
     <xacro:property name="female_diameter" value="0.04" />  <!-- /m -->
     <xacro:property name="female_stopper_width" value="0.05" />  <!-- /m -->
@@ -38,7 +39,7 @@
     <link name="${agent_namespace}_male_link">
         <visual>
-            <origin xyz="0.0 0.0 0.0" rpy="0.0 0.0 0.0"/>
+            <origin xyz="0.0 0.0 0.0" rpy="0.0 ${pi/2} ${-pi/2}"/>
             <geometry>
-                <box size="${male_w} ${male_l} ${male_h}"/>
+                <mesh filename="package://modular_robot/meshes/key.stl" scale="0.001 0.001 0.001"/>
             </geometry>
             <material name="base">
@@ -47,7 +48,25 @@
         </visual>
         <collision>
-            <origin xyz="0.0 0.0 0.0" rpy="0.0 0.0 0.0"/>
+            <origin xyz="0.0 0.0 0.0" rpy="0.0 ${pi/2} ${-pi/2}"/>
             <geometry>
-                <box size="${male_w} ${male_l} ${male_h}"/>
+                <mesh filename="package://modular_robot/meshes/key.stl" scale="0.001 0.001 0.001"/>
+            </geometry>
+        </collision>
+        <xacro:box_inertial m="${male_m}" w="${male_w}" l="${male_l}" h="${male_h}" xyz="0 0 0 " rpy="0 0 0"/>
+    </link>
+    <link name="${agent_namespace}_cover_link">
+        <visual>
+            <origin xyz="0.0 0.0 0.0" rpy="${pi/2} 0.0 ${pi/2}"/>
+            <geometry>
+                <mesh filename="package://modular_robot/meshes/cover.stl" scale="0.001 0.001 0.001"/>
+            </geometry>
+            <material name="base">
+                <color rgba="1.0 1.0 1.0 1.0"/>
+            </material>
+        </visual>
+        <collision>
+            <origin xyz="0.0 0.0 0.0" rpy="${pi/2} 0.0 ${pi/2}"/>
+            <geometry>
+                <mesh filename="package://modular_robot/meshes/cover.stl" scale="0.001 0.001 0.001"/>
             </geometry>
         </collision>
@@ -113,7 +132,12 @@
     <!-- JOINTS -->
     <joint name="${agent_namespace}_base_male_joint" type="fixed">
-        <origin xyz="${(base_w - 0.02) + (male_w*0.5) } 0 0" rpy="0 0 0"/>
+        <origin xyz="${base_w - 0.02 + male_o} 0 0" rpy="0 0 0"/>
         <parent link="${agent_namespace}_base_link"/>
         <child link="${agent_namespace}_male_link"/>
+    </joint>
+    <joint name="${agent_namespace}_base_cover_joint" type="fixed">
+        <origin xyz="${base_w - 0.02 + male_o } 0.0 0.0" rpy="0 0 0"/>
+        <parent link="${agent_namespace}_base_link"/>
+        <child link="${agent_namespace}_cover_link"/>
     </joint>
     <joint name="${agent_namespace}_female_base_joint" type="revolute">

File: ros_ws/src/modular_robot/urdf/mobile_base.xacro (robot description, xacro)
@@ -1,8 +1,8 @@
 <?xml version="1.0" ?>
 <robot name="mobile_base" xmlns:xacro="http://www.ros.org/wiki/xacro">
-    <xacro:property name="base_m" value="0.5" />  <!-- mass /kg -->
-    <xacro:property name="base_w" value="0.15" />  <!-- width /m -->
-    <xacro:property name="base_l" value="0.05" />  <!-- length /m -->
-    <xacro:property name="base_h" value="0.045" />  <!-- height /m -->
+    <xacro:property name="base_m" value="1" />  <!-- mass /kg -->
+    <xacro:property name="base_w" value="0.1045" />  <!-- width /m -->
+    <xacro:property name="base_l" value="0.055" />  <!-- length /m -->
+    <xacro:property name="base_h" value="0.062" />  <!-- height /m -->
     <!-- LINKS -->
     <link name="${agent_namespace}_base_link">

File: ros_ws/src/pipe_swarm/urdf/linkage.xacro (robot description, xacro)
@@ -5,4 +5,5 @@
     <xacro:property name="male_h" value="0.005" />  <!-- height /m -->
     <xacro:property name="male_l" value="0.0575" />  <!-- length /m -->
+    <xacro:property name="male_o" value="0.007" />  <!-- offset /m -->
     <xacro:property name="female_diameter" value="0.04" />  <!-- /m -->
     <xacro:property name="female_stopper_width" value="0.05" />  <!-- /m -->
@@ -109,10 +110,10 @@
     <!-- JOINTS -->
     <joint name="${agent_namespace}_base_cover_joint" type="fixed">
-        <origin xyz="${(base_w*0.5)+0.007} 0.0 0.0" rpy="0 0 0"/>
+        <origin xyz="${(base_w*0.5)+male_o} 0.0 0.0" rpy="0 0 0"/>
         <parent link="${agent_namespace}_base_link"/>
         <child link="${agent_namespace}_cover_link"/>
     </joint>
     <joint name="${agent_namespace}_base_male_joint" type="fixed">
-        <origin xyz="${(base_w*0.5)+0.007} 0.0 0.0" rpy="0 0 0"/>
+        <origin xyz="${(base_w*0.5)+male_o} 0.0 0.0" rpy="0 0 0"/>
         <parent link="${agent_namespace}_base_link"/>
         <child link="${agent_namespace}_male_link"/>

Commit message: adding pivot joint and fixing inertia

File: ros_ws/src/modular_robot/urdf/linkage.xacro (robot description, xacro)
@@ -14,5 +14,6 @@
     <xacro:property name="female_w" value="${(female_diameter/2) + female_stopper_width + female_hole_depth}" />  <!-- width /m -->
     <xacro:property name="female_h" value="${female_diameter}" />  <!-- height /m -->
-    <xacro:property name="female_l" value="0.028" />  <!-- /m -->
+    <xacro:property name="female_l" value="0.028" />  <!-- length /m -->
+    <xacro:property name="pivot_l" value="0.055" />  <!-- length /m -->
     <xacro:macro name="female_rotation_shape">
             <origin xyz="0 0 0" rpy="${pi/2} 0 0"/>
@@ -130,4 +131,22 @@
         <xacro:box_inertial m="${female_m}" w="${female_w}" l="${female_l}" h="${female_h}" xyz="${female_diameter/2 - female_w/2} 0 0 " rpy="0 0 0"/>
     </link>
+    <link name="${agent_namespace}_pivot_link">
+       <visual>
+            <origin xyz="0 ${pivot_l/2} 0" rpy="${pi/2} 0.0 ${-pi/2}"/>
+            <geometry>
+                <mesh filename="package://modular_robot/meshes/pivot.stl" scale="0.001 0.001 0.001"/>
+            </geometry>
+            <material name="base">
+                <color rgba="1.0 1.0 1.0 1.0"/>
+            </material>
+        </visual>
+        <collision>
+            <origin xyz="0 0 0" rpy="${pi/2} 0.0 ${-pi/2}"/>
+            <geometry>
+                <mesh filename="package://modular_robot/meshes/pivot.stl" scale="0.001 0.001 0.001"/>
+            </geometry>
+        </collision>
+        <xacro:box_inertial m="${female_m}" w="0.05" l="0.05" h="0.05" xyz="0 0 0" rpy="0 0 0"/>
+    </link>
     <!-- JOINTS -->
     <joint name="${agent_namespace}_base_male_joint" type="fixed">
@@ -144,8 +163,15 @@
         <origin xyz="0 0 0" rpy="0 0 0"/>
         <parent link="${agent_namespace}_female_link"/>
-        <child link="${agent_namespace}_base_link"/>
+        <child link="${agent_namespace}_pivot_link"/>
         <axis xyz="0 1 0"/>
         <limit lower="${-pi/2}" upper="${pi/2}" effort="1.0" velocity="1.0"/>
         <dynamics damping="0.3" friction="0.5"/>  <!-- Add damping -->
+    </joint>
+    <joint name="${agent_namespace}_pivot_base_joint" type="revolute">
+        <origin xyz="${0.02-0.014} 0 0" rpy="0 0 0"/>
+        <parent link="${agent_namespace}_pivot_link"/>
+        <child link="${agent_namespace}_base_link"/>
+        <axis xyz="0 1 0"/>
+        <limit lower="${-pi/4}" upper="${pi/4}" effort="1.0" velocity="1.0"/>
     </joint>
     <!-- <joint name="${agent_namespace}_footprint_base_joint" type="fixed">

File: ros_ws/src/pipe_swarm/urdf/linkage.xacro (robot description, xacro)
@@ -15,4 +15,5 @@
     <xacro:property name="female_h" value="${female_diameter}" />  <!-- height /m -->
     <xacro:property name="female_l" value="0.028" />   <!-- length /m -->
+    <xacro:property name="pivot_l" value="0.055" />  <!-- length /m -->
     <xacro:macro name="female_rotation_shape">
             <origin xyz="0 0 0" rpy="${pi/2} 0 0"/>
@@ -92,5 +93,5 @@
     <link name="${agent_namespace}_pivot_link">
        <visual>
-            <origin xyz="0 0 0" rpy="${pi/2} 0.0 ${-pi/2}"/>
+            <origin xyz="0 ${pivot_l/2} 0" rpy="${pi/2} 0.0 ${-pi/2}"/>
             <geometry>
                 <mesh filename="package://pipe_swarm/models/hollow_pipe/meshes/pivot.stl" scale="0.001 0.001 0.001"/>
@@ -120,5 +121,5 @@
     </joint>
     <joint name="base_female_joint" type="revolute">
-        <origin xyz="${-(base_w*0.5)+0.014} 0.0275 0.0" rpy="0 0 0"/>
+        <origin xyz="${-(base_w*0.5)+0.014} 0 0" rpy="0 0 0"/>
         <parent link="${agent_namespace}_base_link"/>
         <child link="${agent_namespace}_pivot_link"/>
@@ -132,5 +133,5 @@
     </joint> -->
     <joint name="${agent_namespace}_base_neutral_joint" type="fixed">
-        <origin xyz="-0.0665 -0.0275 0.0" rpy="0 0 0"/>
+        <origin xyz="-0.0665 0 0.0" rpy="0 0 0"/>
         <parent link="${agent_namespace}_pivot_link"/>
         <child link="${agent_namespace}_female_link"/>

Commit message: updating female linkage with stl

File: ros_ws/src/modular_robot/urdf/linkage.xacro (robot description, xacro)
@@ -16,4 +16,6 @@
     <xacro:property name="female_l" value="0.028" />  <!-- length /m -->
     <xacro:property name="pivot_l" value="0.055" />  <!-- length /m -->
+    <xacro:property name="pivot_o" value="0.01" />  <!-- offset from centre of robot /m -->
+    <xacro:property name="lock_w" value="0.0665" />  <!-- width /m -->
     <xacro:macro name="female_rotation_shape">
             <origin xyz="0 0 0" rpy="${pi/2} 0 0"/>
@@ -75,36 +77,9 @@
     </link>
     <link name="${agent_namespace}_female_link">
-        <visual>
-            <xacro:female_rotation_shape />
-            <material name="base">
-                <color rgba="1.0 1.0 1.0 1.0"/>
-            </material>
-        </visual>
-        <visual>
-            <xacro:female_stopper_shape />
-            <material name="base">
-                <color rgba="1.0 1.0 1.0 1.0"/>
-            </material>
-        </visual>
-        <visual>
-            <xacro:female_wall_shape y_offset="0" z_offset="1"/>
-            <material name="base">
-                <color rgba="1.0 1.0 1.0 1.0"/>
-            </material>
-        </visual>
-        <visual>
-            <xacro:female_wall_shape y_offset="1" z_offset="0"/>
-            <material name="base">
-                <color rgba="1.0 1.0 1.0 1.0"/>
-            </material>
-        </visual>
-        <visual>
-            <xacro:female_wall_shape y_offset="-1" z_offset="0"/>
-            <material name="base">
-                <color rgba="1.0 1.0 1.0 1.0"/>
-            </material>
-        </visual>
-        <visual>
-            <xacro:female_wall_shape y_offset="0" z_offset="-1"/>
+       <visual>
+            <origin xyz="${-lock_w/2} 0 0" rpy="0.0 ${pi/2} ${pi/2}"/>
+            <geometry>
+                <mesh filename="package://modular_robot/meshes/lock.stl" scale="0.001 0.001 0.001"/>
+            </geometry>
             <material name="base">
                 <color rgba="1.0 1.0 1.0 1.0"/>
@@ -112,22 +87,9 @@
         </visual>
         <collision>
-            <xacro:female_rotation_shape />
+            <origin xyz="${-lock_w/2} 0 0" rpy="0.0 ${pi/2} ${pi/2}"/>
+            <geometry>
+                <mesh filename="package://modular_robot/meshes/lock.stl" scale="0.001 0.001 0.001"/>
+            </geometry>
         </collision>
-        <collision>
-            <xacro:female_stopper_shape />
-        </collision>
-        <collision>
-            <xacro:female_wall_shape y_offset="0" z_offset="1"/>
-        </collision>
-        <collision>
-            <xacro:female_wall_shape y_offset="0" z_offset="-1"/>
-        </collision>
-        <collision>
-            <xacro:female_wall_shape y_offset="1" z_offset="0"/>
-        </collision>
-        <collision>
-            <xacro:female_wall_shape y_offset="-1" z_offset="0"/>
-        </collision>
-        <xacro:box_inertial m="${female_m}" w="${female_w}" l="${female_l}" h="${female_h}" xyz="${female_diameter/2 - female_w/2} 0 0 " rpy="0 0 0"/>
     </link>
     <link name="${agent_namespace}_pivot_link">
@@ -142,5 +104,5 @@
         </visual>
         <collision>
-            <origin xyz="0 0 0" rpy="${pi/2} 0.0 ${-pi/2}"/>
+            <origin xyz="0 ${pivot_l/2} 0" rpy="${pi/2} 0.0 ${-pi/2}"/>
             <geometry>
                 <mesh filename="package://modular_robot/meshes/pivot.stl" scale="0.001 0.001 0.001"/>
@@ -151,27 +113,25 @@
     <!-- JOINTS -->
     <joint name="${agent_namespace}_base_male_joint" type="fixed">
-        <origin xyz="${base_w - 0.02 + male_o} 0 0" rpy="0 0 0"/>
+        <origin xyz="${base_w - 0.02 + male_o} 0 ${pivot_o}" rpy="0 0 0"/>
         <parent link="${agent_namespace}_base_link"/>
         <child link="${agent_namespace}_male_link"/>
     </joint>
     <joint name="${agent_namespace}_base_cover_joint" type="fixed">
-        <origin xyz="${base_w - 0.02 + male_o } 0.0 0.0" rpy="0 0 0"/>
+        <origin xyz="${base_w - 0.02 + male_o } 0 ${pivot_o}" rpy="0 0 0"/>
         <parent link="${agent_namespace}_base_link"/>
         <child link="${agent_namespace}_cover_link"/>
     </joint>
-    <joint name="${agent_namespace}_female_base_joint" type="revolute">
-        <origin xyz="0 0 0" rpy="0 0 0"/>
+    <joint name="${agent_namespace}_female_pivot_joint" type="fixed">
+        <origin xyz="${lock_w/2} 0 0" rpy="0 0 0"/>
         <parent link="${agent_namespace}_female_link"/>
         <child link="${agent_namespace}_pivot_link"/>
-        <axis xyz="0 1 0"/>
-        <limit lower="${-pi/2}" upper="${pi/2}" effort="1.0" velocity="1.0"/>
-        <dynamics damping="0.3" friction="0.5"/>  <!-- Add damping -->
     </joint>
     <joint name="${agent_namespace}_pivot_base_joint" type="revolute">
-        <origin xyz="${0.02-0.014} 0 0" rpy="0 0 0"/>
+        <origin xyz="${0.02-0.014} 0 ${-pivot_o}" rpy="0 0 0"/>
         <parent link="${agent_namespace}_pivot_link"/>
         <child link="${agent_namespace}_base_link"/>
         <axis xyz="0 1 0"/>
         <limit lower="${-pi/4}" upper="${pi/4}" effort="1.0" velocity="1.0"/>
+        <dynamics damping="0.3" friction="0.5"/>
     </joint>
     <!-- <joint name="${agent_namespace}_footprint_base_joint" type="fixed">

File: ros_ws/src/modular_robot/urdf/modular_robot.urdf.xacro (robot description, xacro)
@@ -8,24 +8,18 @@
     <xacro:pipe_robot agent_namespace="agent_n2" include_gazebo="true"/>
     <xacro:pipe_robot agent_namespace="agent_n3" include_gazebo="true"/>
-    <xacro:pipe_robot agent_namespace="agent_n4" include_gazebo="true"/>
-    <joint name="footprint_agent_n2_joint" type="fixed">
+    <joint name="footprint_agent_n_joint" type="fixed">
         <origin xyz="0 0 0" rpy="0 0 0"/>
+        <parent link="footprint_link"/>
         <child link="agent_n_female_link"/>
-        <parent link="footprint_link"/>
     </joint>
     <joint name="agent_n_agent_n2_joint" type="fixed">
-        <origin xyz="${(0.05+0.02)} 0 0" rpy="0 0 0"/>
+        <origin xyz="0.01 0 0" rpy="0 0 0"/>
         <parent link="agent_n_male_link"/>
         <child link="agent_n2_female_link"/>
     </joint>
     <joint name="agent_n2_agent_n3_joint" type="fixed">
-        <origin xyz="${(0.05+0.02)} 0 0" rpy="0 0 0"/>
+        <origin xyz="0.01 0 0" rpy="0 0 0"/>
         <parent link="agent_n2_male_link"/>
         <child link="agent_n3_female_link"/>
-    </joint>
-    <joint name="agent_n3_agent_n4_joint" type="fixed">
-        <origin xyz="${(0.05+0.02)} 0 0" rpy="0 0 0"/>
-        <parent link="agent_n3_male_link"/>
-        <child link="agent_n4_female_link"/>
     </joint>
     <gazebo>
@@ -40,5 +34,5 @@
             <plugin>gazebo_ros2_control/GazeboSystem</plugin>
         </hardware>
-        <joint name="agent_n_female_base_joint">
+        <joint name="agent_n_pivot_base_joint">
             <command_interface name="position">
                 <param name="min">-pi/2</param>
@@ -51,5 +45,5 @@
             <state_interface name="effort"/>
         </joint>
-        <joint name="agent_n2_female_base_joint">
+        <joint name="agent_n2_pivot_base_joint">
             <command_interface name="position">
                 <param name="min">-pi/2</param>
@@ -62,16 +56,5 @@
             <state_interface name="effort"/>
         </joint>
-        <joint name="agent_n3_female_base_joint">
-            <command_interface name="position">
-                <param name="min">-pi/2</param>
-                <param name="max">pi/2</param>
-            </command_interface>
-            <state_interface name="position">
-                <param name="initial_value">0.0</param>
-            </state_interface>
-            <state_interface name="velocity"/>
-            <state_interface name="effort"/>
-        </joint>
-        <joint name="agent_n4_female_base_joint">
+        <joint name="agent_n3_pivot_base_joint">
             <command_interface name="position">
                 <param name="min">-pi/2</param>

File: ros_ws/src/pipe_swarm/urdf/linkage.xacro (robot description, xacro)
@@ -16,4 +16,5 @@
     <xacro:property name="female_l" value="0.028" />   <!-- length /m -->
     <xacro:property name="pivot_l" value="0.055" />  <!-- length /m -->
+    <xacro:property name="lock_w" value="0.0665" />  <!-- width /m -->
     <xacro:macro name="female_rotation_shape">
             <origin xyz="0 0 0" rpy="${pi/2} 0 0"/>
@@ -76,5 +77,5 @@
     <link name="${agent_namespace}_female_link">
        <visual>
-            <origin xyz="0 0 0" rpy="0.0 ${pi/2} ${pi/2}"/>
+            <origin xyz="${-lock_w/2} 0 0" rpy="0.0 ${pi/2} ${pi/2}"/>
             <geometry>
                 <mesh filename="package://pipe_swarm/models/hollow_pipe/meshes/lock.stl" scale="0.001 0.001 0.001"/>
@@ -85,5 +86,5 @@
         </visual>
         <collision>
-            <origin xyz="0 0 0" rpy="0.0 ${pi/2} ${pi/2}"/>
+            <origin xyz="${-lock_w/2} 0 0" rpy="0.0 ${pi/2} ${pi/2}"/>
             <geometry>
                 <mesh filename="package://pipe_swarm/models/hollow_pipe/meshes/lock.stl" scale="0.001 0.001 0.001"/>
@@ -102,5 +103,5 @@
         </visual>
         <collision>
-            <origin xyz="0 0 0" rpy="${pi/2} 0.0 ${-pi/2}"/>
+            <origin xyz="0 ${pivot_l/2} 0" rpy="${pi/2} 0.0 ${-pi/2}"/>
             <geometry>
                 <mesh filename="package://pipe_swarm/models/hollow_pipe/meshes/pivot.stl" scale="0.001 0.001 0.001"/>
@@ -133,5 +134,5 @@
     </joint> -->
     <joint name="${agent_namespace}_base_neutral_joint" type="fixed">
-        <origin xyz="-0.0665 0 0.0" rpy="0 0 0"/>
+        <origin xyz="${-lock_w/2} 0 0.0" rpy="0 0 0"/>
         <parent link="${agent_namespace}_pivot_link"/>
         <child link="${agent_namespace}_female_link"/>
