Commit message: updating linkage dimensions

File: ros_ws/src/modular_robot/urdf/linkage.xacro (robot description, xacro)
@@ -15,28 +15,9 @@
     <xacro:property name="female_h" value="${female_diameter}" />  <!-- height /m -->
     <xacro:property name="female_l" value="0.028" />  <!-- length /m -->
+    <xacro:property name="pivot_w" value="0.027" />  <!-- length /m -->
     <xacro:property name="pivot_l" value="0.055" />  <!-- length /m -->
     <xacro:property name="pivot_o" value="0.01" />  <!-- offset from centre of robot /m -->
-    <xacro:property name="lock_w" value="0.0665" />  <!-- width /m -->
-    <xacro:macro name="female_rotation_shape">
-            <origin xyz="0 0 0" rpy="${pi/2} 0 0"/>
-            <geometry>
-                <cylinder radius="${female_diameter/2}" length="${female_l}"/>
-            </geometry>
-    </xacro:macro>
-    <xacro:macro name="female_stopper_shape">
-            <origin xyz="${-female_stopper_width/2} 0 0" rpy="0 0 0"/>
-            <geometry>
-                <box size="${female_stopper_width} ${female_l} ${female_diameter}"/>
-            </geometry>
-    </xacro:macro>
-    <xacro:macro name="female_wall_shape" params="y_offset z_offset">
-            <origin xyz="${-(female_stopper_width + female_hole_depth/2)}
-                        ${y_offset * (female_wall_thickness/2 + female_hole_thickness/2)}
-                        ${z_offset * (female_wall_thickness/2 + female_hole_thickness/2)}"
-                        rpy="0 0 0"/>
-            <geometry>
-                <box size="${female_hole_depth} ${female_wall_thickness} ${female_wall_thickness}"/>
-            </geometry>
-    </xacro:macro>
+    <xacro:property name="lock_w" value="0.02" />  <!-- width /m -->
+    <xacro:property name="cover_o" value="0.003" />  <!-- offset /m -->
     <!-- LINKS -->
     <link name="${agent_namespace}_male_link">
@@ -62,5 +43,5 @@
             <origin xyz="0.0 0.0 0.0" rpy="${pi/2} 0.0 ${pi/2}"/>
             <geometry>
-                <mesh filename="package://modular_robot/meshes/cover.stl" scale="0.001 0.001 0.001"/>
+                <mesh filename="package://modular_robot/meshes/cover_v2.stl" scale="0.001 0.001 0.001"/>
             </geometry>
             <material name="base">
@@ -71,5 +52,5 @@
             <origin xyz="0.0 0.0 0.0" rpy="${pi/2} 0.0 ${pi/2}"/>
             <geometry>
-                <mesh filename="package://modular_robot/meshes/cover.stl" scale="0.001 0.001 0.001"/>
+                <mesh filename="package://modular_robot/meshes/cover_v2.stl" scale="0.001 0.001 0.001"/>
             </geometry>
         </collision>
@@ -80,5 +61,5 @@
             <origin xyz="${-lock_w/2} 0 0" rpy="0.0 ${pi/2} ${pi/2}"/>
             <geometry>
-                <mesh filename="package://modular_robot/meshes/lock.stl" scale="0.001 0.001 0.001"/>
+                <mesh filename="package://modular_robot/meshes/lock_v2.stl" scale="0.001 0.001 0.001"/>
             </geometry>
             <material name="base">
@@ -89,5 +70,5 @@
             <origin xyz="${-lock_w/2} 0 0" rpy="0.0 ${pi/2} ${pi/2}"/>
             <geometry>
-                <mesh filename="package://modular_robot/meshes/lock.stl" scale="0.001 0.001 0.001"/>
+                <mesh filename="package://modular_robot/meshes/lock_v2.stl" scale="0.001 0.001 0.001"/>
             </geometry>
         </collision>
@@ -118,15 +99,15 @@
     </joint>
     <joint name="${agent_namespace}_base_cover_joint" type="fixed">
-        <origin xyz="${base_w - 0.02 + male_o } 0 ${pivot_o}" rpy="0 0 0"/>
+        <origin xyz="${base_w - 0.02 + cover_o } 0 ${pivot_o}" rpy="0 0 0"/>
         <parent link="${agent_namespace}_base_link"/>
         <child link="${agent_namespace}_cover_link"/>
     </joint>
     <joint name="${agent_namespace}_female_pivot_joint" type="fixed">
-        <origin xyz="${lock_w/2} 0 0" rpy="0 0 0"/>
+        <origin xyz="${(pivot_w) + (lock_w/2)} 0 0" rpy="0 0 0"/>
         <parent link="${agent_namespace}_female_link"/>
         <child link="${agent_namespace}_pivot_link"/>
     </joint>
     <joint name="${agent_namespace}_pivot_base_joint" type="revolute">
-        <origin xyz="${0.02-0.014} 0 ${-pivot_o}" rpy="0 0 0"/>
+        <origin xyz="${0.02-pivot_o} 0 ${-pivot_o}" rpy="0 0 0"/>
         <parent link="${agent_namespace}_pivot_link"/>
         <child link="${agent_namespace}_base_link"/>
@@ -135,8 +116,3 @@
         <dynamics damping="0.3" friction="0.5"/>
     </joint>
-    <!-- <joint name="${agent_namespace}_footprint_base_joint" type="fixed">
-        <origin xyz="${(base_w*0.5) - female_diameter/2} 0 0" rpy="0 0 0"/>
-        <parent link="${agent_namespace}_footprint_link"/>
-        <child link="${agent_namespace}_base_link"/>
-    </joint> -->
 </robot>

Commit message: removing unused stl

File: ros_ws/src/modular_robot/urdf/linkage.xacro (robot description, xacro)
@@ -43,5 +43,5 @@
             <origin xyz="0.0 0.0 0.0" rpy="${pi/2} 0.0 ${pi/2}"/>
             <geometry>
-                <mesh filename="package://modular_robot/meshes/cover_v2.stl" scale="0.001 0.001 0.001"/>
+                <mesh filename="package://modular_robot/meshes/cover.stl" scale="0.001 0.001 0.001"/>
             </geometry>
             <material name="base">
@@ -52,5 +52,5 @@
             <origin xyz="0.0 0.0 0.0" rpy="${pi/2} 0.0 ${pi/2}"/>
             <geometry>
-                <mesh filename="package://modular_robot/meshes/cover_v2.stl" scale="0.001 0.001 0.001"/>
+                <mesh filename="package://modular_robot/meshes/cover.stl" scale="0.001 0.001 0.001"/>
             </geometry>
         </collision>
@@ -61,5 +61,5 @@
             <origin xyz="${-lock_w/2} 0 0" rpy="0.0 ${pi/2} ${pi/2}"/>
             <geometry>
-                <mesh filename="package://modular_robot/meshes/lock_v2.stl" scale="0.001 0.001 0.001"/>
+                <mesh filename="package://modular_robot/meshes/lock.stl" scale="0.001 0.001 0.001"/>
             </geometry>
             <material name="base">
@@ -70,5 +70,5 @@
             <origin xyz="${-lock_w/2} 0 0" rpy="0.0 ${pi/2} ${pi/2}"/>
             <geometry>
-                <mesh filename="package://modular_robot/meshes/lock_v2.stl" scale="0.001 0.001 0.001"/>
+                <mesh filename="package://modular_robot/meshes/lock.stl" scale="0.001 0.001 0.001"/>
             </geometry>
         </collision>

File: ros_ws/src/pipe_swarm/urdf/linkage.xacro (robot description, xacro)
@@ -63,5 +63,5 @@
             <origin xyz="0.0 0.0 0.0" rpy="${pi/2} 0.0 ${pi/2}"/>
             <geometry>
-                <mesh filename="package://pipe_swarm/models/hollow_pipe/meshes/cover_v2.stl" scale="0.001 0.001 0.001"/>
+                <mesh filename="package://pipe_swarm/models/hollow_pipe/meshes/cover.stl" scale="0.001 0.001 0.001"/>
             </geometry>
             <material name="base">
@@ -72,5 +72,5 @@
             <origin xyz="0.0 0.0 0.0" rpy="${pi/2} 0.0 ${pi/2}"/>
             <geometry>
-                <mesh filename="package://pipe_swarm/models/hollow_pipe/meshes/cover_v2.stl" scale="0.001 0.001 0.001"/>
+                <mesh filename="package://pipe_swarm/models/hollow_pipe/meshes/cover.stl" scale="0.001 0.001 0.001"/>
             </geometry>
         </collision>
@@ -81,5 +81,5 @@
             <origin xyz="${-lock_w/2} 0 0" rpy="0.0 ${pi/2} ${pi/2}"/>
             <geometry>
-                <mesh filename="package://pipe_swarm/models/hollow_pipe/meshes/lock_v2.stl" scale="0.001 0.001 0.001"/>
+                <mesh filename="package://pipe_swarm/models/hollow_pipe/meshes/lock.stl" scale="0.001 0.001 0.001"/>
             </geometry>
             <material name="base">
@@ -90,5 +90,5 @@
             <origin xyz="${-lock_w/2} 0 0" rpy="0.0 ${pi/2} ${pi/2}"/>
             <geometry>
-                <mesh filename="package://pipe_swarm/models/hollow_pipe/meshes/lock_v2.stl" scale="0.001 0.001 0.001"/>
+                <mesh filename="package://pipe_swarm/models/hollow_pipe/meshes/lock.stl" scale="0.001 0.001 0.001"/>
             </geometry>
         </collision>

Commit message: correcting linkage dimensions

File: ros_ws/src/modular_robot/urdf/linkage.xacro (robot description, xacro)
@@ -99,5 +99,5 @@
     </joint>
     <joint name="${agent_namespace}_base_cover_joint" type="fixed">
-        <origin xyz="${base_w - 0.02 + cover_o } 0 ${pivot_o}" rpy="0 0 0"/>
+        <origin xyz="${base_w - 0.02 - cover_o } 0 ${pivot_o}" rpy="0 0 0"/>
         <parent link="${agent_namespace}_base_link"/>
         <child link="${agent_namespace}_cover_link"/>

File: ros_ws/src/modular_robot/urdf/modular_robot.urdf.xacro (robot description, xacro)
@@ -14,10 +14,10 @@
     </joint>
     <joint name="agent_n_agent_n2_joint" type="fixed">
-        <origin xyz="0.01 0 0" rpy="0 0 0"/>
+        <origin xyz="0 0 0" rpy="0 0 0"/>
         <parent link="agent_n_male_link"/>
         <child link="agent_n2_female_link"/>
     </joint>
     <joint name="agent_n2_agent_n3_joint" type="fixed">
-        <origin xyz="0.01 0 0" rpy="0 0 0"/>
+        <origin xyz="0 0 0" rpy="0 0 0"/>
         <parent link="agent_n2_male_link"/>
         <child link="agent_n3_female_link"/>

Commit message: fixing male inertia for modular robot

File: ros_ws/src/modular_robot/urdf/linkage.xacro (robot description, xacro)
@@ -1,23 +1,25 @@
 <?xml version="1.0"?>
 <robot name="linkage" xmlns:xacro="http://www.ros.org/wiki/xacro">
-    <xacro:property name="male_m" value="0.3" />  <!-- mass /kg -->
-    <xacro:property name="male_w" value="0.04" />  <!-- width /m -->
-    <xacro:property name="male_h" value="0.005" />  <!-- height /m -->
-    <xacro:property name="male_l" value="0.005" />  <!-- length /m -->
+    <xacro:property name="cover_m" value="0.1" />  <!-- mass /kg -->
+    <xacro:property name="cover_w" value="0.029" />  <!-- width /m -->
+    <xacro:property name="cover_h" value="0.024" />  <!-- height /m -->
+    <xacro:property name="cover_l" value="0.024" />  <!-- length /m -->
+    <xacro:property name="cover_o" value="0.0045" />  <!-- offset /m -->
+    <xacro:property name="cover_out" value="0.0015" />  <!-- extruded cover /m -->
+    <xacro:property name="male_m" value="0.1" />  <!-- mass /kg -->
+    <xacro:property name="male_w" value="0.014" />  <!-- width /m -->
+    <xacro:property name="male_h" value="0.0128" />  <!-- length /m -->
+    <xacro:property name="male_l" value="0.0054" />  <!-- height /m -->
     <xacro:property name="male_o" value="0.007" />  <!-- offset /m -->
-    <xacro:property name="female_diameter" value="0.04" />  <!-- /m -->
-    <xacro:property name="female_stopper_width" value="0.05" />  <!-- /m -->
-    <xacro:property name="female_hole_depth" value="0.03" />  <!-- /m -->
-    <xacro:property name="female_wall_thickness" value="0.01" />  <!-- /m -->
-    <xacro:property name="female_hole_thickness" value="0.01" />  <!-- /m -->
     <xacro:property name="female_m" value="0.1" />  <!-- mass /kg -->
-    <xacro:property name="female_w" value="${(female_diameter/2) + female_stopper_width + female_hole_depth}" />  <!-- width /m -->
-    <xacro:property name="female_h" value="${female_diameter}" />  <!-- height /m -->
-    <xacro:property name="female_l" value="0.028" />  <!-- length /m -->
+    <xacro:property name="female_w" value="0.02" />  <!-- width /m -->
+    <xacro:property name="female_h" value="0.024" />  <!-- height /m -->
+    <xacro:property name="female_l" value="0.024" />   <!-- length /m -->
     <xacro:property name="pivot_w" value="0.027" />  <!-- length /m -->
     <xacro:property name="pivot_l" value="0.055" />  <!-- length /m -->
     <xacro:property name="pivot_o" value="0.01" />  <!-- offset from centre of robot /m -->
+    <xacro:property name="pivot_zo" value="0.01" />  <!-- offset from centre of robot /m -->
     <xacro:property name="lock_w" value="0.02" />  <!-- width /m -->
-    <xacro:property name="cover_o" value="0.003" />  <!-- offset /m -->
+    <!-- <xacro:property name="cover_o" value="0.003" />  offset /m -->
     <!-- LINKS -->
     <link name="${agent_namespace}_male_link">
@@ -37,5 +39,5 @@
             </geometry>
         </collision>
-        <xacro:box_inertial m="${male_m}" w="${male_w}" l="${male_l}" h="${male_h}" xyz="0 0 0 " rpy="0 0 0"/>
+        <xacro:box_inertial m="${male_m}" w="${male_w}" l="${male_l}" h="${male_h}" xyz="${-male_w/2} 0 0 " rpy="0 0 0"/>
     </link>
     <link name="${agent_namespace}_cover_link">
@@ -55,5 +57,5 @@
             </geometry>
         </collision>
-        <xacro:box_inertial m="${male_m}" w="${male_w}" l="${male_l}" h="${male_h}" xyz="0 0 0 " rpy="0 0 0"/>
+        <xacro:box_inertial m="${cover_m}" w="${cover_w}" l="${cover_l}" h="${cover_h}" xyz="${-cover_o} 0 0 " rpy="0 0 0"/>
     </link>
     <link name="${agent_namespace}_female_link">
@@ -94,10 +96,10 @@
     <!-- JOINTS -->
     <joint name="${agent_namespace}_base_male_joint" type="fixed">
-        <origin xyz="${base_w - 0.02 + male_o} 0 ${pivot_o}" rpy="0 0 0"/>
+        <origin xyz="${base_w - 0.02 + male_o} 0 ${pivot_zo}" rpy="0 0 0"/>
         <parent link="${agent_namespace}_base_link"/>
         <child link="${agent_namespace}_male_link"/>
     </joint>
     <joint name="${agent_namespace}_base_cover_joint" type="fixed">
-        <origin xyz="${base_w - 0.02 - cover_o } 0 ${pivot_o}" rpy="0 0 0"/>
+        <origin xyz="${base_w - 0.02 - cover_o + cover_out} 0 ${pivot_zo}" rpy="0 0 0"/>
         <parent link="${agent_namespace}_base_link"/>
         <child link="${agent_namespace}_cover_link"/>
@@ -109,5 +111,5 @@
     </joint>
     <joint name="${agent_namespace}_pivot_base_joint" type="revolute">
-        <origin xyz="${0.02-pivot_o} 0 ${-pivot_o}" rpy="0 0 0"/>
+        <origin xyz="${0.02-pivot_o} 0 ${-pivot_zo}" rpy="0 0 0"/>
         <parent link="${agent_namespace}_pivot_link"/>
         <child link="${agent_namespace}_base_link"/>

File: ros_ws/src/pipe_swarm/urdf/linkage.xacro (robot description, xacro)
@@ -9,6 +9,6 @@
     <xacro:property name="male_m" value="0.1" />  <!-- mass /kg -->
     <xacro:property name="male_w" value="0.014" />  <!-- width /m -->
+    <xacro:property name="male_h" value="0.0128" />  <!-- length /m -->
     <xacro:property name="male_l" value="0.0054" />  <!-- height /m -->
-    <xacro:property name="male_h" value="0.0128" />  <!-- length /m -->
     <xacro:property name="male_o" value="0.007" />  <!-- offset /m -->
     <xacro:property name="pivot_m" value="0.1" />  <!-- mass /kg -->

Commit message: fixing female inertia for modular robot

File: ros_ws/src/modular_robot/urdf/linkage.xacro (robot description, xacro)
@@ -12,13 +12,15 @@
     <xacro:property name="male_l" value="0.0054" />  <!-- height /m -->
     <xacro:property name="male_o" value="0.007" />  <!-- offset /m -->
+    <xacro:property name="pivot_m" value="0.1" />  <!-- mass /kg -->
+    <xacro:property name="pivot_w" value="0.035" />  <!-- width /m -->
+    <xacro:property name="pivot_h" value="0.024" />  <!-- height /m -->
+    <xacro:property name="pivot_l" value="0.055" />   <!-- length /m -->
+    <xacro:property name="pivot_o" value="0.0075" />  <!-- offset /m -->
+    <xacro:property name="pivot_zo" value="0.01" />  <!-- offset from centre of robot /m -->
     <xacro:property name="female_m" value="0.1" />  <!-- mass /kg -->
     <xacro:property name="female_w" value="0.02" />  <!-- width /m -->
     <xacro:property name="female_h" value="0.024" />  <!-- height /m -->
     <xacro:property name="female_l" value="0.024" />   <!-- length /m -->
-    <xacro:property name="pivot_w" value="0.027" />  <!-- length /m -->
-    <xacro:property name="pivot_l" value="0.055" />  <!-- length /m -->
-    <xacro:property name="pivot_o" value="0.01" />  <!-- offset from centre of robot /m -->
-    <xacro:property name="pivot_zo" value="0.01" />  <!-- offset from centre of robot /m -->
-    <xacro:property name="lock_w" value="0.02" />  <!-- width /m -->
+    <xacro:property name="lock_o" value="0.01" />  <!-- width /m -->
     <!-- <xacro:property name="cover_o" value="0.003" />  offset /m -->
     <!-- LINKS -->
@@ -61,5 +63,5 @@
     <link name="${agent_namespace}_female_link">
        <visual>
-            <origin xyz="${-lock_w/2} 0 0" rpy="0.0 ${pi/2} ${pi/2}"/>
+            <origin xyz="${-female_w/2} 0 0" rpy="0.0 ${pi/2} ${pi/2}"/>
             <geometry>
                 <mesh filename="package://modular_robot/meshes/lock.stl" scale="0.001 0.001 0.001"/>
@@ -70,9 +72,10 @@
         </visual>
         <collision>
-            <origin xyz="${-lock_w/2} 0 0" rpy="0.0 ${pi/2} ${pi/2}"/>
+            <origin xyz="${-female_w/2} 0 0" rpy="0.0 ${pi/2} ${pi/2}"/>
             <geometry>
                 <mesh filename="package://modular_robot/meshes/lock.stl" scale="0.001 0.001 0.001"/>
             </geometry>
         </collision>
+        <xacro:box_inertial m="${female_m}" w="${female_w}" l="${female_l}" h="${female_h}" xyz="0 0 0" rpy="0 0 0"/>
     </link>
     <link name="${agent_namespace}_pivot_link">
@@ -92,5 +95,5 @@
             </geometry>
         </collision>
-        <xacro:box_inertial m="${female_m}" w="0.05" l="0.05" h="0.05" xyz="0 0 0" rpy="0 0 0"/>
+        <xacro:box_inertial m="${pivot_m}" w="${pivot_w}" l="${pivot_l}" h="${pivot_h}" xyz="${-pivot_w/2 + pivot_o} 0 0" rpy="0 0 0"/>
     </link>
     <!-- JOINTS -->
@@ -106,10 +109,10 @@
     </joint>
     <joint name="${agent_namespace}_female_pivot_joint" type="fixed">
-        <origin xyz="${(pivot_w) + (lock_w/2)} 0 0" rpy="0 0 0"/>
+        <origin xyz="${(pivot_l/2) + lock_o} 0 0" rpy="0 0 0"/>
         <parent link="${agent_namespace}_female_link"/>
         <child link="${agent_namespace}_pivot_link"/>
     </joint>
     <joint name="${agent_namespace}_pivot_base_joint" type="revolute">
-        <origin xyz="${0.02-pivot_o} 0 ${-pivot_zo}" rpy="0 0 0"/>
+        <origin xyz="${0.02-lock_o} 0 ${-pivot_zo}" rpy="0 0 0"/>
         <parent link="${agent_namespace}_pivot_link"/>
         <child link="${agent_namespace}_base_link"/>

Commit message: adding configurable root for modular robot

File: ros_ws/src/modular_robot/urdf/linkage.xacro (robot description, xacro)
@@ -108,16 +108,33 @@
         <child link="${agent_namespace}_cover_link"/>
     </joint>
-    <joint name="${agent_namespace}_female_pivot_joint" type="fixed">
-        <origin xyz="${(pivot_l/2) + lock_o} 0 0" rpy="0 0 0"/>
-        <parent link="${agent_namespace}_female_link"/>
-        <child link="${agent_namespace}_pivot_link"/>
-    </joint>
-    <joint name="${agent_namespace}_pivot_base_joint" type="revolute">
-        <origin xyz="${0.02-lock_o} 0 ${-pivot_zo}" rpy="0 0 0"/>
-        <parent link="${agent_namespace}_pivot_link"/>
-        <child link="${agent_namespace}_base_link"/>
-        <axis xyz="0 1 0"/>
-        <limit lower="${-pi/4}" upper="${pi/4}" effort="1.0" velocity="1.0"/>
-        <dynamics damping="0.3" friction="0.5"/>
-    </joint>
+    <xacro:if value="${first_link}">
+        <joint name="${agent_namespace}_female_pivot_joint" type="fixed">
+            <origin xyz="${-(pivot_l/2) - lock_o} 0 0" rpy="0 0 0"/>
+            <parent link="${agent_namespace}_pivot_link"/>
+            <child link="${agent_namespace}_female_link"/>
+        </joint>
+        <joint name="${agent_namespace}_pivot_base_joint" type="revolute">
+            <origin xyz="${-(0.02-lock_o)} 0 ${pivot_zo}" rpy="0 0 0"/>
+            <parent link="${agent_namespace}_base_link"/>
+            <child link="${agent_namespace}_pivot_link"/>
+            <axis xyz="0 1 0"/>
+            <limit lower="${-pi/4}" upper="${pi/4}" effort="1.0" velocity="1.0"/>
+            <dynamics damping="0.3" friction="0.5"/>
+        </joint>
+    </xacro:if>
+    <xacro:unless value="${first_link}">
+        <joint name="${agent_namespace}_female_pivot_joint" type="fixed">
+            <origin xyz="${(pivot_l/2) + lock_o} 0 0" rpy="0 0 0"/>
+            <parent link="${agent_namespace}_female_link"/>
+            <child link="${agent_namespace}_pivot_link"/>
+        </joint>
+        <joint name="${agent_namespace}_pivot_base_joint" type="revolute">
+            <origin xyz="${0.02-lock_o} 0 ${-pivot_zo}" rpy="0 0 0"/>
+            <parent link="${agent_namespace}_pivot_link"/>
+            <child link="${agent_namespace}_base_link"/>
+            <axis xyz="0 1 0"/>
+            <limit lower="${-pi/4}" upper="${pi/4}" effort="1.0" velocity="1.0"/>
+            <dynamics damping="0.3" friction="0.5"/>
+        </joint>
+    </xacro:unless>
 </robot>

File: ros_ws/src/modular_robot/urdf/modular_robot.urdf.xacro (robot description, xacro)
@@ -5,11 +5,21 @@
     <link name="footprint_link" />
     <!-- Call pipe_robot with agent_namespace -->
-    <xacro:pipe_robot agent_namespace="agent_n" include_gazebo="true"/>
-    <xacro:pipe_robot agent_namespace="agent_n2" include_gazebo="true"/>
-    <xacro:pipe_robot agent_namespace="agent_n3" include_gazebo="true"/>
+    <xacro:pipe_robot agent_namespace="agent_n" include_gazebo="true" first_link="true"/>
+    <xacro:pipe_robot agent_namespace="agent_n2" include_gazebo="true" first_link="false"/>
+    <xacro:pipe_robot agent_namespace="agent_n3" include_gazebo="true" first_link="false"/>
+    <xacro:unless value="${include_gazebo}">
+        <link name="world" />
+        <joint name="mobile_joint" type="prismatic">
+        <origin xyz="0 0 0" rpy="0 0 0"/>
+        <parent link="world"/>
+        <child link="footprint_link"/>
+        <axis xyz="1 0 0"/>
+        <limit lower="-1.0" upper="1.0" effort="100" velocity="1.0"/>
+    </joint>
+    </xacro:unless>
     <joint name="footprint_agent_n_joint" type="fixed">
         <origin xyz="0 0 0" rpy="0 0 0"/>
         <parent link="footprint_link"/>
-        <child link="agent_n_female_link"/>
+        <child link="agent_n_base_link"/>
     </joint>
     <joint name="agent_n_agent_n2_joint" type="fixed">

File: ros_ws/src/modular_robot/urdf/pipe_robot.xacro (robot description, xacro)
@@ -1,5 +1,5 @@
 <?xml version="1.0"?>
 <robot name="pipe_robot" xmlns:xacro="http://www.ros.org/wiki/xacro">
-    <xacro:macro name="pipe_robot" params="agent_namespace include_gazebo">
+    <xacro:macro name="pipe_robot" params="agent_namespace include_gazebo first_link">
         <!-- Include shared components -->
         <xacro:include filename="common.xacro"/>

File: ros_ws/src/pipe_swarm/urdf/linkage.xacro (robot description, xacro)
@@ -114,4 +114,5 @@
         <axis xyz="0 1 0"/>
         <limit lower="${-pi/4}" upper="${pi/4}" effort="0.5" velocity="0.5"/>
+        <dynamics damping="0.3" friction="0.5"/>
     </joint>
     <joint name="${agent_namespace}_base_neutral_joint" type="fixed">
