Commit message: setting base agent's female joint as fixed

File: ros_ws/src/modular_robot/urdf/linkage.xacro (robot description, xacro)
@@ -114,11 +114,11 @@
             <child link="${agent_namespace}_female_link"/>
         </joint>
-        <joint name="${agent_namespace}_pivot_base_joint" type="revolute">
+        <joint name="${agent_namespace}_pivot_base_joint" type="fixed">
             <origin xyz="${-(0.02-lock_o)} 0 ${pivot_zo}" rpy="0 0 0"/>
             <parent link="${agent_namespace}_base_link"/>
             <child link="${agent_namespace}_pivot_link"/>
-            <axis xyz="0 1 0"/>
+            <!-- <axis xyz="0 1 0"/>
             <limit lower="${-pi/4}" upper="${pi/4}" effort="1.0" velocity="1.0"/>
-            <dynamics damping="0.3" friction="0.5"/>
+            <dynamics damping="0.3" friction="0.5"/> -->
         </joint>
     </xacro:if>

File: ros_ws/src/modular_robot/urdf/modular_robot.urdf.xacro (robot description, xacro)
@@ -45,15 +45,4 @@
                 <plugin>gazebo_ros2_control/GazeboSystem</plugin>
             </hardware>
-            <joint name="agent_n_pivot_base_joint">
-                <command_interface name="position">
-                    <param name="min">-pi/2</param>
-                    <param name="max">pi/2</param>
-                </command_interface>
-                <state_interface name="position">
-                    <param name="initial_value">0.0</param>
-                </state_interface>
-                <state_interface name="velocity"/>
-                <state_interface name="effort"/>
-            </joint>
             <joint name="agent_n2_pivot_base_joint">
                 <command_interface name="position">

Commit message: updating modular robot weight

File: ros_ws/src/modular_robot/urdf/linkage.xacro (robot description, xacro)
@@ -1,5 +1,5 @@
 <?xml version="1.0"?>
 <robot name="linkage" xmlns:xacro="http://www.ros.org/wiki/xacro">
-    <xacro:property name="cover_m" value="0.1" />  <!-- mass /kg -->
+    <xacro:property name="cover_m" value="0.02" />  <!-- mass /kg -->
     <xacro:property name="cover_w" value="0.029" />  <!-- width /m -->
     <xacro:property name="cover_h" value="0.024" />  <!-- height /m -->
@@ -7,10 +7,10 @@
     <xacro:property name="cover_o" value="0.0045" />  <!-- offset /m -->
     <xacro:property name="cover_out" value="0.0015" />  <!-- extruded cover /m -->
-    <xacro:property name="male_m" value="0.1" />  <!-- mass /kg -->
+    <xacro:property name="male_m" value="0.0065" />  <!-- mass /kg -->
     <xacro:property name="male_w" value="0.014" />  <!-- width /m -->
     <xacro:property name="male_h" value="0.0128" />  <!-- length /m -->
     <xacro:property name="male_l" value="0.0054" />  <!-- height /m -->
     <xacro:property name="male_o" value="0.007" />  <!-- offset /m -->
-    <xacro:property name="pivot_m" value="0.1" />  <!-- mass /kg -->
+    <xacro:property name="pivot_m" value="0.014" />  <!-- mass /kg -->
     <xacro:property name="pivot_w" value="0.035" />  <!-- width /m -->
     <xacro:property name="pivot_h" value="0.024" />  <!-- height /m -->
@@ -18,5 +18,5 @@
     <xacro:property name="pivot_o" value="0.0075" />  <!-- offset /m -->
     <xacro:property name="pivot_zo" value="0.01" />  <!-- offset from centre of robot /m -->
-    <xacro:property name="female_m" value="0.1" />  <!-- mass /kg -->
+    <xacro:property name="female_m" value="0.00825" />  <!-- mass /kg -->
     <xacro:property name="female_w" value="0.02" />  <!-- width /m -->
     <xacro:property name="female_h" value="0.024" />  <!-- height /m -->

File: ros_ws/src/modular_robot/urdf/mobile_base.xacro (robot description, xacro)
@@ -1,5 +1,5 @@
 <?xml version="1.0" ?>
 <robot name="mobile_base" xmlns:xacro="http://www.ros.org/wiki/xacro">
-    <xacro:property name="base_m" value="1" />  <!-- mass /kg -->
+    <xacro:property name="base_m" value="0.25" />  <!-- mass /kg -->
     <xacro:property name="base_w" value="0.1045" />  <!-- width /m -->
     <xacro:property name="base_l" value="0.055" />  <!-- length /m -->

File: ros_ws/src/modular_robot/urdf/wheels.xacro (robot description, xacro)
@@ -1,5 +1,5 @@
 <?xml version="1.0"?>
 <robot name="wheels" xmlns:xacro="http://www.ros.org/wiki/xacro">
-    <xacro:property name="wheel_m" value="0.1" />  <!-- mass /kg -->
+    <xacro:property name="wheel_m" value="0.005" />  <!-- mass /kg -->
     <xacro:property name="wheel_r" value="0.015" />  <!-- radius /m -->
     <xacro:property name="wheel_l" value="0.008" />  <!-- length /m 8 or 3 -->
