Commit message: adding moveit with ros2 control to execute planned steps

File: ros_ws/src/modular_robot/urdf/modular_robot.urdf.xacro (robot description, xacro)
@@ -1,11 +1,11 @@
 <?xml version="1.0"?>
 <robot name="modular_robot" xmlns:xacro="http://www.ros.org/wiki/xacro">
-    <!-- Correct include syntax -->
     <xacro:include filename="pipe_robot.xacro"/>
+    <xacro:property name="include_gazebo" value="false" />
     <link name="footprint_link" />
     <!-- Call pipe_robot with agent_namespace -->
-    <xacro:pipe_robot agent_namespace="agent_n" include_gazebo="true"/>
-    <xacro:pipe_robot agent_namespace="agent_n2" include_gazebo="true"/>
-    <xacro:pipe_robot agent_namespace="agent_n3" include_gazebo="true"/>
+    <xacro:pipe_robot agent_namespace="agent_n" include_gazebo="${include_gazebo}"/>
+    <xacro:pipe_robot agent_namespace="agent_n2" include_gazebo="${include_gazebo}"/>
+    <xacro:pipe_robot agent_namespace="agent_n3" include_gazebo="${include_gazebo}"/>
     <joint name="footprint_agent_n_joint" type="fixed">
         <origin xyz="0 0 0" rpy="0 0 0"/>
@@ -30,41 +30,43 @@
     </gazebo>
     <!-- ros2_control Plugin -->
-    <ros2_control name="GazeboSimSystem" type="system">
-        <hardware>
-            <plugin>gazebo_ros2_control/GazeboSystem</plugin>
-        </hardware>
-        <joint name="agent_n_pivot_base_joint">
-            <command_interface name="position">
-                <param name="min">-pi/2</param>
-                <param name="max">pi/2</param>
-            </command_interface>
-            <state_interface name="position">
-                <param name="initial_value">0.0</param>
-            </state_interface>
-            <state_interface name="velocity"/>
-            <state_interface name="effort"/>
-        </joint>
-        <joint name="agent_n2_pivot_base_joint">
-            <command_interface name="position">
-                <param name="min">-pi/2</param>
-                <param name="max">pi/2</param>
-            </command_interface>
-            <state_interface name="position">
-                <param name="initial_value">0.0</param>
-            </state_interface>
-            <state_interface name="velocity"/>
-            <state_interface name="effort"/>
-        </joint>
-        <joint name="agent_n3_pivot_base_joint">
-            <command_interface name="position">
-                <param name="min">-pi/2</param>
-                <param name="max">pi/2</param>
-            </command_interface>
-            <state_interface name="position">
-                <param name="initial_value">0.0</param>
-            </state_interface>
-            <state_interface name="velocity"/>
-            <state_interface name="effort"/>
-        </joint>
-    </ros2_control>
+    <xacro:if value="${include_gazebo}">
+        <ros2_control name="GazeboSimSystem" type="system">
+            <hardware>
+                <plugin>gazebo_ros2_control/GazeboSystem</plugin>
+            </hardware>
+            <joint name="agent_n_pivot_base_joint">
+                <command_interface name="position">
+                    <param name="min">-pi/2</param>
+                    <param name="max">pi/2</param>
+                </command_interface>
+                <state_interface name="position">
+                    <param name="initial_value">0.0</param>
+                </state_interface>
+                <state_interface name="velocity"/>
+                <state_interface name="effort"/>
+            </joint>
+            <joint name="agent_n2_pivot_base_joint">
+                <command_interface name="position">
+                    <param name="min">-pi/2</param>
+                    <param name="max">pi/2</param>
+                </command_interface>
+                <state_interface name="position">
+                    <param name="initial_value">0.0</param>
+                </state_interface>
+                <state_interface name="velocity"/>
+                <state_interface name="effort"/>
+            </joint>
+            <joint name="agent_n3_pivot_base_joint">
+                <command_interface name="position">
+                    <param name="min">-pi/2</param>
+                    <param name="max">pi/2</param>
+                </command_interface>
+                <state_interface name="position">
+                    <param name="initial_value">0.0</param>
+                </state_interface>
+                <state_interface name="velocity"/>
+                <state_interface name="effort"/>
+            </joint>
+        </ros2_control>
+    </xacro:if>
 </robot>

Commit message: using moveit alongside gazebo

File: ros_ws/src/modular_robot/urdf/modular_robot.urdf.xacro (robot description, xacro)
@@ -5,7 +5,7 @@
     <link name="footprint_link" />
     <!-- Call pipe_robot with agent_namespace -->
-    <xacro:pipe_robot agent_namespace="agent_n" include_gazebo="${include_gazebo}"/>
-    <xacro:pipe_robot agent_namespace="agent_n2" include_gazebo="${include_gazebo}"/>
-    <xacro:pipe_robot agent_namespace="agent_n3" include_gazebo="${include_gazebo}"/>
+    <xacro:pipe_robot agent_namespace="agent_n" include_gazebo="true"/>
+    <xacro:pipe_robot agent_namespace="agent_n2" include_gazebo="true"/>
+    <xacro:pipe_robot agent_namespace="agent_n3" include_gazebo="true"/>
     <joint name="footprint_agent_n_joint" type="fixed">
         <origin xyz="0 0 0" rpy="0 0 0"/>

File: ros_ws/src/modular_robot_moveit_config/config/modular_robot.ros2_control.xacro (robot description, xacro)
@@ -6,6 +6,14 @@
             <hardware>
                 <!-- By default, set up controllers for simulation. This won't work on real hardware -->
-                <plugin>mock_components/GenericSystem</plugin>
+                <!-- <plugin>mock_components/GenericSystem</plugin> -->
+                <plugin>gazebo_ros2_control/GazeboSystem</plugin>
             </hardware>
+            <joint name="agent_n_pivot_base_joint">
+                <command_interface name="position"/>
+                <state_interface name="position">
+                  <param name="initial_value">${initial_positions['agent_n2_pivot_base_joint']}</param>
+                </state_interface>
+                <state_interface name="velocity"/>
+            </joint>
             <joint name="agent_n2_pivot_base_joint">
                 <command_interface name="position"/>

Commit message: correcting indentation and rviz

File: ros_ws/src/modular_robot/urdf/modular_robot.urdf.xacro (robot description, xacro)
@@ -11,10 +11,10 @@
         <link name="world" />
         <joint name="mobile_joint" type="prismatic">
-        <origin xyz="0 0 0" rpy="0 0 0"/>
-        <parent link="world"/>
-        <child link="footprint_link"/>
-        <axis xyz="1 0 0"/>
-        <limit lower="-1.0" upper="1.0" effort="100" velocity="1.0"/>
-    </joint>
+            <origin xyz="0 0 0" rpy="0 0 0"/>
+            <parent link="world"/>
+            <child link="footprint_link"/>
+            <axis xyz="1 0 0"/>
+            <limit lower="-1.0" upper="1.0" effort="100" velocity="1.0"/>
+        </joint>
     </xacro:unless>
     <joint name="footprint_agent_n_joint" type="fixed">

Commit message: adding prismatic joint to control robot planar movement

File: ros_ws/src/modular_robot/urdf/modular_robot.urdf.xacro (robot description, xacro)
@@ -2,25 +2,56 @@
 <robot name="modular_robot" xmlns:xacro="http://www.ros.org/wiki/xacro">
     <xacro:include filename="pipe_robot.xacro"/>
-    <xacro:property name="include_gazebo" value="false" />
+    <xacro:include filename="common.xacro"/>
+    <xacro:property name="include_gazebo" value="true" />
     <link name="footprint_link" />
+    <xacro:property name="prismatic_m" value="1.0" />  <!-- mass /kg -->
+    <xacro:property name="prismatic_w" value="0.01" />  <!-- width /m -->
+    <xacro:property name="prismatic_l" value="0.01" />  <!-- length /m -->
+    <xacro:property name="prismatic_h" value="0.01" />  <!-- height /m -->
+    <link name="prismatic_link">
+        <collision>
+            <origin xyz="0 0 0" rpy="0 0 0"/>
+            <geometry>
+                <box size="${prismatic_w} ${prismatic_l} ${prismatic_h}"/>
+            </geometry>
+        </collision>
+        <xacro:box_inertial m="${prismatic_m}" w="${prismatic_w}" l="${prismatic_l}" h="${prismatic_h}" xyz="0 0 0 " rpy="0 0 0"/>
+    </link>
     <!-- Call pipe_robot with agent_namespace -->
     <xacro:pipe_robot agent_namespace="agent_n" include_gazebo="true" first_link="true"/>
     <xacro:pipe_robot agent_namespace="agent_n2" include_gazebo="true" first_link="false"/>
     <xacro:pipe_robot agent_namespace="agent_n3" include_gazebo="true" first_link="false"/>
-    <xacro:unless value="${include_gazebo}">
-        <link name="world" />
+    <!-- <xacro:unless value="${include_gazebo}">
+        <link name="world_link" />
         <joint name="mobile_joint" type="prismatic">
             <origin xyz="0 0 0" rpy="0 0 0"/>
-            <parent link="world"/>
+            <parent link="world_link"/>
             <child link="footprint_link"/>
             <axis xyz="1 0 0"/>
             <limit lower="-1.0" upper="1.0" effort="100" velocity="1.0"/>
         </joint>
-    </xacro:unless>
-    <joint name="footprint_agent_n_joint" type="fixed">
+    </xacro:unless> -->
+    <joint name="footprint_prismatic_joint" type="fixed">
         <origin xyz="0 0 0" rpy="0 0 0"/>
         <parent link="footprint_link"/>
+        <child link="prismatic_link"/>
+    </joint>
+    <joint name="prismatic_agent_n_joint" type="prismatic">
+        <origin xyz="-0.02 0 0" rpy="0 0 0"/>
+        <parent link="prismatic_link"/>
         <child link="agent_n_base_link"/>
+        <axis xyz="1 0 0"/>
+        <limit lower="-0.3" upper="0.1" effort="100" velocity="0.05"/>
+        <dynamics damping="5.0" friction="2.0"/>
     </joint>
+    <!-- <transmission name="prismatic_agent_n_trans">
+        <type>transmission_interface/SimpleTransmission</type>
+        <joint name="prismatic_agent_n_joint">
+            <hardwareInterface>hardware_interface/PositionJointInterface</hardwareInterface>
+        </joint>
+        <actuator name="prismatic_agent_n_actuator">
+            <mechanicalReduction>1</mechanicalReduction>
+        </actuator>
+    </transmission> -->
     <joint name="agent_n_agent_n2_joint" type="fixed">
         <origin xyz="0 0 0" rpy="0 0 0"/>
@@ -67,4 +98,11 @@
                 <state_interface name="effort"/>
             </joint>
+            <joint name="prismatic_agent_n_joint">
+                <command_interface name="position"/>
+                <state_interface name="position">
+                    <param name="initial_value">0.0</param>
+                </state_interface>
+                <state_interface name="velocity"/>
+            </joint>
         </ros2_control>
     </xacro:if>

Commit message: motion planning with joint and planar in gazebo

File: ros_ws/src/modular_robot/urdf/modular_robot.urdf.xacro (robot description, xacro)
@@ -3,5 +3,5 @@
     <xacro:include filename="pipe_robot.xacro"/>
     <xacro:include filename="common.xacro"/>
-    <xacro:property name="include_gazebo" value="true" />
+    <xacro:property name="include_gazebo" value="false" />
     <link name="footprint_link" />
     <xacro:property name="prismatic_m" value="1.0" />  <!-- mass /kg -->
@@ -22,14 +22,4 @@
     <xacro:pipe_robot agent_namespace="agent_n2" include_gazebo="true" first_link="false"/>
     <xacro:pipe_robot agent_namespace="agent_n3" include_gazebo="true" first_link="false"/>
-    <!-- <xacro:unless value="${include_gazebo}">
-        <link name="world_link" />
-        <joint name="mobile_joint" type="prismatic">
-            <origin xyz="0 0 0" rpy="0 0 0"/>
-            <parent link="world_link"/>
-            <child link="footprint_link"/>
-            <axis xyz="1 0 0"/>
-            <limit lower="-1.0" upper="1.0" effort="100" velocity="1.0"/>
-        </joint>
-    </xacro:unless> -->
     <joint name="footprint_prismatic_joint" type="fixed">
         <origin xyz="0 0 0" rpy="0 0 0"/>
@@ -45,13 +35,4 @@
         <dynamics damping="5.0" friction="2.0"/>
     </joint>
-    <!-- <transmission name="prismatic_agent_n_trans">
-        <type>transmission_interface/SimpleTransmission</type>
-        <joint name="prismatic_agent_n_joint">
-            <hardwareInterface>hardware_interface/PositionJointInterface</hardwareInterface>
-        </joint>
-        <actuator name="prismatic_agent_n_actuator">
-            <mechanicalReduction>1</mechanicalReduction>
-        </actuator>
-    </transmission> -->
     <joint name="agent_n_agent_n2_joint" type="fixed">
         <origin xyz="0 0 0" rpy="0 0 0"/>

File: ros_ws/src/modular_robot_moveit_config/config/modular_robot.ros2_control.xacro (robot description, xacro)
@@ -6,6 +6,6 @@
             <hardware>
                 <!-- By default, set up controllers for simulation. This won't work on real hardware -->
-                <plugin>mock_components/GenericSystem</plugin>
-                <!-- <plugin>gazebo_ros2_control/GazeboSystem</plugin> -->
+                <!-- <plugin>mock_components/GenericSystem</plugin> -->
+                <plugin>gazebo_ros2_control/GazeboSystem</plugin>
             </hardware>
             <joint name="agent_n2_pivot_base_joint">

Commit message: updating robot to update movement range

File: ros_ws/src/modular_robot/urdf/modular_robot.urdf.xacro (robot description, xacro)
@@ -5,5 +5,5 @@
     <xacro:property name="include_gazebo" value="false" />
     <link name="footprint_link" />
-    <xacro:property name="prismatic_m" value="1.0" />  <!-- mass /kg -->
+    <xacro:property name="prismatic_m" value="0.3" />  <!-- mass /kg -->
     <xacro:property name="prismatic_w" value="0.01" />  <!-- width /m -->
     <xacro:property name="prismatic_l" value="0.01" />  <!-- length /m -->
@@ -28,9 +28,9 @@
     </joint>
     <joint name="prismatic_agent_n_joint" type="prismatic">
-        <origin xyz="-0.02 0 0" rpy="0 0 0"/>
+        <origin xyz="-0.06 0 0" rpy="0 0 0"/>
         <parent link="prismatic_link"/>
         <child link="agent_n_base_link"/>
         <axis xyz="1 0 0"/>
-        <limit lower="-0.3" upper="0.1" effort="100" velocity="0.05"/>
+        <limit lower="-0.1" upper="0.27" effort="100" velocity="0.05"/>
         <dynamics damping="5.0" friction="2.0"/>
     </joint>
