Commit message: modifying moveit to not use base robot

File: ros_ws/src/modular_robot_moveit_config/config/modular_robot.ros2_control.xacro (robot description, xacro)
@@ -8,11 +8,4 @@
                 <plugin>mock_components/GenericSystem</plugin>
             </hardware>
-            <joint name="agent_n_pivot_base_joint">
-                <command_interface name="position"/>
-                <state_interface name="position">
-                  <param name="initial_value">${initial_positions['agent_n_pivot_base_joint']}</param>
-                </state_interface>
-                <state_interface name="velocity"/>
-            </joint>
             <joint name="agent_n2_pivot_base_joint">
                 <command_interface name="position"/>

Commit message: adding planar movement to demo moveit with controllers

File: ros_ws/src/modular_robot_moveit_config/config/modular_robot.ros2_control.xacro (robot description, xacro)
@@ -6,6 +6,6 @@
             <hardware>
                 <!-- By default, set up controllers for simulation. This won't work on real hardware -->
-                <!-- <plugin>mock_components/GenericSystem</plugin> -->
-                <plugin>gazebo_ros2_control/GazeboSystem</plugin>
+                <plugin>mock_components/GenericSystem</plugin>
+                <!-- <plugin>gazebo_ros2_control/GazeboSystem</plugin> -->
             </hardware>
             <joint name="agent_n_pivot_base_joint">
@@ -30,4 +30,11 @@
                 <state_interface name="velocity"/>
             </joint>
+            <joint name="mobile_joint">
+                <command_interface name="position"/>
+                <state_interface name="position">
+                  <param name="initial_value">${initial_positions['mobile_joint']}</param>
+                </state_interface>
+                <state_interface name="velocity"/>
+            </joint>
         </ros2_control>
     </xacro:macro>

Commit message: planning path with x translation

File: ros_ws/src/modular_robot_moveit_config/config/modular_robot.ros2_control.xacro (robot description, xacro)
@@ -9,11 +9,4 @@
                 <!-- <plugin>gazebo_ros2_control/GazeboSystem</plugin> -->
             </hardware>
-            <joint name="agent_n_pivot_base_joint">
-                <command_interface name="position"/>
-                <state_interface name="position">
-                  <param name="initial_value">${initial_positions['agent_n2_pivot_base_joint']}</param>
-                </state_interface>
-                <state_interface name="velocity"/>
-            </joint>
             <joint name="agent_n2_pivot_base_joint">
                 <command_interface name="position"/>

Commit message: updating moveit config with prismatic joint

File: ros_ws/src/modular_robot_moveit_config/config/modular_robot.ros2_control.xacro (robot description, xacro)
@@ -23,8 +23,8 @@
                 <state_interface name="velocity"/>
             </joint>
-            <joint name="mobile_joint">
+            <joint name="prismatic_agent_n_joint">
                 <command_interface name="position"/>
                 <state_interface name="position">
-                  <param name="initial_value">${initial_positions['mobile_joint']}</param>
+                  <param name="initial_value">${initial_positions['prismatic_agent_n_joint']}</param>
                 </state_interface>
                 <state_interface name="velocity"/>
